File: felles-devboard/felles-devboard/felles-devboard.kicad_sch (KiCad schematic)
At the start: 17 parts, among them U1 TPS26400PWP, U2 173950336, U3 TCAN332G, U4 BME280

Commit message: more progress
Parts:
- added C10: 100n, symbol Device:C
- added D1: SOT143-4L_8240136, Diode_SMD_Wurth:D_Wurth_WE-TVS-SOT143-4L, symbol Diode_Wurth_WE-TVS:SOT143-4L_8240136
- added Q1: STANDARD_140356145200, Optocoupler_SMD_Wurth:Q_Wurth_WL-OCPT_SOP4-STANDARD, symbol Optocoupler_Wurth_WL-OCPT:STANDARD_140356145200
- added R4, R5, R6, R7: R, symbol Device:R
- added U5: WE-TVS-824015043, Package_TO_SOT_SMD:SOT-23-6, symbol Power_Protection:WE-TVS-824015043
Connections:
- net GNDREF: now also D1.1 (GND), Q1.2 (C), U5.2 (GND)
- net GNDS: now also U1.6 (MODE), C10.2, Q1.3 (E), R4.2, R5.2
- net +3V3: now reaches C5.1, C6.1, C7.1, C8.1, C9.1, U2.3 (VOUT), U3.3 (VCC), U4.6 (VDDIO), U4.8 (VDD)
- net +3V3: now also D1.4 (VDD), U5.5 (VBUS)
- net at U3.1 (TXD): now also D1.3 (2)
- net at U3.4 (RXD): now also D1.2 (1)
- net at U3.6 (CANL): now also R7.2
- net at U3.7 (CANH): now also R7.1
- net at U1.10 (IMON): now also R4.1
- net at U1.11 (ILIM): now also R5.1
- net at U1.12 (dVdT): now also C10.1
- net at U1.7 (~{SHDN}): now also Q1.4 (C)
- new net: Q1.1 (A), R6.2
