File: torpedokontroller/torpedokontroller.kicad_sch (KiCad schematic)
At the start: 3 parts, among them IC1 STM32C542RCT6, IC2 TCAN3414DR, Q1 STANDARD_140356145200

Commit message: Torpedo v0.1
first version of torpedo PCB scematic
still early development
finner ut av det :))
Parts:
- removed Q1: STANDARD_140356145200, Optocoupler_SMD_Wurth:Q_Wurth_WL-OCPT_SOP4-STANDARD, symbol WL-OCPT SOP-4:STANDARD_140356145200
- added C1, C2, C3, C4: 4.7 uF, Capacitor_SMD_Wurth:C_Wurth_WCAP-CSGP-1210_H2.5, symbol Capacitor_Wurth_WCAP-CSGP:1210_H2.5_885012209048
- added C10: 1u, symbol Device:C
- added C5, C6: 22 uF, Capacitor_SMD_Wurth:C_Wurth_WCAP-CSGP-1210_H2.5, symbol Capacitor_Wurth_WCAP-CSGP:1210_H2.5_885012109014
- added C8, C9: 100n, symbol Device:C
- added IC4: TCAN3414DR, Samacsys:SOIC127P600X175-8N, symbol Samacsys:TCAN3414DR
- added L1: 1.0 uH, Inductor_SMD_Wurth:L_Wurth_WE-PD2-4532, symbol Inductor_Wurth_WE-PD2:4532_7447730
- added Q4: PMOS, Package_DIP:DIP-24_W7.62mm, symbol Simulation_SPICE:PMOS
- added Q6: STANDARD_140356145200, Optocoupler_SMD_Wurth:Q_Wurth_WL-OCPT_SOP4-STANDARD, symbol WL-OCPT SOP-4:STANDARD_140356145200
- added R1: 470k, symbol Device:R
- added R2: 15k, symbol Device:R
- added R3: 30k, symbol Device:R
- added R4: 24k9, symbol Device:R
- added R5: 100k, symbol Device:R
- added R6: 1K, symbol Device:R
- added R8: 10k, symbol Device:R
- added U1: TPS26400PWP, Package_SO:HTSSOP-16-1EP_4.4x5mm_P0.65mm_EP3.4x5mm_Mask2.66x2.46mm_ThermalVias, symbol Power_Management:TPS26400PWP
- added U2: 173950336, MagIC_THT_Wurth:U_Wurth_WPME-FDSM_17395xx36, symbol MagIC_Wurth_WPME-FDSM:173950336
- added U4: BME280, Package_LGA:Bosch_LGA-8_2.5x2.5mm_P0.65mm_ClockwisePinNumbering, symbol Sensor:BME280
Connections:
- net at IC1.33 (PB12): now also IC2.4 (RXD)
- net at IC1.34 (PB13): now also IC2.1 (TXD)
- net at IC1.35 (PB14): now also IC2.8 (STB)
- net at IC1.36 (PB15): now also IC2.5 (SHDNVIO)
- net at IC1.51 (PC10): now also Q6.3 (E), R5.1, U1.7 (~{SHDN})
- net at IC1.52 (PC11): now also Q4.2 (G)
- net at IC1.57 (PB5): now also IC4.5 (SHDNVIO)
- net at IC1.58 (PB6): now also IC4.8 (STB)
- net at IC1.59 (PB7): now also IC4.1 (TXD)
- net at IC1.61 (PB8): now also IC4.4 (RXD)
- net Earth: now reaches IC2.2 (GND)
- net Earth: now also IC4.2 (GND), R5.2, R6.2
- net 3V3: now reaches IC2.3 (VCC)
- new net: R1.1, U1.1 (IN), U1.2 (IN)
- new net: R1.2, R2.1, U1.3 (UVLO)
- new net: C1.1, C2.1, L1.1, U1.15 (OUT), U1.16 (OUT)
- new net: C10.1, U1.12 (dVdT)
- new net: R2.2, R3.1, U1.5 (OVP)
- new net: Q6.2 (C), R6.1
- new net: C3.1, C4.1, L1.2, U2.1 (VIN)
- new net: Q4.1 (D), Q6.4 (C)
- new net: R4.1, U1.10 (IMON)
- new net: R8.1, U1.11 (ILIM)
- new net +3V3: C5.1, C6.1, C8.1, C9.1, U2.3 (VOUT), U4.6 (VDDIO), U4.8 (VDD)
- new net GNDREF: C1.2, C2.2, C3.2, C4.2, C5.2, C6.2, C8.2, C9.2, U1.9 (GND), U2.2 (GND), U4.1 (GND), U4.7 (GND)
- new net GNDS: C10.2, R3.2, R4.2, R8.2, U1.17 (RTN), U1.6 (MODE), U1.8 (RTN)
Other:
- moved on the sheet: IC1, IC2

Commit message: Torpedo v0.2
Fiksa ting, fjerna ting, la til ting
fortsatt nokså tidlig i prosessen
gruppert ting wiiii
Parts:
- removed IC2: TCAN3414DR, Samacsys:SOIC127P600X175-8N, symbol Samacsys:TCAN3414DR
- removed U2: 173950336, MagIC_THT_Wurth:U_Wurth_WPME-FDSM_17395xx36, symbol MagIC_Wurth_WPME-FDSM:173950336
- added C11: 1u, symbol Device:C
- added C12, C7: 4.7 uF, Capacitor_SMD_Wurth:C_Wurth_WCAP-CSGP-1210_H2.5, symbol Capacitor_Wurth_WCAP-CSGP:1210_H2.5_885012209048
- added IC5: TCAN3414DR, Samacsys:SOIC127P600X175-8N, symbol Samacsys:TCAN3414DR
- added J1: USB_C_Receptacle_USB2.0_14P, Package_DFN_QFN:WDFN-10-1EP_3x3mm_P0.5mm_EP1.8x2.5mm, symbol Connector:USB_C_Receptacle_USB2.0_14P
- added R10: 15k, symbol Device:R
- added R11: 30k, symbol Device:R
- added R12: 10k, symbol Device:R
- added R13: 24k9, symbol Device:R
- added R9: 470k, symbol Device:R
- added U2: TPS26400PWP, Package_SO:HTSSOP-16-1EP_4.4x5mm_P0.65mm_EP3.4x5mm_Mask2.66x2.46mm_ThermalVias, symbol Power_Management:TPS26400PWP
- added U3: 173950336, MagIC_THT_Wurth:U_Wurth_WPME-FDSM_17395xx36, symbol MagIC_Wurth_WPME-FDSM:173950336
Connections:
- net +3V3 is gone; now on net 3.3v: C5.1, C6.1, C8.1, C9.1, U4.6 (VDDIO), U4.8 (VDD)
- net Earth: now also IC5.2 (GND), J1.A1 (GND), J1.A12 (GND), J1.B1 (GND), J1.B12 (GND)
- net GNDREF: now also C12.2, C7.2, U2.9 (GND), U3.2 (GND)
- net GNDS: now also C11.2, R11.2, R12.2, R13.2, U2.17 (RTN), U2.6 (MODE), U2.8 (RTN)
- net at C1.1, C2.1, L1.1: now also U2.15 (OUT), U2.16 (OUT); no longer U1.15 (OUT), U1.16 (OUT)
- net 3.3v: now reaches IC1.19 (VDD_1)
- net 3.3v: now also IC1.32 (VDD_2), IC1.48 (VDD_3), IC1.64 (VDD_4), IC4.3 (VCC), Q4.3 (S), C12.1, C7.1, IC5.3 (VCC), U3.3 (VOUT)
- net tcan2_RX: now reaches IC1.33 (PB12)
- net tcan2_RX: now also IC5.4 (RXD)
- net tcan2_TX: now reaches IC1.34 (PB13)
- net tcan2_TX: now also IC5.1 (TXD)
- net tcan2_STB: now reaches IC1.35 (PB14)
- net tcan2_STB: now also IC5.8 (STB)
- net tcan2_SHDNVIO: now reaches IC1.36 (PB15)
- net USB_D-: now reaches IC1.44 (PA11)
- net USB_D-: now also J1.A7 (D-), J1.B7 (D-)
- net USB_D+: now reaches IC1.45 (PA12)
- net USB_D+: now also J1.A6 (D+), J1.B6 (D+)
- net OPT_Output: now reaches IC1.51 (PC10), Q6.3 (E), R5.1, U1.7 (~{SHDN})
- net MCU_Killswitch: now reaches IC1.52 (PC11), Q4.2 (G)
- net tcan1_SHDNIVO: now reaches IC1.57 (PB5), IC4.5 (SHDNVIO)
- net tcan1_STB: now reaches IC1.58 (PB6), IC4.8 (STB)
- net tcan1_TX: now reaches IC1.59 (PB7), IC4.1 (TXD)
- net tcan1_RX: now reaches IC1.61 (PB8), IC4.4 (RXD)
- net at C3.1, C4.1, L1.2: now also U3.1 (VIN)
- net tcan1_L: now reaches IC4.6 (CANL)
- net tcan1_H: now reaches IC4.7 (CANH)
- new net: R13.1, U2.10 (IMON)
- new net: R12.1, U2.11 (ILIM)
- new net: C11.1, U2.12 (dVdT)
- new net: R10.1, R9.2, U2.3 (UVLO)
- new net: R10.2, R11.1, U2.5 (OVP)
- new net: U1.15 (OUT), U1.16 (OUT)
- new net: J1.A4 (VBUS), J1.A9 (VBUS), J1.B4 (VBUS), J1.B9 (VBUS)
- new net tcan2_H: IC5.7 (CANH)
- new net tcan2_L: IC5.6 (CANL)
- new net tcan2_SHDNIVO: IC5.5 (SHDNVIO)
- new net v-batt: R9.1, U2.1 (IN), U2.2 (IN)
Other:
- added sheet TCAN_1 (bus) (untitled.kicad_sch)
- added sheet tcan_2 (servo) (tcan2.kicad_sch)
- added sheet v-batt_to_3v3 (v-batt_to_3v3.kicad_sch)
- moved on the sheet: C10, C8, C9, IC1, IC4, Q4, Q6, R1, R2, R3, R4, R5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
