File: torpedokontroller/torpedokontroller.kicad_sch (KiCad schematic)
At the start: 5 parts, among them J1 USB_C_Receptacle_USB2.0_14P, Q4 PMOS, Q6 STANDARD_140356145200

Commit message: Torpedo v0.4
Proper nesting
improved power handling
fixed efuse FLT LEDs
Better layout, descriptions and setup
and more stuff idk
Parts:
- removed J1: USB_C_Receptacle_USB2.0_14P, Package_DFN_QFN:WDFN-10-1EP_3x3mm_P0.5mm_EP1.8x2.5mm, symbol Connector:USB_C_Receptacle_USB2.0_14P
- removed Q4: PMOS, Package_DIP:DIP-24_W7.62mm, symbol Simulation_SPICE:PMOS
- removed Q6: STANDARD_140356145200, Optocoupler_SMD_Wurth:Q_Wurth_WL-OCPT_SOP4-STANDARD, symbol WL-OCPT SOP-4:STANDARD_140356145200
- removed R5: 100k, symbol Device:R
- removed R6: 1K, symbol Device:R
Other:
- removed sheet CAN BUS
- removed sheet CAN SERVO
- removed sheet Microprocessor
- removed sheet Microprocessor Power
- removed sheet Telematic (BME280)
- removed sheet V-batt to Servo
- added sheet Input (input.kicad_sch)
- added sheet output (output.kicad_sch)
- added sheet processing (processing.kicad_sch)
