File: torpedokontroller/torpedokontroller.kicad_sch (KiCad schematic)
At the start: 0 parts

Commit message: v 0.6
New MCU package
Added SWD, Rest and boot
Moved USB2.0 to MCU page
Other small changes
Other:
- sheet Input ports: added none; removed USB_D+, USB_D-
- sheet processing ports: added none; removed USB_D+, USB_D-
Changed lines of the file:
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@@
 	(paper "A5")
 	(title_block
-		(date "2026-10-03")
+		(date "2026-10-07")
 		(comment 1 "Simon Torvund")
 	)
@@
 	(wire
 		(pts
-			(xy 66.04 76.2) (xy 80.01 76.2)
-		)
-		(stroke
-			(width 0)
-			(type default)
-		)
-	)
-	(wire
-		(pts
 			(xy 116.84 59.69) (xy 129.54 59.69)
 		)
@@
 	(wire
 		(pts
-			(xy 66.04 72.39) (xy 80.01 72.39)
-		)
-		(stroke
-			(width 0)
-			(type default)
-		)
-	)
-	(wire
-		(pts
 			(xy 66.04 59.69) (xy 80.01 59.69)
 		)
@@
 	)
 	(label "Check resistor values for LEDs"
-		(at 33.02 115.57 0)
+		(at 33.02 113.03 0)
 		(effects
 			(font
@@
 		)
 	)
-	(label "New MCU package"
-		(at 33.02 113.03 0)
-		(effects
-			(font
-				(size 1.27 1.27)
-			)
-			(justify left bottom)
-		)
-	)
 	(label "BMS pogopads"
 		(at 33.02 110.49 0)
@@
 		)
 	)
-	(label "Boot, reset, and clock MCU pins?"
+	(label "Oscillator"
 		(at 33.02 107.95 0)
 		(effects
@@
 			)
 		)
-		(pin "CAN2_RX" input
+		(pin "CAN2_RX" output
 			(at 80.01 41.91 180)
 			(effects
@@
 			)
 		)
-		(pin "CAN1_RX" input
+		(pin "CAN1_RX" output
 			(at 116.84 41.91 0)
 			(effects
@@
 		(pin "SPI1_MOSI" output
 			(at 80.01 63.5 180)
-			(effects
-				(font
-					(size 1.27 1.27)
-				)
-				(justify left)
-			)
-		)
-		(pin "USB_D+" input
-			(at 80.01 72.39 180)
-			(effects
-				(font
-					(size 1.27 1.27)
-				)
-				(justify left)
-			)
-		)
-		(pin "USB_D-" input
-			(at 80.01 76.2 180)
 			(effects
 				(font
@@
 			(effects
 				(font
-					(size 1.27 1.27)
-				)
-				(justify right)
-			)
-		)
-		(pin "USB_D+" output
-			(at 66.04 72.39 0)
-			(effects
-				(font
-					(size 1.27 1.27)
-				)
-				(justify right)
-			)
-		)
-		(pin "USB_D-" output
-			(at 66.04 76.2 0)
-			(effects
-				(font

Commit message: v 0.7
fiksa ting la til ting fjerna ting
Other:
- sheet output ports: added none; removed CANH, CANL, vdd_servo

Commit message: v 0.8
Fixed one billion things
tvs
many values
connections
cleaned up
Other:
- sheet output ports: added D_OC, MCU_KillSwitch; removed DOC, MCU_killswitch, OPT_output
- sheet processing ports: added D_OC, MCU_KillSwitch; removed DOC, MCU_killSwitch, OPT_output

Commit message: v 1.0
Ferdigish

CAN tvs-packages
Ground hook
Test pads
fixed some i/o issues
Changed lines of the file:
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@@
 			)
 		)
-		(pin "CAN2_RX" output
+		(pin "CAN2_RX" input
 			(at 80.01 36.83 180)
 			(effects
@@
 			)
 		)
-		(pin "CAN1_RX" output
+		(pin "CAN1_RX" input
 			(at 116.84 36.83 0)
 			(effects

Commit message: post-schematic_review 💯
fixed stuff
added stuff
GND is good
I2C BME280
memes
fixed pins
more stuff
💯
Other:
- sheet Input ports: added IMON_SMALL, SDI; removed CSB, SPI1_MISO, SPI1_MOIS
- sheet output ports: added IMON_BIG; removed IMON
- sheet processing ports: added IMON_BIG, IMON_SMALL, SDI; removed CSB, IMON, SPI1_MISO, SPI1_MOSI
Changed lines of the file:
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@@
 	(paper "A5")
 	(title_block
-		(date "2026-10-21")
+		(date "2026-10-23")
 		(comment 1 "Simon Torvund")
 	)
@@
 	(wire
 		(pts
+			(xy 116.84 58.42) (xy 129.54 58.42)
+		)
+		(stroke
+			(width 0)
+			(type default)
+		)
+	)
+	(wire
+		(pts
+			(xy 116.84 33.02) (xy 129.54 33.02)
+		)
+		(stroke
+			(width 0)
+			(type default)
+		)
+	)
+	(wire
+		(pts
 			(xy 66.04 58.42) (xy 80.01 58.42)
 		)
@@
 	(wire
 		(pts
-			(xy 116.84 58.42) (xy 129.54 58.42)
-		)
-		(stroke
-			(width 0)
-			(type default)
-		)
-	)
-	(wire
-		(pts
-			(xy 116.84 33.02) (xy 129.54 33.02)
-		)
-		(stroke
-			(width 0)
-			(type default)
-		)
-	)
-	(wire
-		(pts
 			(xy 116.84 36.83) (xy 129.54 36.83)
 		)
@@
 		(pts
 			(xy 116.84 46.99) (xy 129.54 46.99)
-		)
-		(stroke
-			(width 0)
-			(type default)
-		)
-	)
-	(wire
-		(pts
-			(xy 66.04 54.61) (xy 80.01 54.61)
 		)
 		(stroke
@@
 			)
 		)
-		(pin "CSB" output
+		(pin "SDI" input
 			(at 80.01 46.99 180)
 			(effects
@@
 			)
 		)
-		(pin "SPI1_MISO" input
-			(at 80.01 54.61 180)
-			(effects
-				(font
-					(size 1.27 1.27)
-				)
-				(justify left)
-			)
-		)
-		(pin "SPI1_MOSI" output
-			(at 80.01 58.42 180)
-			(effects
-				(font
-					(size 1.27 1.27)
-				)
-				(justify left)
-			)
-		)
 		(pin "D_OC" input
 			(at 116.84 50.8 0)
@@
 			)
 		)
-		(pin "IMON" input
+		(pin "IMON_BIG" input
 			(at 116.84 58.42 0)
 			(effects
@@
 				)
 				(justify right)
+			)
+		)
+		(pin "IMON_SMALL" input
+			(at 80.01 58.42 180)
+			(effects
+				(font
+					(size 1.27 1.27)
+				)
+				(justify left)
 			)
 		)
@@
 			)
 		)
-		(pin "IMON" output
+		(pin "IMON_BIG" output
 			(at 129.54 58.42 180)
 			(effects
@@
 			)
 		)
-		(pin "CSB" input
+		(pin "SDI" output
 			(at 66.04 46.99 0)
 			(effects
@@
 			)
 		)
-		(pin "SPI1_MISO" output
-			(at 66.04 54.61 0)
-			(effects
-				(font
-					(size 1.27 1.27)
-				)
-				(justify right)
-			)
-		)
-		(pin "SPI1_MOIS" input
-			(at 66.04 58.42 0)
-			(effects
-				(font
-					(size 1.27 1.27)
-				)
-				(justify right)
-			)
-		)
 		(pin "CAN2_RX" output
 			(at 66.04 36.83 0)
@@
 			(effects
 				(font
+					(size 1.27 1.27)
+				)
+				(justify right)
+			)
+		)
+		(pin "IMON_SMALL" output
+			(at 66.04 58.42 0)
+			(effects
+				(font
