File: torpedokontroller/Microprocessor.kicad_sch (KiCad schematic)
At the start: 1 part, among them IC2 STM32C542RCT6

Commit message: Torpedo v0.4
Proper nesting
improved power handling
fixed efuse FLT LEDs
Better layout, descriptions and setup
and more stuff idk
Parts:
- added D4: green, symbol Device:LED
- added D5: yellow, symbol Device:LED
- added D6: red, symbol Device:LED
- added R19, R20, R4: 1k, symbol Device:R
Connections:
- net at IC2.10 (PC2): now also R20.2
- net at IC2.8 (PC0): now also R4.2
- net at IC2.9 (PC1): now also R19.2
- new net: D6.2 (A), R20.1
- new net: D4.2 (A), R4.1
- new net: D5.2 (A), R19.1
- new net Earth: D4.1 (K), D5.1 (K), D6.1 (K)
Other:
- note added: "LEDs to signal MCU state:"
