File: torpedokontroller/Microprocessor_Power.kicad_sch (KiCad schematic)
At the start: 15 parts, among them U5 TPS26400PWP, U6 173950336

Commit message: Torpedo v0.4
Proper nesting
improved power handling
fixed efuse FLT LEDs
Better layout, descriptions and setup
and more stuff idk
Parts:
- added D1: blue, symbol Device:LED
- added D2: red, symbol Device:LED
- added R1, R2: 1k, symbol Device:R
- added R5: 10k, symbol Device:R
Connections:
- net +3.3V: now also R1.1
- net GNDREF: now also D1.1 (K), D2.1 (K)
- net at C15.1, C7.1, L2.1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: now also R5.1
- net at U5.14 (~{FLT}): now also R2.1, R5.2
- new net: D2.2 (A), R2.2
- new net: D1.2 (A), R1.2
- no-connect marks 0 -> 1
Other:
- moved on the sheet: C14, C15, C16, C17, C18, C19, C7, L2, R14, R15, R16, R17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
