File: torpedokontroller/V-batt_to_Servo.kicad_sch (KiCad schematic)
At the start: 5 parts, among them J1 USB_C_Receptacle_USB2.0_14P, Q4 PMOS, Q6 STANDARD_140356145200

Commit message: Torpedo v0.3
Proper pages
Telematic sensor
improved visuals / cleraty
fixde stuff moved stuff removed stuff :)
Parts:
- removed J1: USB_C_Receptacle_USB2.0_14P, Package_DFN_QFN:WDFN-10-1EP_3x3mm_P0.5mm_EP1.8x2.5mm, symbol Connector:USB_C_Receptacle_USB2.0_14P
- removed Q4: PMOS, Package_DIP:DIP-24_W7.62mm, symbol Simulation_SPICE:PMOS
- removed Q6: STANDARD_140356145200, Optocoupler_SMD_Wurth:Q_Wurth_WL-OCPT_SOP4-STANDARD, symbol WL-OCPT SOP-4:STANDARD_140356145200
- removed R5: 100k, symbol Device:R
- removed R6: 1K, symbol Device:R
- added C11: 1u, symbol Device:C
- added Q5: PMOS, Package_DIP:DIP-24_W7.62mm, symbol Simulation_SPICE:PMOS
- added Q7: STANDARD_140356145200, Optocoupler_SMD_Wurth:Q_Wurth_WL-OCPT_SOP4-STANDARD, symbol WL-OCPT SOP-4:STANDARD_140356145200
- added R10: 30k, symbol Device:R
- added R11: 10k, symbol Device:R
- added R12: 24k9, symbol Device:R
- added R13: 100k, symbol Device:R
- added R7: 470k, symbol Device:R
- added R8: 1K, symbol Device:R
- added R9: 15k, symbol Device:R
- added U2: TPS26400PWP, Package_SO:HTSSOP-16-1EP_4.4x5mm_P0.65mm_EP3.4x5mm_Mask2.66x2.46mm_ThermalVias, symbol Power_Management:TPS26400PWP
Connections:
- net +3.3V: now also Q5.3 (S)
- net Earth: now also R13.2, R8.2
- net vdd_servo: now also U2.15 (OUT), U2.16 (OUT)
- new net: R7.2, R9.1, U2.3 (UVLO)
- new net: R10.1, R9.2, U2.5 (OVP)
- new net: R12.1, U2.10 (IMON)
- new net: R11.1, U2.11 (ILIM)
- new net: C11.1, U2.12 (dVdT)
- new net: Q7.3 (E), R13.1, U2.7 (~{SHDN})
- new net: Q7.2 (C), R8.1
- new net: Q5.1 (D), Q7.4 (C)
- new net GNDREF: U2.9 (GND)
- new net GNDS: C11.2, R10.2, R11.2, R12.2, U2.17 (RTN), U2.6 (MODE), U2.8 (RTN)
- new net MCU_killswitch: Q5.2 (G)
- new net v_batt: R7.1, U2.1 (IN), U2.2 (IN)
- new net v_batt_opt: Q7.1 (A)
Other:
- removed sheet CAN BUS
- removed sheet CAN SERVO
- removed sheet Microprocessor
- removed sheet Microprocessor Power
- removed sheet Telematic (BME280)
- removed sheet V-batt to Servo
- note added: "Trenger en regulator lwk"

Commit message: Torpedo v0.4
Proper nesting
improved power handling
fixed efuse FLT LEDs
Better layout, descriptions and setup
and more stuff idk
Parts:
- added D7: blue, symbol Device:LED
- added D8: red, symbol Device:LED
- added R21, R22: 1k, symbol Device:R
- added R3: 10k, symbol Device:R
Connections:
- net v_batt_opt is gone; now on net v_batt: Q7.1 (A)
- net GNDREF: now also D7.1 (K), D8.1 (K)
- net vdd_servo: now also R21.1, R3.1
- net at U2.14 (~{FLT}): now also R22.1, R3.2
- new net: D8.2 (A), R22.2
- new net: D7.2 (A), R21.2
