File: torpedokontroller/tcan2.kicad_sch (KiCad schematic)
At the start: 0 parts

Commit message: Torpedo v0.3
Proper pages
Telematic sensor
improved visuals / cleraty
fixde stuff moved stuff removed stuff :)
Parts:
- added C13: 4.7 uF, Capacitor_SMD_Wurth:C_Wurth_WCAP-CSGP-1210_H2.5, symbol Capacitor_Wurth_WCAP-CSGP:1210_H2.5_885012209048
- added IC7: TCAN3414DR, Samacsys:SOIC127P600X175-8N, symbol Samacsys:TCAN3414DR
Connections:
- new net +3.3V: C13.1, IC7.3 (VCC)
- new net CANH: IC7.7 (CANH)
- new net CANL: IC7.6 (CANL)
- new net CANRX: IC7.4 (RXD)
- new net CANTX: IC7.1 (TXD)
- new net Earth: IC7.2 (GND), IC7.5 (SHDNVIO), IC7.8 (STB)
- new net GNDREF: C13.2
