File: torpedokontroller/input.kicad_sch (KiCad schematic)
At the start: 25 parts, among them IC8 TCAN3414DR, J3 USB_C_Receptacle_USB2.0_14P, U10 173950336, U8 BME280, U9 TPS26400PWP

Commit message: v0.5
USB2.0 implemented fr
many other things
Parts:
- removed J3: USB_C_Receptacle_USB2.0_14P, Package_DFN_QFN:WDFN-10-1EP_3x3mm_P0.5mm_EP1.8x2.5mm, symbol Connector:USB_C_Receptacle_USB2.0_14P
- added D1: 18V, Diode_SMD:D_SMA, symbol Diode:SMAJ18A
- added D8: NSR0530HT1G, SOD2512X110N, symbol Schottky NSR0530HT1G:NSR0530HT1G
- added J2: 653104124022, Connector_SMD_Wurth:J_Wurth_WR-WTB_653104124022, symbol WR-WTB:653104124022
- added J8: USB_C_Receptacle_USB2.0_16P, Connector_SMD_Wurth:J_Wurth_WR-USB_629722000214, symbol Connector:USB_C_Receptacle_USB2.0_16P
- added R42, R43: 5k1, symbol Device:R
- added TP1: GND POGO, Optocoupler_SMD_Wurth:Q_Wurth_WL-OCPT_SOP4-STANDARD, symbol Connector:TestPoint
- added TP2: V-BAT POGO, Optocoupler_SMD_Wurth:Q_Wurth_WL-OCPT_SOP4-STANDARD, symbol Connector:TestPoint
- added U4: WE-TVS-82400102, Package_TO_SOT_SMD:SOT-23-6, symbol Power_Protection:WE-TVS-82400102
Connections:
- net Earth: now also D1.2 (A2), J2.4, J8.A1 (GND), J8.A12 (GND1), J8.B1 (GND3), J8.B12 (GND2), J8.S1 (SHIELD), J8.S2 (SHIELD), J8.S3 (SHIELD), J8.S4 (SHIELD), J8.S5 (SHIELD), J8.S6 (SHIELD), R42.2, R43.2, TP1.1, U4.2
- net USB_D+: now also U4.6
- net USB_D-: now also U4.4
- net VBAT-CON: now reaches R23.1, R7.1, U9.1 (IN), U9.2 (IN)
- net VBAT-CON: now also D1.1 (A1), TP2.1
- net CANH renamed CAN2_H
- net CAN2_H: now also J2.2
- net CANL renamed CAN2_L
- net CAN2_L: now also J2.3
- net VBUS renamed +VBUS
- net +VBUS: now also D8.1 (K)
- new net: D8.2 (A), J8.A4 (VBUS), J8.A9 (VBUS1), J8.B4 (VBUS3), J8.B9 (VBUS2), U4.5
- new net: J8.A6 (D+), J8.B6 (D+), U4.1
- new net: J8.A7 (D-), J8.B7 (D-), U4.3
- new net: J8.A5 (CC1), R43.1
- new net: J8.A9 (VBUS1), J8.B4 (VBUS3), J8.B9 (VBUS2)
- new net: J8.B5 (CC2), R42.1
- new net KILLSWITCH: J2.1
- no-connect marks 1 -> 3
Other:
- moved on the sheet: C21, C22, C23, C24, C25, C26, C27, C28, C30, C8, L3, R23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

Commit message: v 0.6
New MCU package
Added SWD, Rest and boot
Moved USB2.0 to MCU page
Other small changes
Parts:
- removed D8: NSR0530HT1G, SOD2512X110N, symbol Schottky NSR0530HT1G:NSR0530HT1G
- removed J8: USB_C_Receptacle_USB2.0_16P, Connector_SMD_Wurth:J_Wurth_WR-USB_629722000214, symbol Connector:USB_C_Receptacle_USB2.0_16P
- removed R42, R43: 5k1, symbol Device:R
- removed U4: WE-TVS-82400102, Package_TO_SOT_SMD:SOT-23-6, symbol Power_Protection:WE-TVS-82400102
Connections:
- no-connect marks 3 -> 1
Other:
- moved on the sheet: C21, C22, C23, C24, C25, C26, C27, C28, C30, C8, D1, J2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

Commit message: v 0.7
fiksa ting la til ting fjerna ting
Parts:
- added C29, C32, C33, C9: 4.7 uF, Capacitor_SMD_Wurth:C_Wurth_WCAP-CSGP-1210_H2.5, symbol Capacitor_Wurth_WCAP-CSGP:1210_H2.5_885012209048
- added C34, C35: 22 uF, Capacitor_SMD_Wurth:C_Wurth_WCAP-CSGP-1210_H2.5, symbol Capacitor_Wurth_WCAP-CSGP:1210_H2.5_885012109014
- added D3, D5: WE-VE_0603, WE-VE_0603:WE-VE_0603, symbol WE-VE_0603:WE-VE_0603
- added L4: 1.0 uH, Inductor_SMD_Wurth:L_Wurth_WE-PD2-4532, symbol Inductor_Wurth_WE-PD2:4532_7447730
- added U1: 173950536, MagIC_THT_Wurth:U_Wurth_WPME-FDSM_17395xx36, symbol WR-WPME:173950536
Connections:
- net +VBUS: now also C29.1, C9.1, L4.1
- net CAN2_H: now also D5.1
- net CAN2_L: now also D3.1
- net Earth: now also D3.2, D5.2
- net GNDREF: now also C29.2, C32.2, C33.2, C34.2, C35.2, C9.2, U1.2 (GND)
- net at D9.2 (A): now also R29.1; no longer R29.2
- net +3.3V renamed +3V3
- net +3V3: no longer C27.1, C28.1, R29.1, U10.3 (VOUT)
- new net: C27.1, C28.1, R29.2, U10.3 (VOUT)
- new net: C32.1, C33.1, L4.2, U1.1 (VIN)
- new net +5V: C34.1, C35.1, U1.3 (VOUT)
Other:
- moved on the sheet: C21, C22, C23, C24, C25, C26, C27, C28, C30, C8, J2, L3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

Commit message: v 0.8
Fixed one billion things
tvs
many values
connections
cleaned up
Parts:
- removed D4: red, symbol Device:LED
- removed D9: blue, symbol Device:LED
- added D11: 0603_150060RS55040, LED_SMD_Wurth:D_Wurth_WL-SMCD-0603, symbol WL-SMCD:0603_150060RS55040
- added D16: 0603_150060BS55040, LED_SMD_Wurth:D_Wurth_WL-SMCD-0603, symbol WL-SMCD:0603_150060BS55040
- added R57: 120, symbol Device:R
- added SW6: 472223010110, Switch_THT_Wurth:SW_Wurth_WS-TOTV_472223010110_NOLOCKING, symbol WS-TOTV:472223010110
- R23: value 470k -> 330k
- R24: value 15k -> 11k
- R25: value 30k -> 24,9k
- R29: value 1k -> 4k7
- R7: value 10k -> 1k7
Connections:
- net +3V3: now also C27.1, C28.1, R29.2, U10.3 (VOUT)
- net +VBUS: now also C25.1, C26.1, L3.2, U10.1 (VIN)
- net CAN2_H: now also R57.1
- net CAN2_L: now also SW6.2
- net FLT: now also D11.1 (-)
- net GNDREF: now also D16.1 (-)
- net at R29.1: now also D16.2 (+)
- net at R7.2: now also D11.2 (+)
- new net: R57.2, SW6.1
- no-connect marks 1 -> 2
Other:
- note added: "LED Resistor values calculated from (Vf - 3v3) / 8mA, as it gives ca 250mcd"
- note added: "TCAN"
- note added: "Telematic"
- note added: "V-Bat to +3V3"
- moved on the sheet: C21, C22, C30, D3, D5, J2, U8

Commit message: v 0.9
vet ikke
Other:
- note added: "Switch used in testing to simulate tcan being last in chain"
- note added: "Values from datasheet"
- note added: "Values from datasheet, LED resistors calculated for 10mcd"
- note removed: "LED Resistor values calculated from (Vf - 3v3) / 8mA, as it gives ca 250mcd"
- moved on the sheet: D1
Changed lines of the file:
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@@
 		)
 	)
-	(text "LED Resistor values calculated from (Vf - 3v3) / 8mA, as it gives ca 250mcd"
+	(text "Switch used in testing to simulate tcan being last in chain"
 		(exclude_from_sim no)
-		(at 59.69 76.2 0)
+		(at 50.292 156.718 0)
+		(effects
+			(font
+				(size 1.27 1.27)
+			)
+		)
+	)
+	(text "Values from datasheet, LED resistors calculated for 10mcd"
+		(exclude_from_sim no)
+		(at 50.292 75.946 0)
 		(effects
 			(font
@@
 		)
 	)
+	(text "Values from datasheet"
+		(exclude_from_sim no)
+		(at 32.004 154.432 0)
+		(effects
+			(font
+				(size 1.27 1.27)
+			)
+		)
+	)
+	(text "Values from datasheet"
+		(exclude_from_sim no)
+		(at 185.928 156.464 0)
+		(effects
+			(font
+				(size 1.27 1.27)
+			)
+		)
+	)
 	(junction
 		(at 168.91 33.02)
@@
 	)
 	(junction
-		(at 57.15 33.02)
+		(at 55.88 33.02)
 		(diameter 0)
 		(color 0 0 0 0)
@@
 	(wire
 		(pts
-			(xy 57.15 33.02) (xy 72.39 33.02)
-		)
-		(stroke
-			(width 0)
-			(type default)
-		)
-	)
-	(wire
-		(pts
 			(xy 199.39 59.69) (xy 209.55 59.69)
 		)
@@
 	(wire
 		(pts
-			(xy 57.15 33.02) (xy 57.15 34.29)
+			(xy 55.88 33.02) (xy 55.88 38.1)
 		)
 		(stroke
@@
 	(wire
 		(pts
+			(xy 40.64 33.02) (xy 72.39 33.02)
+		)
+		(stroke
+			(width 0)
+			(type default)
+		)
+	)
+	(wire
+		(pts
 			(xy 231.14 71.12) (xy 231.14 68.58)
 		)
@@
 	(wire
 		(pts
-			(xy 40.64 33.02) (xy 57.15 33.02)
-		)
-		(stroke
-			(width 0)
-			(type default)
-		)
-	)
-	(wire
-		(pts
 			(xy 153.67 44.45) (xy 153.67 41.91)
 		)
@@
 	(wire
 		(pts
-			(xy 57.15 41.91) (xy 57.15 49.53)
+			(xy 55.88 45.72) (xy 55.88 49.53)
 		)
 		(stroke
@@
 	(symbol
 		(lib_id "power:Earth")
-		(at 57.15 49.53 0)
+		(at 55.88 49.53 0)
 		(unit 1)
 		(body_style 1)
@@
 		(fields_autoplaced yes)
 		(property "Reference" "#PWR016"
-			(at 57.15 55.88 0)
+			(at 55.88 55.88 0)
 			(hide yes)
 			(show_name no)
@@
 		)
 		(property "Value" "Earth"
-			(at 57.15 54.61 0)
+			(at 55.88 54.61 0)
 			(hide yes)
 			(show_name no)
@@
 		)
 		(property "Footprint" ""
-			(at 57.15 49.53 0)
+			(at 55.88 49.53 0)
 			(hide yes)
 			(show_name no)
@@
 		)
 		(property "Datasheet" ""
-			(at 57.15 49.53 0)
+			(at 55.88 49.53 0)
 			(hide yes)
 			(show_name no)
@@
 		)
 		(property "Description" "Power symbol creates a global label with name \"Earth\""
-			(at 57.15 49.53 0)
+			(at 55.88 49.53 0)
 			(hide yes)
 			(show_name no)
@@
 	(symbol
 		(lib_id "Diode:SMAJ18A")
-		(at 57.15 38.1 270)
+		(at 55.88 41.91 270)
 		(unit 1)
 		(body_style 1)
@@
 		(fields_autoplaced yes)
 		(property "Reference" "D1"
-			(at 59.69 36.8299 90)
+			(at 58.42 40.6399 90)
 			(show_name no)
 			(do_not_autoplace no)
@@
 		)
 		(property "Value" "18V"
-			(at 59.69 39.3699 90)
+			(at 58.42 43.1799 90)
 			(show_name no)
 			(do_not_autoplace no)
@@
 		)
 		(property "Footprint" "Diode_SMD:D_SMA"
-			(at 52.07 38.1 0)
+			(at 50.8 41.91 0)
 			(hide yes)
 			(show_name no)
@@
 		)
 		(property "Datasheet" "https://www.littelfuse.com/media?resourcetype=datasheets&itemid=75e32973-b177-4ee3-a0ff-cedaf1abdb93&filename=smaj-datasheet"
-			(at 57.15 36.83 0)
+			(at 55.88 40.64 0)
 			(hide yes)
 			(show_name no)
@@
 		)
 		(property "Description" "400W unidirectional Transient Voltage Suppressor, 18.0Vr, SMA(DO-214AC)"
-			(at 57.15 38.1 0)
+			(at 55.88 41.91 0)
 			(hide yes)
 			(show_name no)

Commit message: v 1.0
Ferdigish

CAN tvs-packages
Ground hook
Test pads
fixed some i/o issues
Parts:
- removed D3, D5: WE-VE_0603, WE-VE_0603:WE-VE_0603, symbol WE-VE_0603:WE-VE_0603
- added D18: SOT23-3L_824094024, Diode_SMD_Wurth:D_Wurth_WE-TVS-SOT23-3L, symbol Diode_Wurth_WE-TVSP:SOT23-3L_824094024
- added J4: Ground_hook, Connector_THT_Wurth:J_Wurth_WR-PHD_61300111121, symbol Connector_Wurth_WR-PHD:61300111121
- added TP3, TP4, TP7, TP8: TestPoint, TestPoint:TestPoint_Pad_D1.5mm, symbol Connector:TestPoint
Connections:
- net CAN2_H: now also D18.1 (I/O1)
- net CAN2_L: now also D18.2 (I/O2)
- net CSB: now also TP8.1
- net Earth: now also D18.3 (GND)
- net GNDREF: now also J4.1
- net SCK: now also TP4.1
- net SPI1_MISO: now also TP3.1
- net SPI1_MOIS: now also TP7.1
- net FLT renamed ~{FLT}
Other:
- note added: "Ground hook"
- moved on the sheet: C21, C22, C23, C24, C25, C26, C27, C28, C29, C30, C32, C33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

Commit message: some footprints + print
Parts:
- C21, C22, C23: footprint (none) -> Capasitors:C_Wurth_WCAP-CSGP-0603_R
- C24, C25, C26, C27, C28, C29, C30, C32, C33, C34, C35, C8, C9: footprint Capacitor_SMD_Wurth:C_Wurth_WCAP-CSGP-1210_H2.5 -> Capasitors:C_Wurth_WCAP-CSGP-0603_R
- D11, D16: footprint LED_SMD_Wurth:D_Wurth_WL-SMCD-0603 -> WL-LED:D_Wurth_WL-SMCD-0603
- D18: footprint Diode_SMD_Wurth:D_Wurth_WE-TVS-SOT23-3L -> Package_TO_SOT_SMD:SOT-23-3
- R23, R24, R27, R28, R29, R57, R7: footprint (none) -> WE-Resistors:R_Wurth_WRIS-KSKE-0603
- R25: value 24,9k -> 24k9; footprint (none) -> WE-Resistors:R_Wurth_WRIS-KSKE-0603
Changed lines of the file:
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@@
 			)
 		)
-		(property "Footprint" "Capacitor_SMD_Wurth:C_Wurth_WCAP-CSGP-1210_H2.5"
+		(property "Footprint" "Capasitors:C_Wurth_WCAP-CSGP-0603_R"
 			(at 156.21 44.45 0)
 			(hide yes)
@@
 			)
 		)
-		(property "Footprint" ""
+		(property "Footprint" "WE-Resistors:R_Wurth_WRIS-KSKE-0603"
 			(at 123.952 63.5 90)
 			(hide yes)
@@
 			)
 		)
-		(property "Value" "24,9k"
+		(property "Value" "24k9"
 			(at 85.09 53.3399 0)
 			(show_name no)
@@
 			)
 		)
-		(property "Footprint" ""
+		(property "Footprint" "WE-Resistors:R_Wurth_WRIS-KSKE-0603"
 			(at 80.772 52.07 90)
 			(hide yes)
@@
 			)
 		)
-		(property "Footprint" "Capacitor_SMD_Wurth:C_Wurth_WCAP-CSGP-1210_H2.5"
+		(property "Footprint" "Capasitors:C_Wurth_WCAP-CSGP-0603_R"
 			(at 201.93 17.78 0)
 			(hide yes)
@@
 			)
 		)
-		(property "Footprint" ""
+		(property "Footprint" "WE-Resistors:R_Wurth_WRIS-KSKE-0603"
 			(at 265.43 31.242 90)
 			(hide yes)
@@
 			)
 		)
-		(property "Footprint" "Capacitor_SMD_Wurth:C_Wurth_WCAP-CSGP-1210_H2.5"
+		(property "Footprint" "Capasitors:C_Wurth_WCAP-CSGP-0603_R"
 			(at 171.45 44.45 0)
 			(hide yes)
@@
 			)
 		)
-		(property "Footprint" "Capacitor_SMD_Wurth:C_Wurth_WCAP-CSGP-1210_H2.5"
+		(property "Footprint" "Capasitors:C_Wurth_WCAP-CSGP-0603_R"
 			(at 247.65 44.45 0)
 			(hide yes)
@@
 			)
 		)
-		(property "Footprint" ""
+		(property "Footprint" "WE-Resistors:R_Wurth_WRIS-KSKE-0603"
 			(at 68.072 38.1 90)
 			(hide yes)
@@
 			)
 		)
-		(property "Footprint" ""
+		(property "Footprint" "WE-Resistors:R_Wurth_WRIS-KSKE-0603"
 			(at 64.262 115.57 90)
 			(hide yes)
@@
 			)
 		)
-		(property "Footprint" ""
+		(property "Footprint" "Capasitors:C_Wurth_WCAP-CSGP-0603_R"
 			(at 168.6052 114.3 0)
 			(hide yes)
@@
 			)
 		)
-		(property "Footprint" "Capacitor_SMD_Wurth:C_Wurth_WCAP-CSGP-1210_H2.5"
+		(property "Footprint" "Capasitors:C_Wurth_WCAP-CSGP-0603_R"
 			(at 233.68 17.78 0)
 			(hide yes)
@@
 			)
 		)
-		(property "Footprint" "Capacitor_SMD_Wurth:C_Wurth_WCAP-CSGP-1210_H2.5"
+		(property "Footprint" "Capasitors:C_Wurth_WCAP-CSGP-0603_R"
 			(at 156.21 17.78 0)
 			(hide yes)
@@
 			)
 		)
-		(property "Footprint" "Capacitor_SMD_Wurth:C_Wurth_WCAP-CSGP-1210_H2.5"
+		(property "Footprint" "Capasitors:C_Wurth_WCAP-CSGP-0603_R"
 			(at 201.93 44.45 0)
 			(hide yes)
@@
 			)
 		)
-		(property "Footprint" "Capacitor_SMD_Wurth:C_Wurth_WCAP-CSGP-1210_H2.5"
+		(property "Footprint" "Capasitors:C_Wurth_WCAP-CSGP-0603_R"
 			(at 171.45 17.78 0)
 			(hide yes)
@@
 			)
 		)
-		(property "Footprint" "LED_SMD_Wurth:D_Wurth_WL-SMCD-0603"
+		(property "Footprint" "WL-LED:D_Wurth_WL-SMCD-0603"
 			(at 248.92 26.67 0)
 			(hide yes)
@@
 			)
 		)
-		(property "Footprint" "Capacitor_SMD_Wurth:C_Wurth_WCAP-CSGP-1210_H2.5"
+		(property "Footprint" "Capasitors:C_Wurth_WCAP-CSGP-0603_R"
 			(at 186.69 44.45 0)
 			(hide yes)
@@
 			)
 		)
-		(property "Footprint" ""
+		(property "Footprint" "Capasitors:C_Wurth_WCAP-CSGP-0603_R"
 			(at 180.0352 114.3 0)
 			(hide yes)
@@
 			)
 		)
-		(property "Footprint" ""
+		(property "Footprint" "WE-Resistors:R_Wurth_WRIS-KSKE-0603"
 			(at 80.772 44.45 90)
 			(hide yes)
@@
 			)
 		)
-		(property "Footprint" ""
+		(property "Footprint" "WE-Resistors:R_Wurth_WRIS-KSKE-0603"
 			(at 131.572 63.5 90)
 			(hide yes)
@@
 			)
 		)
-		(property "Footprint" ""
+		(property "Footprint" "Capasitors:C_Wurth_WCAP-CSGP-0603_R"
 			(at 117.8052 67.31 0)
 			(hide yes)
@@
 			)
 		)
-		(property "Footprint" "LED_SMD_Wurth:D_Wurth_WL-SMCD-0603"
+		(property "Footprint" "WL-LED:D_Wurth_WL-SMCD-0603"
 			(at 49.53 34.29 0)
 			(hide yes)
@@
 			)
 		)
-		(property "Footprint" "Capacitor_SMD_Wurth:C_Wurth_WCAP-CSGP-1210_H2.5"
+		(property "Footprint" "Capasitors:C_Wurth_WCAP-CSGP-0603_R"
 			(at 233.68 44.45 0)
 			(hide yes)
@@
 			)
 		)
-		(property "Footprint" "Capacitor_SMD_Wurth:C_Wurth_WCAP-CSGP-1210_H2.5"
+		(property "Footprint" "Capasitors:C_Wurth_WCAP-CSGP-0603_R"
 			(at 115.57 87.63 0)
 			(hide yes)
@@
 			)
 		)
-		(property "Footprint" "Capacitor_SMD_Wurth:C_Wurth_WCAP-CSGP-1210_H2.5"
+		(property "Footprint" "Capasitors:C_Wurth_WCAP-CSGP-0603_R"
 			(at 186.69 17.78 0)
 			(hide yes)
@@
 			)
 		)
-		(property "Footprint" ""
+		(property "Footprint" "WE-Resistors:R_Wurth_WRIS-KSKE-0603"
 			(at 80.772 36.83 90)
 			(hide yes)
@@
 			)
 		)
-		(property "Footprint" "Diode_SMD_Wurth:D_Wurth_WE-TVS-SOT23-3L"
+		(property "Footprint" "Package_TO_SOT_SMD:SOT-23-3"
 			(at 67.31 147.32 0)
 			(hide yes)
@@
 			)
 		)
-		(property "Footprint" "Capacitor_SMD_Wurth:C_Wurth_WCAP-CSGP-1210_H2.5"
+		(property "Footprint" "Capasitors:C_Wurth_WCAP-CSGP-0603_R"
 			(at 247.65 17.78 0)
 			(hide yes)

Commit message: v 1.1
Fiksa ting
starta layout
bedre schematic design
whooppppppwhhoop
Parts:
- removed D18: SOT23-3L_824094024, Package_TO_SOT_SMD:SOT-23-3, symbol Diode_Wurth_WE-TVSP:SOT23-3L_824094024
- removed J2: 653104124022, Connector_SMD_Wurth:J_Wurth_WR-WTB_653104124022, symbol WR-WTB:653104124022
- removed SW6: 472223010110, Switch_THT_Wurth:SW_Wurth_WS-TOTV_472223010110_NOLOCKING, symbol WS-TOTV:472223010110
- removed TP1: GND POGO, Optocoupler_SMD_Wurth:Q_Wurth_WL-OCPT_SOP4-STANDARD, symbol Connector:TestPoint
- removed TP2: V-BAT POGO, Optocoupler_SMD_Wurth:Q_Wurth_WL-OCPT_SOP4-STANDARD, symbol Connector:TestPoint
- added D20: SOT23-3L_824094024, Package_TO_SOT_SMD:SOT-23-3, symbol Diode_Wurth_WE-TVSP:SOT23-3L_824094024
- added D3: 18V, Diode_SMD:D_SMA, symbol Diode:SMAJ18A
- added J11: 61302021121, Connectors_tht:J_Wurth_WR-PHD_61302021121, symbol Connector_Wurth_WR-PHD:61302021121
- added R2: 0, WE-Resistors:R_Wurth_WRIS-KSKE-0603, symbol Device:R
- added SW3: 418127270901, Switch_THT:SW_Wurth_WS-DITV_418127270901, symbol Switch_Wurth_WS-DITV:418127270901
- added U0, U1, U10, U11, U2, U3, U4, U5, U6, U7, U8, U9: 7982-1-15-20-75-14-11-0, Samacsys:7982115207514110, symbol 7982-1-15-20-75-14-11-0:7982-1-15-20-75-14-11-0
- J4: footprint Connector_THT_Wurth:J_Wurth_WR-PHD_61300111121 -> Connectors_tht:J_Wurth_WR-PHD_61300111121
- L3, L4: footprint Inductor_SMD_Wurth:L_Wurth_WE-PD2-4532 -> Inductor:L_Wurth_WE-PD2-4532
- U12: renamed from U10; footprint MagIC_THT_Wurth:U_Wurth_WPME-FDSM_17395xx36 -> Buck_down:173950536
- U13: renamed from U1; footprint MagIC_THT_Wurth:U_Wurth_WPME-FDSM_17395xx36 -> Buck_down:173950536
- renumbered U8 to U14, U9 to U16
Connections:
- net +VBUS: now also R2.1; no longer C24.1, C29.1, C8.1, C9.1, L3.1, L4.1
- net CAN2_H: now also D20.2 (I/O2), J11.19, U10.1
- net CAN2_L: now also D20.1 (I/O1), J11.20, SW3.1, U11.1
- net Earth: now also D20.3 (GND), D3.2 (A2), J11.10, J11.11, J11.12, J11.13, J11.14, J11.15, J11.16, J11.17, J11.9, U4.1, U5.1, U6.1, U7.1, U8.1
- net KILLSWITCH: now also J11.18, U9.1
- net VBAT-CON: now also D3.1 (A1), J11.1, J11.2, J11.3, J11.4, J11.5, J11.6, J11.7, J11.8, U0.1, U1.1, U2.1, U3.1
- net at R57.2: now also SW3.A1
- new net: C24.1, C29.1, C8.1, C9.1, L3.1, L4.1, R2.2
- no-connect marks 2 -> 1
Other:
- note added: "BMS Connector"
- note added: "POGO-PADS"
- note added: "VBAT to +3V3"
- note removed: "V-Bat to +3V3"
- moved on the sheet: C21, C22, C23, C24, C25, C26, C27, C28, C29, C30, C32, C33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
