File: torpedokontroller/input.kicad_sch (KiCad schematic)
At the start: 56 parts, among them IC8 TCAN3414DR, J11 61302021121, J4 Ground_hook, SW3 418127270901, U0 7982-1-15-20-75-14-11-0, U1 7982-1-15-20-75-14-11-0, U10 7982-1-15-20-75-14-11-0, U11 7982-1-15-20-75-14-11-0, U12 173950336, U13 173950536, U14 BME280, U16 TPS26400PWP, U2 7982-1-15-20-75-14-11-0, U3 7982-1-15-20-75-14-11-0, U4 7982-1-15-20-75-14-11-0, U5 7982-1-15-20-75-14-11-0, U6 7982-1-15-20-75-14-11-0, U7 7982-1-15-20-75-14-11-0, U8 7982-1-15-20-75-14-11-0, U9 7982-1-15-20-75-14-11-0

Commit message: post-schematic_review 💯
fixed stuff
added stuff
GND is good
I2C BME280
memes
fixed pins
more stuff
💯
Parts:
- removed D20: SOT23-3L_824094024, Package_TO_SOT_SMD:SOT-23-3, symbol Diode_Wurth_WE-TVSP:SOT23-3L_824094024
- removed D3: 18V, Diode_SMD:D_SMA, symbol Diode:SMAJ18A
- removed J11: 61302021121, Connectors_tht:J_Wurth_WR-PHD_61302021121, symbol Connector_Wurth_WR-PHD:61302021121
- removed TP3, TP8: TestPoint, TestPoint:TestPoint_Pad_D1.5mm, symbol Connector:TestPoint
- added D21: SOT23-3L_824094024, Package_TO_SOT_SMD:SOT-23-3, symbol Diode_Wurth_WE-TVSP:SOT23-3L_824094024
- added R30, R31: 4k7, WE-Resistors:R_Wurth_WRIS-KSKE-0603, symbol Device:R
- added TP15: TestPoint, TestPoint:TestPoint_Pad_D1.5mm, symbol Connector:TestPoint
Connections:
- net CSB is gone; now on net +3V3: U14.2 (CSB)
- net GNDREF is gone; now on net Earth: C21.2, C22.2, C24.2, C25.2, C26.2, C27.2, C28.2, C29.2, C30.2, C32.2, C33.2, C34.2, C35.2, C8.2, C9.2, D16.1 (-), J4.1, U12.2 (GND), U13.2 (GND), U14.1 (GND), U14.7 (GND), U16.9 (GND)
- net SPI1_MISO is gone; now on net Earth: U14.5 (SDO)
- net +3V3: now also R30.1, R31.1
- net CAN2_H: now also D21.2 (I/O2)
- net CAN2_L: now also D21.1 (I/O1)
- net Earth: now also D21.3 (GND)
- net SCK: now also R30.2
- net IMON_SMALL: now reaches R28.1, U16.10 (IMON)
- net IMON_SMALL: now also TP15.1
- net SPI1_MOIS renamed SDI
- net SDI: now also R31.2
Other:
- note added: "Telematic BME280"
- note added: "VBAT to +3V3 / +5V"
- note removed: "BMS Connector"
- note removed: "Telematic"
- note removed: "VBAT to +3V3"
- moved on the sheet: C21, C22, C23, C24, C25, C26, C27, C28, C29, C30, C32, C33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

Commit message: v 1.2
PWM SERVOS :)) YAAADDAAAAAa
Layout begynner å komme seg
Connections:
- net +VBUS: no longer C25.1, C26.1, L3.2, U12.1 (VIN)
- net +VBUS_OUT: now reaches C24.1, C29.1, C8.1, C9.1, L3.1, L4.1, R2.2
- net +VBUS_OUT_INDUCTOR: now reaches C32.1, C33.1, L4.2, U13.1 (VIN)
- net +VBUS_OUT_INDUCTOR: now also C25.1, C26.1, L3.2, U12.1 (VIN)
Changed lines of the file:
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@@
 	(paper "A4")
 	(title_block
-		(date "2026-10-23")
+		(date "2026-10-26")
 		(comment 1 "Simon Torvund")
 	)
@@
 	)
 	(junction
-		(at 121.92 90.17)
-		(diameter 0)
-		(color 0 0 0 0)
-	)
-	(junction
 		(at 175.26 90.17)
 		(diameter 0)
@@
 	)
 	(junction
+		(at 120.65 90.17)
+		(diameter 0)
+		(color 0 0 0 0)
+	)
+	(junction
 		(at 67.31 149.86)
 		(diameter 0)
@@
 	(wire
 		(pts
+			(xy 120.65 88.9) (xy 120.65 90.17)
+		)
+		(stroke
+			(width 0)
+			(type default)
+		)
+	)
+	(wire
+		(pts
 			(xy 110.49 39.37) (xy 110.49 41.91)
 		)
@@
 	(wire
 		(pts
-			(xy 107.95 90.17) (xy 121.92 90.17)
+			(xy 107.95 90.17) (xy 120.65 90.17)
 		)
 		(stroke
@@
 	(wire
 		(pts
-			(xy 121.92 86.36) (xy 121.92 90.17)
-		)
-		(stroke
-			(width 0)
-			(type default)
-		)
-	)
-	(wire
-		(pts
 			(xy 222.25 90.17) (xy 236.22 90.17)
 		)
@@
 	(wire
 		(pts
-			(xy 175.26 90.17) (xy 190.5 90.17)
-		)
-		(stroke
-			(width 0)
-			(type default)
-		)
-	)
-	(wire
-		(pts
 			(xy 80.01 181.61) (xy 95.25 181.61)
 		)
@@
 	(wire
 		(pts
-			(xy 121.92 90.17) (xy 124.46 90.17)
+			(xy 160.02 116.84) (xy 163.83 116.84)
 		)
 		(stroke
@@
 	(wire
 		(pts
-			(xy 160.02 116.84) (xy 163.83 116.84)
+			(xy 95.25 163.83) (xy 95.25 165.1)
 		)
 		(stroke
@@
 	(wire
 		(pts
-			(xy 95.25 163.83) (xy 95.25 165.1)
+			(xy 175.26 90.17) (xy 190.5 90.17)
 		)
 		(stroke
@@
 	(wire
 		(pts
+			(xy 120.65 90.17) (xy 124.46 90.17)
+		)
+		(stroke
+			(width 0)
+			(type default)
+		)
+	)
+	(wire
+		(pts
 			(xy 43.18 39.37) (xy 48.26 39.37)
 		)
@@
 		)
 	)
-	(label "+VBUS"
-		(at 177.8 90.17 0)
+	(label "+VBUS_OUT"
+		(at 134.62 90.17 0)
 		(effects
 			(font
@@
 		)
 	)
-	(label "CAN2_H"
-		(at 161.29 33.02 0)
+	(label "+VBUS_OUT_INDUCTOR"
+		(at 175.26 116.84 0)
 		(effects
 			(font
@@
 		)
 	)
-	(label "RTN"
-		(at 85.09 125.73 0)
+	(label "+VBUS_OUT_INDUCTOR"
+		(at 175.26 90.17 0)
 		(effects
 			(font
@@
 		)
 	)
-	(global_label "+VBUS"
-		(shape input)
-		(at 121.92 86.36 90)
-		(fields_autoplaced yes)
+	(label "CAN2_H"
+		(at 161.29 33.02 0)
 		(effects
 			(font
 				(size 1.27 1.27)
 			)
-			(justify left)
+			(justify left bottom)
 		)
-		(property "Intersheetrefs" "${INTERSHEET_REFS}"
-			(at 121.92 76.9038 90)
-			(hide yes)
-			(show_name no)
-			(do_not_autoplace no)
-			(effects
-				(font
-					(size 1.27 1.27)
-				)
-				(justify left)
+	)
+	(label "RTN"
+		(at 85.09 125.73 0)
+		(effects
+			(font
+				(size 1.27 1.27)
 			)
+			(justify left bottom)
 		)
 	)
@@
 		(lib_id "Device:C")
 		(at 110.49 120.65 0)
+		(mirror y)
 		(unit 1)
 		(body_style 1)
@@
 		(dnp no)
 		(property "Reference" "C23"
-			(at 104.14 120.65 0)
+			(at 107.696 119.888 0)
 			(show_name no)
 			(do_not_autoplace no)
@@
 		)
 		(property "Value" "1u"
-			(at 104.648 122.428 0)
+			(at 107.188 121.666 0)
 			(show_name no)
 			(do_not_autoplace no)
@@
 		)
 		(property "Footprint" "Capasitors:C_Wurth_WCAP-CSGP-0603_R"
-			(at 111.4552 124.46 0)
+			(at 109.5248 124.46 0)
 			(hide yes)
 			(show_name no)
@@
 					(unit 1)
 				)
+			)
+		)
+	)
+	(symbol
+		(lib_id "power:VCC")
+		(at 120.65 88.9 0)
+		(unit 1)
+		(body_style 1)
+		(exclude_from_sim no)
+		(in_bom yes)
+		(on_board yes)
+		(in_pos_files yes)
+		(dnp no)
+		(property "Reference" "#PWR081"
+			(at 120.65 92.71 0)
+			(hide yes)
+			(show_name no)
+			(do_not_autoplace no)
+			(effects
+				(font
+					(size 1.27 1.27)
+				)
+			)
+		)
+		(property "Value" "+VBUS"
+			(at 120.396 85.344 0)
+			(show_name no)
+			(do_not_autoplace no)
+			(effects
+				(font
+					(size 1.27 1.27)
+				)
+			)
+		)
+		(property "Footprint" ""
+			(at 120.65 88.9 0)
+			(hide yes)
+			(show_name no)
+			(do_not_autoplace no)
+			(effects
+				(font
+					(size 1.27 1.27)
+				)
+			)
+		)
+		(property "Datasheet" ""
+			(at 120.65 88.9 0)
+			(hide yes)
+			(show_name no)
+			(do_not_autoplace no)
+			(effects
+				(font
+					(size 1.27 1.27)
+				)
+			)
+		)
+		(property "Description" "Power symbol creates a global label with name \"VCC\""
+			(at 120.65 88.9 0)
+			(hide yes)
+			(show_name no)
+			(do_not_autoplace no)
+			(effects
+				(font
+					(size 1.27 1.27)
+				)
+			)
+		)
+		(pin "1"
+		)
+		(instances
+			(project "torpedokontroller"
+				(path "/e42df04f-3e58-4415-86e6-9a5d9df63a21/e120803b-a57e-427e-b241-e167c0d83487"
+					(reference "#PWR081")
+					(unit 1)
+				)
