File: torpedokontroller/processing.kicad_sch (KiCad schematic)
At the start: 16 parts, among them IC3 STM32C542RCT6, J1 61300211021, J4 62701021621

Commit message: v 0.6
New MCU package
Added SWD, Rest and boot
Moved USB2.0 to MCU page
Other small changes
Parts:
- removed C10: 2.2 uF, Capacitor_SMD_Wurth:C_Wurth_WCAP-CSGP-1210_H2.5, symbol Capacitor_Wurth_WCAP-CSGP:1210_H2.5_885012209048
- removed C32, C33, C34, C35, C36: 100n, symbol Device:C
- removed C9: 4.7 uF, Capacitor_SMD_Wurth:C_Wurth_WCAP-CSGP-1210_H2.5, symbol Capacitor_Wurth_WCAP-CSGP:1210_H2.5_885012209048
- removed D10: green, symbol Device:LED
- removed D11: yellow, symbol Device:LED
- removed D12: red, symbol Device:LED
- removed IC3: STM32C542RCT6, Samacsys:QFP50P1200X1200X160-64N, symbol Samacsys:STM32C542RCT6
- removed J1: 61300211021, Connector_THT_Wurth:J_Wurth_WR-PHD_61300211021, symbol Connector_Wurth_WR-PHD:61300211021
- removed J4: 62701021621, Connector_THT_Wurth:J_Wurth_WR-BHD_62701021621, symbol SWD-Header:62701021621
- removed R30, R31, R32: 1k, symbol Device:R
- added C11: 4.7 uF, Capacitor_SMD_Wurth:C_Wurth_WCAP-CSGP-1210_H2.5, symbol Capacitor_Wurth_WCAP-CSGP:1210_H2.5_885012209048
- added C12: 2.2 uF, Capacitor_SMD_Wurth:C_Wurth_WCAP-CSGP-1210_H2.5, symbol Capacitor_Wurth_WCAP-CSGP:1210_H2.5_885012209048
- added C13: 0.1 uF, Capacitor_SMD_Wurth:C_Wurth_WCAP-CSGP-1210_H2.5, symbol Capacitor_Wurth_WCAP-CSGP:1210_H2.5_885012209048
- added C39, C43, C44, C45: 100n, symbol Device:C
- added D10: NSR0530HT1G, SOD2512X110N, symbol Schottky NSR0530HT1G:NSR0530HT1G
- added D13: green, symbol Device:LED
- added D14: yellow, symbol Device:LED
- added D15: red, symbol Device:LED
- added IC2: STM32C542CCT6, QFP50P900X900X160-48N, symbol STM32C542CCT6:STM32C542CCT6
- added J4: 61300211021, Connector_THT_Wurth:J_Wurth_WR-PHD_61300211021, symbol Connector_Wurth_WR-PHD:61300211021
- added J5: 62701021621, Connector_THT_Wurth:J_Wurth_WR-BHD_62701021621, symbol SWD-Header:62701021621
- added J9: USB_C_Receptacle_USB2.0_16P, Connector_SMD_Wurth:J_Wurth_WR-USB_629722000214, symbol Connector:USB_C_Receptacle_USB2.0_16P
- added R35, R36, R37: 1k, symbol Device:R
- added R38, R39: 10k, symbol Device:R
- added R53, R54: 5k1, symbol Device:R
- added SW1, SW2: 434123025826, Switch_SMD_Wurth:SW_Wurth_WS-TASV_434123025826, symbol WS-TASV:434123025826
- added U5: WE-TVS-82400102, Package_TO_SOT_SMD:SOT-23-6, symbol Power_Protection:WE-TVS-82400102
Connections:
- net +3.3V: now also C11.1, C39.2, C43.1, C44.1, C45.1, IC2.24 (VDD_1), IC2.36 (VDD_2), IC2.48 (VDD_3), IC2.9 (VREF+), J5.1, R38.2
- net CAN1_RX: now also IC2.45 (PB8)
- net CAN1_TX: now also IC2.41 (PB5)
- net CAN2_RX: now also IC2.42 (PB6)
- net CAN2_TX: now also IC2.43 (PB7)
- net CSB: now also IC2.16 (PA6)
- net Earth: now also C11.2, C12.2, C13.2, C39.1, C43.2, C44.2, C45.2, D13.1 (K), D14.1 (K), D15.1 (K), IC2.23 (VSS_1), IC2.35 (VSS_2), IC2.47 (VSS_3), IC2.8 (VREF-), J5.3, J5.5, J5.9, J9.A1 (GND), J9.A12 (GND1), J9.B1 (GND3), J9.B12 (GND2), J9.S1 (SHIELD), J9.S2 (SHIELD), J9.S3 (SHIELD), J9.S4 (SHIELD), J9.S5 (SHIELD), J9.S6 (SHIELD), R39.2, R53.2, R54.2, SW1.3, SW1.4, U5.2
- net GOK: now also IC2.20 (PB2)
- net IMON: now also IC2.19 (PB1)
- net SCK: now also IC2.15 (PA5)
- net SPI1_MISO: now also IC2.18 (PB0)
- net SPI1_MOSI: now also IC2.17 (PA7)
- net UART_RX: now also IC2.31 (PA10), J4.2
- net UART_TX: now also IC2.46 (PB9), J4.1
- net USB_D+: now also IC2.33 (PA12), U5.6
- net USB_D-: now also IC2.32 (PA11), U5.4
- new net: D10.2 (A), J9.A4 (VBUS), J9.A9 (VBUS1), J9.B4 (VBUS3), J9.B9 (VBUS2), U5.5
- new net: C12.1, IC2.22 (VCAP)
- new net: R39.1, SW2.3, SW2.4
- new net: IC2.10 (PA0), R35.2
- new net: IC2.11 (PA1), R36.2
- new net: IC2.12 (PA2), R37.2
- new net: D15.2 (A), R37.1
- new net: J9.A5 (CC1), R54.1
- new net: D13.2 (A), R35.1
- new net: D14.2 (A), R36.1
- new net: J9.A6 (D+), J9.B6 (D+), U5.1
- new net: J9.A7 (D-), J9.B7 (D-), U5.3
- new net: J9.A9 (VBUS1), J9.B4 (VBUS3), J9.B9 (VBUS2)
- new net: J9.B5 (CC2), R53.1
- new net +VBUS: D10.1 (K)
- new net BOOT0: IC2.44 (PH2-BOOT0), R38.1, SW2.1, SW2.2
- new net D_OC: IC2.21 (PB10)
- new net NRST: C13.1, IC2.7 (NRST), J5.10, SW1.1, SW1.2
- new net SWCLK: IC2.34 (PA13), J5.4
- new net SWDIO: IC2.37 (PA14), J5.2
- new net SWO: IC2.39 (PB3), J5.6
- no-connect marks 0 -> 4

Commit message: v 0.7
fiksa ting la til ting fjerna ting
Parts:
- added C14: 0.1 uF, Capacitor_SMD_Wurth:C_Wurth_WCAP-CSGP-1210_H2.5, symbol Capacitor_Wurth_WCAP-CSGP:1210_H2.5_885012209048
- added C15: 100nF, Capacitor_SMD_Wurth:C_Wurth_WCAP-CSGP-1210_H2.5, symbol Capacitor_Wurth_WCAP-CSGP:1210_H2.5_885012209048
- added C16: 1u, Capacitor_SMD_Wurth:C_Wurth_WCAP-CSGP-1210_H2.5, symbol Capacitor_Wurth_WCAP-CSGP:1210_H2.5_885012209048
- added IC3: SN74AHCT1G125DCKR, SOT65P210X110-5N, symbol AHCT:SN74AHCT1G125DCKR
- added J3: 653104124022, Connector_SMD_Wurth:J_Wurth_WR-WTB_653104124022, symbol WR-WTB:653104124022
- added Y1: 48 MHz, Crystal_SMD_Wurth:Y_Wurth_WE-SPXO-CFPS-39, symbol WE-SPXO:CFPS-39_830207659609
Connections:
- net Earth: now also C14.2, C15.2, C16.2, IC3.1 (~{OE}), IC3.3 (GND), J3.3, Y1.2 (GND)
- net LED_MOSI: now reaches IC2.14 (PA4)
- net LED_MOSI: now also IC3.2 (A)
- net OSC48M: now reaches IC2.5 (PH0-OSC_IN)
- net OSC48M: now also Y1.3 (OUT)
- net +3.3V renamed +3V3
- net +3V3: now also C14.1, Y1.4 (+VS)
- new net: IC3.4 (Y), J3.2
- new net +5V: C15.1, C16.1, IC3.5 (VCC), J3.1
- no-connect marks 4 -> 20
Other:
- moved on the sheet: C11, C12, C13, C39, C43, C44, C45, D10, IC2, J4, J5, J9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

Commit message: v 0.8
Fixed one billion things
tvs
many values
connections
cleaned up
Parts:
- removed D13: green, symbol Device:LED
- removed D14: yellow, symbol Device:LED
- removed D15: red, symbol Device:LED
- added D13: 0603_150060YS55040, LED_SMD_Wurth:D_Wurth_WL-SMCD-0603, symbol WL-SMCD:0603_150060YS55040
- added D4: SOT23-6L_824015043, Diode_SMD_Wurth:D_Wurth_WE-TVS-SOT23-6L, symbol TVS:SOT23-6L_824015043
- added D6: SOT143-4L_8240136, Diode_SMD_Wurth:D_Wurth_WE-TVS-SOT143-4L, symbol Diode_Wurth_WE-TVSP:SOT143-4L_8240136
- added D7: 0603_150060GS55040, LED_SMD_Wurth:D_Wurth_WL-SMCD-0603, symbol WL-SMCD:0603_150060GS55040
- added D9: 0603_150060RS55040, LED_SMD_Wurth:D_Wurth_WL-SMCD-0603, symbol WL-SMCD:0603_150060RS55040
- R: renamed from R36; value 1k -> 680
- R35: value 1k -> 4k
- R37: value 1k -> 750
Connections:
- net +3V3: now also D4.5 (VDD), D6.4 (VDD)
- net Earth: now also D13.1 (-), D4.2 (GND), D6.1 (GND), D7.1 (-), D9.1 (-)
- net NRST: now also D4.3
- net SWCLK: now also D4.6
- net SWDIO: now also D4.4
- net SWO: now also D4.1
- net UART_RX: now also D6.2 (1)
- net UART_TX: now also D6.3 (2)
- net Y: now reaches IC3.4 (Y), J3.2
- net MCU_KillSwitch: now reaches IC2.28 (PB15)
- net at R37.1: now also D9.2 (+)
- net at R35.1: now also D7.2 (+)
- net at R.1: now also D13.2 (+)
- no-connect marks 20 -> 19
Other:
- note added: "Capacitor values from datasheet"
- note added: "LED Resistor values calculated from (Vf - 3v3) / 8mA, as it gives ca 250mcd"
- note added: "Microprocessor"
- note added: "Oscillator"
- note added: "RESET / BOOT"
- note added: "RGB_LED"
- note added: "SWD"
- note added: "UART"
- note added: "USB2.0"
- moved on the sheet: C11, C12, C13, C15, C16, C39, C43, C44, C45, IC2, IC3, J3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

Commit message: v 0.9
vet ikke
Other:
- note added: "LED Resistor values calculated to give ca 10mcd"
- note removed: "LED Resistor values calculated from (Vf - 3v3) / 8mA, as it gives ca 250mcd"
- moved on the sheet: C13, C15, C16, D6, IC3, J3, SW1

Commit message: v 1.0
Ferdigish

CAN tvs-packages
Ground hook
Test pads
fixed some i/o issues
Parts:
- removed J4: 61300211021, Connector_THT_Wurth:J_Wurth_WR-PHD_61300211021, symbol Connector_Wurth_WR-PHD:61300211021
- added J6: 61300311021, Connector_THT_Wurth:J_Wurth_WR-PHD_61300311021, symbol Connector_Wurth_WR-PHD:61300311021
- added TP13, TP14: TestPoint, TestPoint:TestPoint_Pad_D1.5mm, symbol Connector:TestPoint
- renumbered R to R1
Connections:
- net Earth: now also J6.3
- net UART_RX: now also J6.2, TP13.1
- net UART_TX: now also J6.1, TP14.1

Commit message: some footprints + print
Parts:
- C11, C12, C13, C14, C15, C16: footprint Capacitor_SMD_Wurth:C_Wurth_WCAP-CSGP-1210_H2.5 -> Capasitors:C_Wurth_WCAP-CSGP-0603_R
- C39, C43, C44, C45: footprint (none) -> Capasitors:C_Wurth_WCAP-CSGP-0603_R
- D10: footprint SOD2512X110N -> Diode_SMD:D_SMB
- D13, D7, D9: footprint LED_SMD_Wurth:D_Wurth_WL-SMCD-0603 -> WL-LED:D_Wurth_WL-SMCD-0603
- D4: footprint Diode_SMD_Wurth:D_Wurth_WE-TVS-SOT23-6L -> Package_TO_SOT_SMD:SOT-23-6
- IC2: footprint QFP50P900X900X160-48N -> Package_QFP:LQFP-48_7x7mm_P0.5mm
- IC3: footprint SOT65P210X110-5N -> Package_TO_SOT_SMD:SOT-23-5
- R1, R35, R37, R38, R39, R53, R54: footprint (none) -> WE-Resistors:R_Wurth_WRIS-KSKE-0603
Changed lines of the file:
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@@
 			)
 		)
-		(property "Footprint" "Capacitor_SMD_Wurth:C_Wurth_WCAP-CSGP-1210_H2.5"
+		(property "Footprint" "Capasitors:C_Wurth_WCAP-CSGP-0603_R"
 			(at 132.08 156.21 0)
 			(hide yes)
@@
 			)
 		)
-		(property "Footprint" "SOD2512X110N"
+		(property "Footprint" "Diode_SMD:D_SMB"
 			(at 243.51 40.64 0)
 			(hide yes)
@@
 			)
 		)
-		(property "Footprint" "SOT65P210X110-5N"
+		(property "Footprint" "Package_TO_SOT_SMD:SOT-23-5"
 			(at 234.95 172.39 0)
 			(hide yes)
@@
 			)
 		)
-		(property "Footprint" "Diode_SMD_Wurth:D_Wurth_WE-TVS-SOT23-6L"
+		(property "Footprint" "Package_TO_SOT_SMD:SOT-23-6"
 			(at 237.49 116.84 0)
 			(hide yes)
@@
 		(dnp no)
 		(property "Reference" "D6"
-			(at 148.844 134.62 90)
+			(at 161.036 130.048 90)
 			(show_name no)
 			(do_not_autoplace no)
@@
 			)
 		)
-		(property "Footprint" "Capacitor_SMD_Wurth:C_Wurth_WCAP-CSGP-1210_H2.5"
+		(property "Footprint" "Capasitors:C_Wurth_WCAP-CSGP-0603_R"
 			(at 97.79 35.56 0)
 			(hide yes)
@@
 			)
 		)
-		(property "Footprint" ""
+		(property "Footprint" "WE-Resistors:R_Wurth_WRIS-KSKE-0603"
 			(at 245.11 50.038 90)
 			(hide yes)
@@
 			)
 		)
-		(property "Footprint" ""
+		(property "Footprint" "Capasitors:C_Wurth_WCAP-CSGP-0603_R"
 			(at 42.2148 72.39 0)
 			(hide yes)
@@
 			)
 		)
-		(property "Footprint" "Capacitor_SMD_Wurth:C_Wurth_WCAP-CSGP-1210_H2.5"
+		(property "Footprint" "Capasitors:C_Wurth_WCAP-CSGP-0603_R"
 			(at 252.73 67.31 0)
 			(hide yes)
@@
 			)
 		)
-		(property "Footprint" "Capacitor_SMD_Wurth:C_Wurth_WCAP-CSGP-1210_H2.5"
+		(property "Footprint" "Capasitors:C_Wurth_WCAP-CSGP-0603_R"
 			(at 261.62 67.31 0)
 			(hide yes)
@@
 			)
 		)
-		(property "Footprint" "LED_SMD_Wurth:D_Wurth_WL-SMCD-0603"
+		(property "Footprint" "WL-LED:D_Wurth_WL-SMCD-0603"
 			(at 8.89 154.94 0)
 			(hide yes)
@@
 			)
 		)
-		(property "Footprint" "QFP50P900X900X160-48N"
+		(property "Footprint" "Package_QFP:LQFP-48_7x7mm_P0.5mm"
 			(at 86.36 187.63 0)
 			(hide yes)
@@
 			)
 		)
-		(property "Footprint" "Capacitor_SMD_Wurth:C_Wurth_WCAP-CSGP-1210_H2.5"
+		(property "Footprint" "Capasitors:C_Wurth_WCAP-CSGP-0603_R"
 			(at 228.6 24.13 0)
 			(hide yes)
@@
 			)
 		)
-		(property "Footprint" ""
+		(property "Footprint" "WE-Resistors:R_Wurth_WRIS-KSKE-0603"
 			(at 245.11 31.242 90)
 			(hide yes)
@@
 			)
 		)
-		(property "Footprint" ""
+		(property "Footprint" "WE-Resistors:R_Wurth_WRIS-KSKE-0603"
 			(at 43.688 158.75 90)
 			(hide yes)
@@
 			)
 		)
-		(property "Footprint" ""
+		(property "Footprint" "Capasitors:C_Wurth_WCAP-CSGP-0603_R"
 			(at 48.26 53.0352 0)
 			(hide yes)
@@
 			)
 		)
-		(property "Footprint" ""
+		(property "Footprint" "Capasitors:C_Wurth_WCAP-CSGP-0603_R"
 			(at 58.42 47.9552 0)
 			(hide yes)
@@
 			)
 		)
-		(property "Footprint" ""
+		(property "Footprint" "WE-Resistors:R_Wurth_WRIS-KSKE-0603"
 			(at 179.578 85.09 90)
 			(hide yes)
@@
 			)
 		)
-		(property "Footprint" ""
+		(property "Footprint" "Capasitors:C_Wurth_WCAP-CSGP-0603_R"
 			(at 68.58 42.8752 0)
 			(hide yes)
@@
 			)
 		)
-		(property "Footprint" "Capacitor_SMD_Wurth:C_Wurth_WCAP-CSGP-1210_H2.5"
+		(property "Footprint" "Capasitors:C_Wurth_WCAP-CSGP-0603_R"
 			(at 72.39 39.37 0)
 			(hide yes)
@@
 			)
 		)
-		(property "Footprint" "LED_SMD_Wurth:D_Wurth_WL-SMCD-0603"
+		(property "Footprint" "WL-LED:D_Wurth_WL-SMCD-0603"
 			(at 15.24 154.94 0)
 			(hide yes)
@@
 			)
 		)
-		(property "Footprint" ""
+		(property "Footprint" "WE-Resistors:R_Wurth_WRIS-KSKE-0603"
 			(at 37.338 158.75 90)
 			(hide yes)
@@
 			)
 		)
-		(property "Footprint" ""
+		(property "Footprint" "WE-Resistors:R_Wurth_WRIS-KSKE-0603"
 			(at 30.988 158.75 90)
 			(hide yes)
@@
 			)
 		)
-		(property "Footprint" ""
+		(property "Footprint" "WE-Resistors:R_Wurth_WRIS-KSKE-0603"
 			(at 174.498 85.09 90)
 			(hide yes)
@@
 			)
 		)
-		(property "Footprint" "LED_SMD_Wurth:D_Wurth_WL-SMCD-0603"
+		(property "Footprint" "WL-LED:D_Wurth_WL-SMCD-0603"
 			(at 21.59 154.94 0)
 			(hide yes)

Commit message: v 1.1
Fiksa ting
starta layout
bedre schematic design
whooppppppwhhoop
Parts:
- removed J5: 62701021621, Connector_THT_Wurth:J_Wurth_WR-BHD_62701021621, symbol SWD-Header:62701021621
- removed R38, R39: 10k, WE-Resistors:R_Wurth_WRIS-KSKE-0603, symbol Device:R
- removed SW2: 434123025826, Switch_SMD_Wurth:SW_Wurth_WS-TASV_434123025826, symbol WS-TASV:434123025826
- added J5: 62701020621, Connector_SMD_Wurth:J_Wurth_WR-BHD_62701020621, symbol SWD-Header:62701020621
- J3: footprint Connector_SMD_Wurth:J_Wurth_WR-WTB_653104124022 -> Connectors_tht:J_Wurth_WR-MPC4_64900411122
- J6: footprint Connector_THT_Wurth:J_Wurth_WR-PHD_61300311021 -> Connectors_tht:J_Wurth_WR-PHD_61300311021
- J9: footprint Connector_SMD_Wurth:J_Wurth_WR-USB_629722000214 -> Conectors:J_Wurth_WR-USB_629722000214
- SW1: footprint Switch_SMD_Wurth:SW_Wurth_WS-TASV_434123025826 -> Switch:SW_Wurth_WS-TASV_434123025826
- renumbered U5 to U15
Connections:
- net +3V3: now also J5.1
- net Earth: now also J5.3, J5.5, J5.9
- net NRST: now also J5.10
- net SWCLK: now also J5.4
- net SWDIO: now also J5.2
- net SWO: now also J5.6
Other:
- note added: "RESET"
- note added: "RGB LED"
- note removed: "RESET / BOOT"
- note removed: "RGB_LED"

Commit message: post-schematic_review 💯
fixed stuff
added stuff
GND is good
I2C BME280
memes
fixed pins
more stuff
💯
Parts:
- removed J3: 653104124022, Connectors_tht:J_Wurth_WR-MPC4_64900411122, symbol WR-WTB:653104124022
- added J2: 61300421121, Connectors_tht:J_Wurth_WR-PHD_61300421121, symbol Connector_Wurth_WR-PHD:61300421121
Connections:
- net +5V: now also J2.1
- net CAN1_TX: now also IC2.46 (PB9); no longer IC2.41 (PB5)
- net CAN2_RX: now also IC2.41 (PB5); no longer IC2.42 (PB6)
- net CAN2_TX: now also IC2.42 (PB6); no longer IC2.43 (PB7)
- net Earth: now also J2.3
- net OSC48M: now also IC2.3 (PC14-OSC32_IN); no longer IC2.5 (PH0-OSC_IN)
- net SCK: now also IC2.6 (PH1-OSC_OUT); no longer IC2.15 (PA5)
- net UART_TX: now also IC2.30 (PA9); no longer IC2.46 (PB9)
- net Y: now also J2.2
- net CSB: no longer names the net of IC2.16 (PA6)
- net IMON renamed IMON_BIG
- net SPI1_MISO renamed IMON_SMALL
- net SPI1_MOSI: no longer names the net of IC2.17 (PA7)
- new net SDI: IC2.5 (PH0-OSC_IN)
- no-connect marks 19 -> 20
Other:
- moved on the sheet: C14, D13, D6, D7, D9, IC2, J6, TP13, TP14, Y1
