File: torpedokontroller/processing.kicad_sch (KiCad schematic)
At the start: 32 parts, among them IC2 STM32C542CCT6, IC3 SN74AHCT1G125DCKR, J2 61300421121, J5 62701020621, J6 61300311021, J9 USB_C_Receptacle_USB2.0_16P, SW1 434123025826, U15 WE-TVS-82400102, Y1 48 MHz

Commit message: v 1.2
PWM SERVOS :)) YAAADDAAAAAa
Layout begynner å komme seg
Parts:
- removed J6: 61300311021, Connectors_tht:J_Wurth_WR-PHD_61300311021, symbol Connector_Wurth_WR-PHD:61300311021
- added J3: 61300311021, Connectors_tht:J_Wurth_WR-PHD_62000311121, symbol Connector_Wurth_WR-PHD:61300311021
- D6: footprint Diode_SMD_Wurth:D_Wurth_WE-TVS-SOT143-4L -> uglyass:8240136
Connections:
- net Earth: now also J3.3
- net UART_RX: now also J3.2
- net UART_TX: now also J3.1
- net +VBUS_USB: now reaches D10.2 (A), J9.A4 (VBUS), J9.A9 (VBUS1), J9.B4 (VBUS3), J9.B9 (VBUS2), U15.5
