File: torpedokontroller/torpedokontroller.kicad_pcb (KiCad board)
At the start: 2 copper layers, 7 parts, among them IC1 STM32C542RCT6, IC2 TCAN3414DR, IC3 TPS26400PWPR, IC4 TCAN3414DR, Q3 PMOS

Commit message: v 1.1
Fiksa ting
starta layout
bedre schematic design
whooppppppwhhoop
Parts:
- removed IC4: TCAN3414DR, Samacsys:SOIC127P600X175-8N
- removed Q3: PMOS, Package_DIP:DIP-24_W7.62mm
- removed R3: R, Package_QFP:LQFP-100_14x14mm_P0.5mm
- added C11: 4.7 uF, Capasitors:C_Wurth_WCAP-CSGP-0603_R, F.Cu at (148.6, 156.4)
- added C12: 2.2 uF, Capasitors:C_Wurth_WCAP-CSGP-0603_R, F.Cu at (156.2, 99.5)
- added C13: 0.1 uF, Capasitors:C_Wurth_WCAP-CSGP-0603_R, F.Cu at (163.7, 98.8)
- added C14: 0.1 uF, Capasitors:C_Wurth_WCAP-CSGP-0603_R, F.Cu at (164.4, 96.5)
- added C15: 100nF, Capasitors:C_Wurth_WCAP-CSGP-0603_R, F.Cu at (102.0, 157.6)
- added C16: 1u, Capasitors:C_Wurth_WCAP-CSGP-0603_R, F.Cu at (98.2, 165.4)
- added C21: 100n, Capasitors:C_Wurth_WCAP-CSGP-0603_R, F.Cu at (94.2, 73.2)
- added C22: 100n, Capasitors:C_Wurth_WCAP-CSGP-0603_R, F.Cu at (94.2, 75.6)
- added C23: 1u, Capasitors:C_Wurth_WCAP-CSGP-0603_R, F.Cu at (94.2, 78.1)
- added C24: 4.7 uF, Capasitors:C_Wurth_WCAP-CSGP-0603_R, F.Cu at (94.2, 80.5)
- added C25: 4.7 uF, Capasitors:C_Wurth_WCAP-CSGP-0603_R, F.Cu at (98.1, 68.3)
- added C26: 4.7 uF, Capasitors:C_Wurth_WCAP-CSGP-0603_R, F.Cu at (98.1, 70.7)
- added C27: 22 uF, Capasitors:C_Wurth_WCAP-CSGP-0603_R, F.Cu at (98.1, 73.2)
- added C28: 22 uF, Capasitors:C_Wurth_WCAP-CSGP-0603_R, F.Cu at (98.1, 75.6)
- added C29: 4.7 uF, Capasitors:C_Wurth_WCAP-CSGP-0603_R, F.Cu at (98.1, 78.1)
- added C30: 4.7 uF, Capasitors:C_Wurth_WCAP-CSGP-0603_R, F.Cu at (98.1, 80.5)
- added C31: 4.7 uF, Capasitors:C_Wurth_WCAP-CSGP-0603_R, F.Cu at (176.9, 126.4)
- added C32: 4.7 uF, Capasitors:C_Wurth_WCAP-CSGP-0603_R, F.Cu at (101.9, 68.3)
- added C33: 4.7 uF, Capasitors:C_Wurth_WCAP-CSGP-0603_R, F.Cu at (61.0, 96.2)
- added C34: 22 uF, Capasitors:C_Wurth_WCAP-CSGP-0603_R, F.Cu at (101.9, 73.2)
- added C35: 22 uF, Capasitors:C_Wurth_WCAP-CSGP-0603_R, F.Cu at (60.8, 91.2)
- added C37: 330nF, Capasitors:C_Wurth_WCAP-CSGP-0603_R, F.Cu at (163.0, 131.5)
- added C38: 0.1uF, Capasitors:C_Wurth_WCAP-CSGP-0603_R, F.Cu at (164.5, 132.8)
- added C39: 100n, Capasitors:C_Wurth_WCAP-CSGP-0603_R, F.Cu at (161.4, 96.3)
- added C41: 4.7 uF, Capasitors:C_Wurth_WCAP-CSGP-0603_R, F.Cu at (176.9, 133.7)
- added C42: 0.1uF, Capasitors:C_Wurth_WCAP-CSGP-0603_R, F.Cu at (176.9, 136.2)
- added C43: 100n, Capasitors:C_Wurth_WCAP-CSGP-0603_R, F.Cu at (154.7, 99.5)
- added C44: 100n, Capasitors:C_Wurth_WCAP-CSGP-0603_R, F.Cu at (152.9, 92.8)
- added C45: 100n, Capasitors:C_Wurth_WCAP-CSGP-0603_R, F.Cu at (159.7, 91.0)
- added C46: 10nF, Capasitors:C_Wurth_WCAP-CSGP-0603_R, F.Cu at (176.9, 138.6)
- added C8: 4.7 uF, Capasitors:C_Wurth_WCAP-CSGP-0603_R, F.Cu at (94.2, 68.3)
- added C9: 4.7 uF, Capasitors:C_Wurth_WCAP-CSGP-0603_R, F.Cu at (94.2, 70.7)
- added D1: 18V, Diode_SMD:D_SMA, F.Cu at (131.4, 87.6)
- added D10: NSR0530HT1G, Diode_SMD:D_SMB, F.Cu at (115.0, 165.0)
- added D11: 0603_150060RS55040, WL-LED:D_Wurth_WL-SMCD-0603, F.Cu at (79.6, 86.4)
- added D13: 0603_150060YS55040, WL-LED:D_Wurth_WL-SMCD-0603, F.Cu at (155.4, 95.5)
- added D14: 0603_150060BS55040, WL-LED:D_Wurth_WL-SMCD-0603, F.Cu at (202.2, 152.7)
- added D15: 0603_150060RS55040, WL-LED:D_Wurth_WL-SMCD-0603, F.Cu at (202.2, 155.0)
- added D16: 0603_150060BS55040, WL-LED:D_Wurth_WL-SMCD-0603, F.Cu at (76.2, 89.5)
- added D17: SOT23-3L_824094024, Package_TO_SOT_SMD:SOT-23-3, F.Cu at (176.0, 92.4)
- added D19: 18V, Diode_SMD:D_SMA, F.Cu at (177.4, 99.6)
- added D2: DO214-AA-600W_BI_824521261, Diode_SMD:D_SMB, F.Cu at (219.0, 151.2)
- added D20: SOT23-3L_824094024, Package_TO_SOT_SMD:SOT-23-3, F.Cu at (211.9, 105.6)
- added D3: 18V, Diode_SMD:D_SMA, F.Cu at (213.4, 101.1)
- added D4: SOT23-6L_824015043, Package_TO_SOT_SMD:SOT-23-6, F.Cu at (188.5, 49.0)
- added D7: 0603_150060GS55040, WL-LED:D_Wurth_WL-SMCD-0603, F.Cu at (155.4, 94.2)
- added D9: 0603_150060RS55040, WL-LED:D_Wurth_WL-SMCD-0603, F.Cu at (155.4, 97.0)
- added IC8: TCAN3414DR, Samacsys:SOIC127P600X175-8N, F.Cu at (156.1, 85.8)
- added IC9: TCAN3414DR, Samacsys:SOIC127P600X175-8N, F.Cu at (190.4, 149.6)
- added J1: 64900411122, Connectors_tht:J_Wurth_WR-MPC4_64900411122, B.Cu at (182.0, 99.6)
- added J11: 61302021121, Connectors_tht:J_Wurth_WR-PHD_61302021121, F.Cu at (204.5, 93.8)
- added J3: 653104124022, Connectors_tht:J_Wurth_WR-MPC4_64900411122, B.Cu at (95.4, 165.4)
- added J4: Ground_hook, Connectors_tht:J_Wurth_WR-PHD_61300111121, F.Cu at (99.8, 84.0)
- added J5: 62701020621, Connector_SMD_Wurth:J_Wurth_WR-BHD_62701020621, B.Cu at (188.5, 48.8)
- added J6: 61300311021, Connectors_tht:J_Wurth_WR-PHD_61300311021, F.Cu at (195.8, 61.3)
- added J7: H, Connectors_tht:J_Wurth_WR-PHD_61300111121, F.Cu at (177.2, 96.0)
- added J8: L, Connectors_tht:J_Wurth_WR-PHD_61300111121, F.Cu at (177.2, 88.8)
- added J9: USB_C_Receptacle_USB2.0_16P, Conectors:J_Wurth_WR-USB_629722000214, F.Cu at (131.2, 101.2)
- added L3: 1.0 uH, Inductor:L_Wurth_WE-PD2-4532, F.Cu at (110.7, 70.2)
- added L4: 1.0 uH, Inductor:L_Wurth_WE-PD2-4532, F.Cu at (110.7, 76.3)
- added Q1: STANDARD_140356145200, WL-OCPT:Q_Wurth_WL-OCPT_SOP4-STANDARD, F.Cu at (141.0, 155.8)
- added Q2: SiS443DN, Package_SO:Vishay_PowerPAK_1212-8_Single, F.Cu at (197.6, 153.9)
- added R2: 0, WE-Resistors:R_Wurth_WRIS-KSKE-0603, F.Cu at (80.9, 61.4)
- added R23: 330k, WE-Resistors:R_Wurth_WRIS-KSKE-0603, F.Cu at (105.6, 70.7)
- added R24: 11k, WE-Resistors:R_Wurth_WRIS-KSKE-0603, F.Cu at (105.6, 73.2)
- added R25: 24k9, WE-Resistors:R_Wurth_WRIS-KSKE-0603, F.Cu at (105.6, 75.6)
- added R27: 10k, WE-Resistors:R_Wurth_WRIS-KSKE-0603, F.Cu at (105.6, 78.1)
- added R28: 24k9, WE-Resistors:R_Wurth_WRIS-KSKE-0603, F.Cu at (105.6, 80.5)
- added R29: 4k7, WE-Resistors:R_Wurth_WRIS-KSKE-0603, F.Cu at (105.6, 82.9)
- added R33: 1K, WE-Resistors:R_Wurth_WRIS-KSKE-0603, F.Cu at (134.4, 159.2)
- added R34: 100k, WE-Resistors:R_Wurth_WRIS-KSKE-0603, F.Cu at (154.5, 131.5)
- added R35: 4k, WE-Resistors:R_Wurth_WRIS-KSKE-0603, F.Cu at (158.2, 93.3)
- added R37: 750, WE-Resistors:R_Wurth_WRIS-KSKE-0603, F.Cu at (158.2, 96.3)
- added R44: 2k, WE-Resistors:R_Wurth_WRIS-KSKE-0603, F.Cu at (180.6, 131.3)
- added R45: 42k, WE-Resistors:R_Wurth_WRIS-KSKE-0603, F.Cu at (180.6, 133.7)
- added R46: 4k7, WE-Resistors:R_Wurth_WRIS-KSKE-0603, F.Cu at (180.6, 136.2)
- added R47: 8k2, WE-Resistors:R_Wurth_WRIS-KSKE-0603, F.Cu at (174.0, 145.0)
- added R48: 33k, WE-Resistors:R_Wurth_WRIS-KSKE-0603, F.Cu at (184.2, 128.9)
- added R49: 2k, WE-Resistors:R_Wurth_WRIS-KSKE-0603, F.Cu at (184.2, 131.3)
- added R50: 1k, WE-Resistors:R_Wurth_WRIS-KSKE-0603, F.Cu at (184.2, 133.7)
- added R51: 10k, WE-Resistors:R_Wurth_WRIS-KSKE-0603, F.Cu at (184.2, 136.2)
- added R52: 160, WE-Resistors:R_Wurth_WRIS-KSKE-0603, F.Cu at (187.7, 126.4)
- added R53: 5k1, WE-Resistors:R_Wurth_WRIS-KSKE-0603, F.Cu at (137.7, 105.3)
- added R54: 5k1, WE-Resistors:R_Wurth_WRIS-KSKE-0603, F.Cu at (137.4, 99.3)
- added R55: 120, WE-Resistors:R_Wurth_WRIS-KSKE-0603, F.Cu at (187.7, 128.9)
- added R56: 120, WE-Resistors:R_Wurth_WRIS-KSKE-0603, F.Cu at (187.7, 131.3)
- added R57: 120, WE-Resistors:R_Wurth_WRIS-KSKE-0603, F.Cu at (154.6, 81.3)
- added R58: 10, WE-Resistors:R_Wurth_WRIS-KSKE-0603, F.Cu at (187.7, 133.7)
- added R7: 1k7, WE-Resistors:R_Wurth_WRIS-KSKE-0603, F.Cu at (105.6, 68.3)
- added SW1: 434123025826, Switch:SW_Wurth_WS-TASV_434123025826, F.Cu at (159.9, 99.0)
- added SW3: 418127270901, Switch_THT:SW_Wurth_WS-DITV_418127270901, F.Cu at (151.4, 85.1)
- added TP11: TestPoint, TestPoint:TestPoint_Pad_D1.5mm, F.Cu at (176.8, 148.7)
- added TP12: TestPoint, TestPoint:TestPoint_Pad_D1.5mm, F.Cu at (176.8, 152.3)
- added TP13: TestPoint, TestPoint:TestPoint_Pad_D1.5mm, F.Cu at (113.9, 116.9)
- added TP14: TestPoint, TestPoint:TestPoint_Pad_D1.5mm, F.Cu at (113.9, 120.5)
- added TP3: TestPoint, TestPoint:TestPoint_Pad_D1.5mm, B.Cu at (154.2, 104.0)
- added TP4: TestPoint, TestPoint:TestPoint_Pad_D1.5mm, B.Cu at (163.9, 107.0)
- added TP7: TestPoint, TestPoint:TestPoint_Pad_D1.5mm, B.Cu at (163.9, 104.5)
- added TP8: TestPoint, TestPoint:TestPoint_Pad_D1.5mm, B.Cu at (163.9, 102.0)
- added U0: 7982-1-15-20-75-14-11-0, Samacsys:7982115207514110, B.Cu at (129.0, 81.2)
- added U1: 7982-1-15-20-75-14-11-0, Samacsys:7982115207514110, B.Cu at (129.0, 85.4)
- added U10: 7982-1-15-20-75-14-11-0, Samacsys:7982115207514110, F.Cu at (101.8, 49.8)
- added U11: 7982-1-15-20-75-14-11-0, Samacsys:7982115207514110, F.Cu at (106.0, 49.8)
- added U12: 173950336, Buck_down:173950536, F.Cu at (87.6, 76.9)
- added U13: 173950536, Buck_down:173950536, F.Cu at (54.5, 96.3)
- added U14: BME280, Package_LGA:Bosch_LGA-8_2.5x2.5mm_P0.65mm_ClockwisePinNumbering, F.Cu at (158.4, 103.5)
- added U15: WE-TVS-82400102, Package_TO_SOT_SMD:SOT-23-6, F.Cu at (137.8, 102.1)
- added U16: TPS26400PWP, Package_SO:HTSSOP-16-1EP_4.4x5mm_P0.65mm_EP3.4x5mm_Mask2.66x2.46mm_ThermalVias, F.Cu at (111.8, 82.5)
- added U2: 7982-1-15-20-75-14-11-0, Samacsys:7982115207514110, B.Cu at (129.0, 89.6)
- added U3: 7982-1-15-20-75-14-11-0, Samacsys:7982115207514110, B.Cu at (129.0, 93.8)
- added U4: 7982-1-15-20-75-14-11-0, Samacsys:7982115207514110, F.Cu at (100.1, 59.3)
- added U5: 7982-1-15-20-75-14-11-0, Samacsys:7982115207514110, F.Cu at (100.1, 64.5)
- added U6: 7982-1-15-20-75-14-11-0, Samacsys:7982115207514110, F.Cu at (105.2, 54.5)
- added U7: 7982-1-15-20-75-14-11-0, Samacsys:7982115207514110, F.Cu at (105.3, 59.3)
- added U8: 7982-1-15-20-75-14-11-0, Samacsys:7982115207514110, F.Cu at (105.3, 64.5)
- added U9: 7982-1-15-20-75-14-11-0, Samacsys:7982115207514110, F.Cu at (100.5, 54.5)
- added Y1: 48 MHz, Crystal_SMD_Wurth:Y_Wurth_WE-SPXO-CFPS-39, F.Cu at (162.2, 92.0)
- IC1: value STM32C542RCT6 -> NCP81296MNTXG; footprint Samacsys:QFP50P1200X1200X160-64N -> big_efuse:QFN50P500X500X140-33N
- IC2: value TCAN3414DR -> STM32C542CCT6; footprint Samacsys:SOIC127P600X175-8N -> Package_QFP:LQFP-48_7x7mm_P0.5mm; moved to B.Cu
- IC3: value TPS26400PWPR -> SN74AHCT1G125DCKR; footprint Samacsys:SOP65P640X120-17N -> Package_TO_SOT_SMD:SOT-23-5
- R1: value R -> 680; footprint Package_QFP:LQFP-100_14x14mm_P0.5mm -> WE-Resistors:R_Wurth_WRIS-KSKE-0603
- moved IC3 75.6 mm to (102.0, 160.8)
- moved IC1 35.9 mm to (158.9, 131.8)
- moved R1 17.0 mm to (158.2, 94.8)
- moved IC2 15.3 mm to (157.2, 95.3), turned to 180 degrees
Connections:
- IC1 pad 10: unconnected-(IC1-PC2-Pad10) -> +VBAT
- IC1 pad 11: unconnected-(IC1-PC3-Pad11) -> +VBAT
- IC1 pad 12: unconnected-(IC1-VREF--Pad12) -> +VBAT
- IC1 pad 13: unconnected-(IC1-VREF+-Pad13) -> +VBAT
- IC1 pad 14: unconnected-(IC1-PA0-Pad14) -> +VBAT
- IC1 pad 15: unconnected-(IC1-PA1-Pad15) -> +VBAT
- IC1 pad 16: unconnected-(IC1-PA2-Pad16) -> +VBAT
- IC1 pad 18: unconnected-(IC1-VSS_1-Pad18) -> Net-(IC1-VTEMP)
- IC1 pad 19: unconnected-(IC1-VDD_1-Pad19) -> Net-(IC1-SS)
- IC1 pad 20: unconnected-(IC1-PA4-Pad20) -> Earth
- IC1 pad 21: unconnected-(IC1-PA5-Pad21) -> Net-(IC1-VDD)
- IC1 pad 22: unconnected-(IC1-PA6-Pad22) -> /output/IMON
- IC1 pad 23: unconnected-(IC1-PA7-Pad23) -> Net-(IC1-CS)
- IC1 pad 24: unconnected-(IC1-PC4-Pad24) -> Net-(IC1-CLREF)
- IC1 pad 25: unconnected-(IC1-PC5-Pad25) -> +VDD_servo
- IC1 pad 26: unconnected-(IC1-PB0-Pad26) -> +VDD_servo
- IC1 pad 27: unconnected-(IC1-PB1-Pad27) -> +VDD_servo
- IC1 pad 28: unconnected-(IC1-PB2-Pad28) -> +VDD_servo
- IC1 pad 29: unconnected-(IC1-PB10-Pad29) -> +VDD_servo
- IC1 pad 3: unconnected-(IC1-PC14-OSC32_IN-Pad3) -> /output/D_OC
- IC1 pad 30: unconnected-(IC1-VCAP-Pad30) -> +VDD_servo
- IC1 pad 31: unconnected-(IC1-VSS_2-Pad31) -> +VDD_servo
- IC1 pad 32: unconnected-(IC1-VDD_2-Pad32) -> +VDD_servo
- IC1 pad 33: Net-(IC1-PB12) -> +VBAT
- IC1 pad 4: unconnected-(IC1-PC15-OSC32_OUT-Pad4) -> /output/killswitch
- IC1 pad 5: unconnected-(IC1-PH0-OSC_IN-Pad5) -> /output/GOK
- IC1 pad 7: unconnected-(IC1-NRST-Pad7) -> Net-(IC1-VINF)
- IC1 pad 9: unconnected-(IC1-PC1-Pad9) -> +VBAT
- IC2 pad 1: Net-(IC1-PB13) -> unconnected-(IC2-PE2-Pad1)
- IC2 pad 2: Earth -> unconnected-(IC2-PC13-Pad2)
- IC2 pad 3: Net-(IC1-VDD_3) -> unconnected-(IC2-PC14-OSC32_IN-Pad3)
- IC2 pad 4: Net-(IC1-PB12) -> unconnected-(IC2-PC15-OSC32_OUT-Pad4)
- IC2 pad 5: Net-(IC1-PB15) -> /processing/OSC48M
- IC2 pad 7: unconnected-(IC2-CANH-Pad7) -> /processing/NRST
- IC2 pad 8: Net-(IC1-PB14) -> Earth
- IC3 pad 1: unconnected-(IC3-IN_1-Pad1) -> Earth
- IC3 pad 2: unconnected-(IC3-IN_2-Pad2) -> /processing/LED_MOSI
- IC3 pad 3: unconnected-(IC3-UVLO-Pad3) -> Earth
- IC3 pad 4: unconnected-(IC3-NC_1-Pad4) -> /processing/Y
- IC3 pad 5: unconnected-(IC3-OVP-Pad5) -> +5V
- R1 pad 2: unconnected-(R1-Pad2) -> Net-(IC2-PA1)
Routing:
- net /Input/CAN2_L: track 0.00 -> 17.8 mm
- net VBAT-CON: track 0.00 -> 15.0 mm
- net /output/CANH: track 0.00 -> 13.3 mm, vias 0 -> 1
- net /Input/SCK: track 0.00 -> 12.4 mm, vias 0 -> 2
- net /output/CANL: track 0.00 -> 12.2 mm, vias 0 -> 1
- net /Input/SPI1_MOIS: track 0.00 -> 11.6 mm, vias 0 -> 2
- net Earth: track 0.00 -> 10.7 mm, vias 0 -> 4
- net /Input/CAN2_H: track 0.00 -> 10.4 mm, vias 0 -> 2
- net +3V3: track 0.00 -> 9.84 mm, vias 0 -> 4
- net /Input/CSB: track 0.00 -> 9.51 mm, vias 0 -> 1
- net /Input/SPI1_MISO: track 0.00 -> 9.38 mm, vias 0 -> 1
- net Net-(J9-D+-PadA6): track 0.00 -> 8.22 mm
- net /Input/CAN2_TX: track 0.00 -> 6.74 mm, vias 0 -> 1
- net /output/IMON: track 0.00 -> 5.96 mm
- net /processing/NRST: track 0.00 -> 5.71 mm, vias 0 -> 1
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Other:
- board outline added: 65 x 65 mm

Commit message: post-schematic_review 💯
fixed stuff
added stuff
GND is good
I2C BME280
memes
fixed pins
more stuff
💯
Parts:
- removed D2: DO214-AA-600W_BI_824521261, Diode_SMD:D_SMB
- removed D20: SOT23-3L_824094024, Package_TO_SOT_SMD:SOT-23-3
- removed D3: 18V, Diode_SMD:D_SMA
- removed J11: 61302021121, Connectors_tht:J_Wurth_WR-PHD_61302021121
- removed J3: 653104124022, Connectors_tht:J_Wurth_WR-MPC4_64900411122
- removed R55: 120, WE-Resistors:R_Wurth_WRIS-KSKE-0603
- added D21: SOT23-3L_824094024, Package_TO_SOT_SMD:SOT-23-3, F.Cu at (141.1, 90.3)
- added J2: 61300421121, Connectors_tht:J_Wurth_WR-PHD_61300421121, F.Cu at (181.3, 81.7)
- J1: moved to F.Cu
- U10, U11, U4, U5, U6, U7, U8, U9: moved to B.Cu
- moved IC3 108.5 mm to (174.9, 80.5)
- moved D11 76.4 mm to (154.1, 103.2)
- moved Q2 73.3 mm to (141.1, 107.2), turned to 180 degrees
- moved D15 73.1 mm to (172.1, 88.4)
- moved TP12 67.0 mm to (165.6, 86.2)
- moved TP14 57.9 mm to (154.0, 78.6)
- moved R58 57.8 mm to (133.6, 113.6), turned to 180 degrees
- moved U10 57.2 mm to (139.8, 92.4), turned to 90 degrees
- moved TP13 56.0 mm to (162.8, 89.5)
- moved IC9 54.3 mm to (158.5, 105.7), turned to -90 degrees
- moved U9 51.7 mm to (135.6, 92.4), turned to 90 degrees
- moved U11 51.2 mm to (139.8, 88.2), turned to 90 degrees
- moved R33 51.0 mm to (130.1, 108.3), turned to -90 degrees
- moved C46 50.6 mm to (133.8, 112.2)
- moved Q1 48.6 mm to (134.8, 107.5)
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Connections:
- net +VDD_servo renamed /output/+VVD_Servo
- IC9 pad 6: Net-(IC9-CANL) -> /output/CANL
- IC9 pad 7: Net-(IC9-CANH) -> /output/CANH
- R56 pad 1: /output/CANL -> /output/CANH
- R56 pad 2: Net-(IC9-CANL) -> /output/CANL
Routing:
- net /processing/LED_MOSI: track 0.00 -> 12.8 mm, vias 0 -> 1
- net VBAT-CON: track 15.0 -> 27.5 mm
- net /Input/CAN2_L: track 17.8 -> 9.58 mm
- net /Input/CAN2_H: track 10.4 -> 3.30 mm, vias 2 -> 0
- net /output/CANH: track 13.3 -> 17.6 mm, vias 1 -> 3
- net /output/MCU_KillSwitch: track 0.00 -> 3.47 mm, vias 0 -> 1
- net /processing/Y: track 0.00 -> 2.87 mm
- net Net-(R57-Pad2): track 5.27 -> 2.68 mm
- net /output/CANL: track 12.2 -> 14.0 mm

Commit message: v 1.2
PWM SERVOS :)) YAAADDAAAAAa
Layout begynner å komme seg
Parts:
- removed J6: 61300311021, Connectors_tht:J_Wurth_WR-PHD_61300311021
- removed TP3, TP8: TestPoint, TestPoint:TestPoint_Pad_D1.5mm
- added D5: DFN1610-2L_824045817, zener:824045817, F.Cu at (141.3, 86.5)
- added D6: SOT143-4L_8240136, uglyass:8240136, F.Cu at (170.7, 113.9)
- added J3: 61300311021, Connectors_tht:J_Wurth_WR-PHD_62000311121, F.Cu at (168.4, 109.9)
- added Q3: AO3401A, Package_TO_SOT_SMD:SOT-23, F.Cu at (136.6, 92.1)
- added R30: 4k7, WE-Resistors:R_Wurth_WRIS-KSKE-0603, F.Cu at (164.1, 88.4)
- added R31: 4k7, WE-Resistors:R_Wurth_WRIS-KSKE-0603, F.Cu at (166.6, 87.9)
- added TP15: TestPoint, TestPoint:TestPoint_Pad_D1.5mm, F.Cu at (146.3, 113.0)
- added U18: TO263-7EP_171032401, MagIC_SMD_Wurth:U_Wurth_WPME-VDRM-TO263-7EP, F.Cu at (113.4, 92.1)
- U12, U13: moved to B.Cu
- moved C16 104.8 mm to (168.3, 87.5), turned to 90 degrees
- moved C35 103.7 mm to (161.9, 114.0)
- moved U13 101.7 mm to (154.9, 112.7), turned to 0 degrees
- moved C15 97.3 mm to (169.6, 87.5), turned to 90 degrees
- moved C33 92.8 mm to (151.0, 119.0), turned to 180 degrees
- moved D16 89.2 mm to (163.9, 105.8), turned to 90 degrees
- moved D10 82.7 mm to (168.1, 101.6), turned to 90 degrees
- moved R2 79.7 mm to (147.5, 105.2)
- moved C11 76.2 mm to (161.3, 81.2)
- moved C21 75.0 mm to (166.1, 94.5), turned to -90 degrees
- moved C22 72.9 mm to (164.6, 94.5), turned to -90 degrees
- moved U12 71.9 mm to (154.9, 102.2), turned to 0 degrees
- moved C34 71.8 mm to (161.9, 112.7)
- moved C28 70.0 mm to (162.6, 102.9), turned to -90 degrees
- moved C27 69.8 mm to (161.2, 102.9), turned to -90 degrees
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Connections:
- net /output/IMON renamed /output/IMON_BIG
- net /output/killswitch renamed /output/killswitch_output
- net Net-(D5-GND) renamed /output/RP_G
- C21 pad 2: GNDREF -> Earth
- C22 pad 2: GNDREF -> Earth
- C24 pad 2: GNDREF -> Earth
- C25 pad 1: +VBUS -> Net-(U12-VIN)
- C25 pad 2: GNDREF -> Earth
- C26 pad 1: +VBUS -> Net-(U12-VIN)
- C26 pad 2: GNDREF -> Earth
- C27 pad 2: GNDREF -> Earth
- C28 pad 2: GNDREF -> Earth
- C29 pad 2: GNDREF -> Earth
- C30 pad 2: GNDREF -> Earth
- C31 pad 2: GNDREF -> Earth
- C32 pad 2: GNDREF -> Earth
- C33 pad 2: GNDREF -> Earth
- C34 pad 2: GNDREF -> Earth
- C35 pad 2: GNDREF -> Earth
- C38 pad 1: Earth -> /output/vtemp_unfilterd
- C38 pad 2: Net-(IC1-VTEMP) -> Earth
- C8 pad 2: GNDREF -> Earth
- C9 pad 2: GNDREF -> Earth
- D16 pad 1: GNDREF -> Earth
- IC1 pad 18: Net-(IC1-VTEMP) -> /output/vtemp_unfilterd
- IC2 pad 15: /Input/SCK -> unconnected-(IC2-PA5-Pad15)
- IC2 pad 16: /Input/CSB -> unconnected-(IC2-PA6-Pad16)
- IC2 pad 17: /Input/SPI1_MOIS -> unconnected-(IC2-PA7-Pad17)
- IC2 pad 18: /Input/SPI1_MISO -> /Input/IMON_SMALL
- IC2 pad 3: unconnected-(IC2-PC14-OSC32_IN-Pad3) -> /processing/OSC48M
- IC2 pad 30: unconnected-(IC2-PA9-Pad30) -> /processing/UART_TX
- IC2 pad 41: /output/CAN1_TX -> /Input/CAN2_RX
- IC2 pad 42: /Input/CAN2_RX -> /Input/CAN2_TX
- IC2 pad 43: /Input/CAN2_TX -> unconnected-(IC2-PB7-Pad43)
- IC2 pad 46: /processing/UART_TX -> /output/CAN1_TX
- IC2 pad 5: /processing/OSC48M -> /Input/SDI
- IC2 pad 6: unconnected-(IC2-PH1-OSC_OUT-Pad6) -> /Input/SCK
- J4 pad 1: GNDREF -> Earth
- L3 pad 2: +VBUS -> Net-(U12-VIN)
- R28 pad 1: Net-(U16-IMON) -> /Input/IMON_SMALL
- R50 pad 2: Net-(IC1-VTEMP) -> /output/vtemp_unfilterd
- TP7 pad 1: /Input/SPI1_MOIS -> /Input/SDI
- U12 pad 1: +VBUS -> Net-(U12-VIN)
- U12 pad 2: GNDREF -> Earth
- U13 pad 2: GNDREF -> Earth
- U14 pad 1: GNDREF -> Earth
- U14 pad 2: /Input/CSB -> +3V3
- U14 pad 3: /Input/SPI1_MOIS -> /Input/SDI
- U14 pad 5: /Input/SPI1_MISO -> Earth
- U14 pad 7: GNDREF -> Earth
- U16 pad 10: Net-(U16-IMON) -> /Input/IMON_SMALL
- U16 pad 9: GNDREF -> Earth
Routing:
- net +VBUS: track 0.00 -> 26.3 mm, vias 0 -> 2
- net VBAT-CON: track 27.5 -> 5.00 mm
- net /Input/SDI: track 0.00 -> 18.1 mm, vias 0 -> 2
- net +3V3: track 9.84 -> 25.2 mm
- net Net-(C24-Pad1): track 0.00 -> 14.2 mm
- net /output/IMON_BIG: track 5.96 -> 19.0 mm, vias 0 -> 1
- net Net-(U13-VIN): track 0.00 -> 12.2 mm, vias 0 -> 1
- net /Input/SPI1_MOIS: track 11.6 -> 0.00 mm, vias 2 -> 0
- net /output/killswitch_output: track 0.00 -> 10.4 mm, vias 0 -> 2
- net /Input/CAN2_L: track 9.58 -> 0.00 mm
- net KILLSWITCH: track 0.00 -> 9.52 mm
- net /Input/CSB: track 9.51 -> 0.00 mm, vias 1 -> 0
- net /Input/IMON_SMALL: track 0.00 -> 9.30 mm
- net /output/GOK: track 5.45 -> 14.7 mm
- net /Input/SPI1_MISO: track 8.94 -> 0.00 mm, vias 1 -> 0
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Other:
- board size 65 x 65 mm -> 72 x 72 mm
- board text added: "litt jævlig å route MCU_KS"
