File: torpedokontroller/_restore_backup_2026-10-03T16-05-05-732/processing.kicad_sch (KiCad schematic)
At the start: 16 parts, among them IC3 STM32C542RCT6, J1 61300211021, J4 62701021621

Commit message: v0.5
USB2.0 implemented fr
many other things
Parts:
- removed J1: 61300211021, Connector_THT_Wurth:J_Wurth_WR-PHD_61300211021, symbol Connector_Wurth_WR-PHD:61300211021
- removed J4: 62701021621, Connector_THT_Wurth:J_Wurth_WR-BHD_62701021621, symbol SWD-Header:62701021621
