File: orin-bob/Connectors.kicad_sch (KiCad schematic)
At the start: 1 part, among them J2 62501021621

Commit message: Finished schematic for bob
Connections:
- net SCL2 renamed SCL
- net SDA2 renamed SDA
- net UART1_RX renamed UART1_RX1
Changed lines of the file:
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@@
 		)
 	)
-	(label "SCLK"
-		(at 125.73 59.69 180)
+	(hierarchical_label "SDI"
+		(shape output)
+		(at 92.71 62.23 180)
 		(effects
 			(font
 				(size 1.27 1.27)
 			)
-			(justify right bottom)
+			(justify right)
 		)
 	)
-	(label "SCL2"
-		(at 125.73 54.61 180)
+	(hierarchical_label "CS"
+		(shape bidirectional)
+		(at 92.71 59.69 180)
 		(effects
 			(font
 				(size 1.27 1.27)
 			)
-			(justify right bottom)
+			(justify right)
 		)
 	)
-	(label "SDA2"
-		(at 92.71 54.61 0)
+	(hierarchical_label "SDA"
+		(shape bidirectional)
+		(at 92.71 54.61 180)
 		(effects
 			(font
 				(size 1.27 1.27)
 			)
-			(justify left bottom)
+			(justify right)
 		)
 	)
-	(label "UART1_TX"
-		(at 92.71 57.15 0)
+	(hierarchical_label "UART1_TX"
+		(shape input)
+		(at 92.71 57.15 180)
 		(effects
 			(font
 				(size 1.27 1.27)
 			)
-			(justify left bottom)
+			(justify right)
 		)
 	)
-	(label "CANH"
-		(at 92.71 64.77 0)
+	(hierarchical_label "SCLK"
+		(shape bidirectional)
+		(at 125.73 59.69 0)
 		(effects
 			(font
 				(size 1.27 1.27)
 			)
-			(justify left bottom)
+			(justify left)
 		)
 	)
-	(label "UART1_RX"
-		(at 125.73 57.15 180)
+	(hierarchical_label "CANL"
+		(shape bidirectional)
+		(at 125.73 64.77 0)
 		(effects
 			(font
 				(size 1.27 1.27)
 			)
-			(justify right bottom)
+			(justify left)
 		)
 	)
-	(label "CANL"
-		(at 125.73 64.77 180)
+	(hierarchical_label "UART1_RX1"
+		(shape output)
+		(at 125.73 57.15 0)
 		(effects
 			(font
 				(size 1.27 1.27)
 			)
-			(justify right bottom)
+			(justify left)
 		)
 	)
-	(label "CS"
-		(at 92.71 59.69 0)
+	(hierarchical_label "SCL"
+		(shape bidirectional)
+		(at 125.73 54.61 0)
 		(effects
 			(font
 				(size 1.27 1.27)
 			)
-			(justify left bottom)
+			(justify left)
 		)
 	)
-	(label "SDI"
-		(at 92.71 62.23 0)
+	(hierarchical_label "CANH"
+		(shape bidirectional)
+		(at 92.71 64.77 180)
 		(effects
 			(font
 				(size 1.27 1.27)
 			)
-			(justify left bottom)
+			(justify right)
 		)
 	)
-	(label "SDO"
-		(at 125.73 62.23 180)
+	(hierarchical_label "SDO"
+		(shape input)
+		(at 125.73 62.23 0)
 		(effects
 			(font
 				(size 1.27 1.27)
 			)
-			(justify right bottom)
+			(justify left)
 		)
 	)

Commit message: some small changes
Parts:
- J2: footprint Connector_THT_Wurth:J_Wurth_WR-BHD_62501021621 -> 61201021621:61201021621
Changed lines of the file:
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@@
 			)
 		)
-		(property "Footprint" "Connector_THT_Wurth:J_Wurth_WR-BHD_62501021621"
+		(property "Footprint" "61201021621:61201021621"
 			(at 124.46 59.69 0)
 			(hide yes)

Commit message: Almost done schematic & PCB
Other:
- note added: "CAN + GND"
- note added: "WR-MPC3 Male Header Single Row x4"
Changed lines of the file:
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@@
 	(generator_version "10.0")
 	(paper "A5")
+	(text "CAN + GND"
+		(exclude_from_sim no)
+		(at 149.098 84.582 0)
+		(effects
+			(font
+				(size 1.27 1.27)
+			)
+		)
+	)
+	(text "WR-MPC3 Male Header Single Row x4\n"
+		(exclude_from_sim no)
+		(at 111.252 84.836 0)
+		(effects
+			(font
+				(size 1.27 1.27)
+			)
+		)
+	)
 	(wire
 		(pts

Commit message: Updated bob pcb
Parts:
- removed J2: 62501021621, 61201021621:61201021621, symbol 61230820621:62501021621
- added J10, J9: 653106131822, Wurth_WR-WTB:J_Wurth_WR-WTB_653106131822, symbol Wurth_WR-WTB:653106131822
- added J6: 653104131822, Wurth_WR-WTB:J_Wurth_WR-WTB_653104131822, symbol Wurth_WR-WTB:653104131822
- added J8: 653105131822, Wurth_WR-WTB:J_Wurth_WR-WTB_653105131822, symbol Wurth_WR-WTB:653105131822
Connections:
- net CANH: now also J8.2
- net CANL: now also J8.3
- net CS: now also J10.2
- net SCL: now also J6.3
- net SCLK: now also J10.3
- net SDA: now also J6.2
- net SDI: now also J10.5
- net SDO: now also J10.4
- net UART1_TX: now also J9.3
- new net +3V3_ISO_SPI: J10.1, J6.1, J8.1
- new net +3V3_ISO_UART: J9.1
- new net GND_ISO: J10.6, J6.4, J8.5, J9.6
- new net GPIOIN_ISO: J9.5
- new net GPIOOUT_ISO: J8.4
- new net PWM: J9.2
- new net UART1_RX: J9.4
Other:
- note added: "CAN"
- note added: "I2C"
- note added: "SPI"
- note added: "UART-config"

Commit message: Finished Version 1 BoB pcb
Connections:
- net +3V3_ISO_SPI: no longer J8.1
- net CANH: now also J8.3; no longer J8.2
- net CANL: now also J8.2; no longer J8.3
- net CS: now also J10.5; no longer J10.2
- net GPIOIN_ISO: now also J8.4; no longer J9.5
- net GPIOOUT_ISO: now also J9.2; no longer J8.4
- net PWM: now also J9.5; no longer J9.2
- net SCL: now also J6.2; no longer J6.3
- net SCLK: now also J10.4; no longer J10.3
- net SDA: now also J6.3; no longer J6.2
- net SDI: now also J10.2; no longer J10.5
- net SDO: now also J10.3; no longer J10.4
- net UART1_RX: now also J9.3; no longer J9.4
- net UART1_TX: now also J9.4; no longer J9.3
- new net +3V3_ISO_CAN: J8.1

Commit message: Fikset en god del småting i schematic
GPIO IN og OUT var flippet.
Mange små utsene ting.
La til Vortex Logo
Other:
- note removed: "CAN + GND"
- note removed: "WR-MPC3 Male Header Single Row x4"
- company: (none) -> Vortex NTNU
- title: (none) -> ORIN-BOB
Changed lines of the file:
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@@
 	(generator_version "10.0")
 	(paper "A5")
+	(title_block
+		(title "ORIN-BOB")
+		(date "2026-10-12")
+		(rev "1.0")
+		(company "Vortex NTNU")
+		(comment 1 "Yamn Sultan Salim")
+	)
 	(text "SPI\n"
 		(exclude_from_sim no)
@@
 		)
 	)
-	(text "CAN + GND"
-		(exclude_from_sim no)
-		(at 235.204 87.122 0)
-		(effects
-			(font
-				(size 1.27 1.27)
-			)
-		)
-	)
-	(text "WR-MPC3 Male Header Single Row x4\n"
-		(exclude_from_sim no)
-		(at 232.664 79.502 0)
-		(effects
-			(font
-				(size 1.27 1.27)
-			)
-		)
-	)
 	(wire
 		(pts
@@
 	)
 	(hierarchical_label "UART1_RX"
-		(shape input)
+		(shape output)
 		(at 146.05 82.55 180)
 		(effects
@@
 	)
 	(hierarchical_label "SDO"
-		(shape output)
+		(shape input)
 		(at 152.4 38.1 180)
 		(effects
@@
 	)
 	(hierarchical_label "PWM"
-		(shape output)
+		(shape input)
 		(at 146.05 87.63 180)
 		(effects
@@
 	)
 	(hierarchical_label "GPIOOUT_ISO"
-		(shape output)
+		(shape input)
 		(at 146.05 80.01 180)
 		(effects
@@
 	)
 	(hierarchical_label "UART1_TX"
-		(shape output)
+		(shape input)
 		(at 146.05 85.09 180)
 		(effects
@@
 	)
 	(hierarchical_label "SDI"
-		(shape input)
+		(shape output)
 		(at 152.4 35.56 180)
 		(effects
@@
 	)
 	(hierarchical_label "CS"
-		(shape bidirectional)
+		(shape input)
 		(at 152.4 43.18 180)
 		(effects
@@
 	)
 	(hierarchical_label "SCL"
-		(shape bidirectional)
+		(shape input)
 		(at 57.15 36.83 180)
 		(effects
@@
 	)
 	(hierarchical_label "SCLK"
-		(shape bidirectional)
+		(shape input)
 		(at 152.4 40.64 180)
 		(effects

Commit message: Viking Fix rest
Parts:
- removed J8: 653105131822, Wurth_WR-WTB:J_Wurth_WR-WTB_653105131822, symbol Wurth_WR-WTB:653105131822
- added J7: 653104131822, Wurth_WR-WTB:J_Wurth_WR-WTB_653104131822, symbol Wurth_WR-WTB:653104131822
Connections:
- net CANH: now also J7.3
- net CANL: now also J7.2
- net GND_ISO: now also J7.4
- net GPIOIN_ISO: now also J7.1

Commit message: Finished: Orin-BoB
Connections:
- net GPIOIN_ISO: now also J9.5; no longer J7.1
- net PWM: now also J7.1; no longer J9.5
Changed lines of the file:
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@@
+		)
+	)
+	(wire
+		(pts
+			(xy 146.05 87.63) (xy 158.75 87.63)
+		)
+		(stroke
+			(width 0)
+			(type default)
 		)
 	)
@@
 	(wire
 		(pts
+			(xy 158.75 30.48) (xy 158.75 33.02)
+		)
+		(stroke
+			(width 0)
+			(type default)
+		)
+	)
+	(wire
+		(pts
 			(xy 53.34 85.09) (xy 63.5 85.09)
 		)
@@
 	(wire
 		(pts
-			(xy 158.75 30.48) (xy 158.75 33.02)
-		)
-		(stroke
-			(width 0)
-			(type default)
-		)
-	)
-	(wire
-		(pts
 			(xy 157.48 74.93) (xy 157.48 77.47)
 		)
@@
 		(pts
 			(xy 152.4 35.56) (xy 160.02 35.56)
-		)
-		(stroke
-			(width 0)
-			(type default)
-		)
-	)
-	(wire
-		(pts
-			(xy 146.05 87.63) (xy 158.75 87.63)
 		)
 		(stroke
@@
 	(hierarchical_label "PWM"
 		(shape input)
-		(at 146.05 87.63 180)
+		(at 53.34 85.09 180)
 		(effects
 			(font
@@
 	(hierarchical_label "GPIOIN_ISO"
 		(shape output)
-		(at 53.34 85.09 180)
-		(effects
-			(font
+		(at 146.05 87.63 180)
+		(effects
+			(font
