File: orin-bob/digital_isolator.kicad_sch (KiCad schematic)
At the start: 25 parts, among them IC1 TCAN3414DR, U2 SOIC-8NB_18032011, U3 18024215401H, U4 18024215401H, U5 18024115401H

Commit message: Finished schematic for bob
Connections:
- net GND_out is gone; now on net GND_OUT: C15.2, IC1.2 (GND), IC1.8 (STB), U2.5 (GND2), U3.10 (SEL), U3.9 (GND2), U4.10 (SEL), U4.9 (GND2), U5.10 (SEL), U5.9 (GND2)
- net CAN0_DIN: no longer U4.5 (OUTC)
- net CAN0_DOUT: no longer U4.4 (INB)
- net CS: no longer U5.3 (INA)
- net GND: no longer C4.2
- net SCLK: no longer U5.4 (INB)
- net SDI: now also U5.11 (IND); no longer U5.12 (OUTC), U5.6 (OUTD)
- net SDO: now also U5.12 (OUTC); no longer U5.11 (IND), U5.5 (INC)
- net UART1_RX: no longer U3.5 (OUTC)
- net UART1_TX: no longer U3.4 (INB)
- net GND_OUT: now reaches C10.2, U3.15 (GND2)
- net GND_OUT: now also C14.2, C2.2, C4.2, U4.15 (GND2), U5.15 (GND2)
- net SCL1 renamed I2C5_CLK1
- net SCL2 renamed SCL
- net SDA1 renamed I2C5_DAT1
- net SDA2 renamed SDA
- net Vcc renamed 3V3
- net 3V3: now also C15.1, IC1.3 (VCC)
- net Vout renamed 3V3_ISO
- net 3V3_ISO: now also C14.1, U4.16 (VOUT)
- removed net Vout_C: C14.1, C15.1, IC1.3 (VCC), U4.16 (VOUT)
- net orin_GND renamed ORIN_GND
- new net CAN0_DIN1: U4.5 (OUTC)
- new net CAN0_DOUT1: U4.4 (INB)
- new net SPI1_CS0_N1: U5.3 (INA)
- new net SPI1_MISO1: U5.6 (OUTD)
- new net SPI1_MOSI1: U5.5 (INC)
- new net SPI1_SCK1: U5.4 (INB)
- new net UART1_RX1: U3.5 (OUTC)
- new net UART1_TX1: U3.4 (INB)
Other:
- note added: "SPI1_MOSI1"

Commit message: some small changes
Parts:
- removed C10, C7, C8, C9: 10uF, symbol Device:C_Small
- added C16, C17, C18, C19: 10uF, Capacitor_SMD:C_0201_0603Metric, symbol Device:C_Small
- C1, C11, C12, C13, C14, C15, C2, C3, C4, C5, C6: footprint (none) -> Capacitor_SMD:C_0201_0603Metric
- R1, R2, R3, R4, R5: footprint (none) -> Resistor_SMD:R_0603_1608Metric
- U2: footprint Snapeda:U_Wurth_WPME-CDI2C-SOIC8NB -> 18032111:U_Wurth_WPME-CDI2C-SOIC8NB
- U3, U4: footprint MagIC_SMD_Wurth:U_Wurth_WPME-CDIP_SOIC-16WB -> 18024215401H:U_Wurth_WPME-CDIP_SOIC-16WB
- U5: footprint MagIC_SMD_Wurth:U_Wurth_WPME-CDIP_SOIC-16WB -> 18024115401H:WPME-CDIP_SOIC16
Connections:
- net ORIN_GND is gone; now on net GND: U2.4 (GND1), U3.8 (GND1), U4.8 (GND1), U5.8 (GND1)
- net 3V3: now also C16.1, C17.1, C18.1; no longer C15.1, IC1.3 (VCC)
- net 3V3_ISO: now also C15.1, IC1.3 (VCC), C19.1
- net GND: now also C1.2, C11.2, C12.2, C13.2, C5.2, C6.2, U3.2 (GND1), U4.2 (GND1), U5.2 (GND1), C16.2, C17.2, C18.2
- net GND_OUT: now also C19.2; no longer C15.2, IC1.2 (GND), IC1.8 (STB), U2.5 (GND2), U3.10 (SEL), U3.9 (GND2), U4.10 (SEL), U4.9 (GND2), U5.10 (SEL), U5.9 (GND2)
- new net GND_ISO: C15.2, IC1.2 (GND), IC1.8 (STB), U2.5 (GND2), U3.10 (SEL), U3.9 (GND2), U4.10 (SEL), U4.9 (GND2), U5.10 (SEL), U5.9 (GND2)
- no-connect marks 6 -> 10
Other:
- note removed: "SPI1_MOSI1"

Commit message: Almost done schematic & PCB
Parts:
- removed C11, C12, C13, C14, C15: 10uF, Capacitor_SMD:C_0201_0603Metric, symbol Device:C_Small
- removed IC1: TCAN3414DR, Samacsys:SOIC127P600X175-8N, symbol Samacsys:TCAN3414DR
- removed R5: 120, Resistor_SMD:R_0603_1608Metric, symbol Device:R_Small
- removed U4: 18024215401H, 18024215401H:U_Wurth_WPME-CDIP_SOIC-16WB, symbol 18024215401H:18024215401H
- added C22, C24: 0.01uF, Capacitor_SMD:C_0603_1608Metric_Pad1.08x0.95mm_HandSolder, symbol Device:C_Small
- added C23, C25, C28: 0.1uF, Capacitor_SMD:C_0603_1608Metric_Pad1.08x0.95mm_HandSolder, symbol Device:C_Small
- added C26, C29: 10uF, Capacitor_SMD:C_0603_1608Metric_Pad1.08x0.95mm_HandSolder, symbol Device:C_Small
- added C27: 0.22uF, Capacitor_SMD:C_0603_1608Metric_Pad1.08x0.95mm_HandSolder, symbol Device:C_Small
- added FB1, FB2: BLM15HD182SN1D, BLM15HD182SN1D:IND_BLM15_0402_MUR-M, symbol Device:FerriteBead_Small
- added R6: 120, Resistor_SMD:R_0603_1608Metric_Pad0.98x0.95mm_HandSolder, symbol Device:R_Small
- added U6: ADM3057ExRW, Package_SO:SOIC-20W_7.5x12.8mm_P1.27mm, symbol Interface_CAN_LIN:ADM3057ExRW
- C1, C16, C17, C18, C19, C2, C3, C4, C5, C6: footprint Capacitor_SMD:C_0201_0603Metric -> Capacitor_SMD:C_0603_1608Metric_Pad1.08x0.95mm_HandSolder
- R1, R2, R3, R4: footprint Resistor_SMD:R_0603_1608Metric -> Resistor_SMD:R_0603_1608Metric_Pad0.98x0.95mm_HandSolder
Connections:
- net CAN0_DIN1: now also U6.5 (RXD)
- net CAN0_DOUT1: now also U6.7 (TXD)
- net CANH: now also R6.1, U6.14 (CANH)
- net CANL: now also R6.2, U6.13 (CANL)
- net GND: now also C24.1, C25.1, C28.1, C29.1, U6.1 (GND1), U6.10 (GND1), U6.2 (GND1)
- net GND_ISO: now also C22.1, C23.1, C26.1, FB2.2, U6.11 (GND2), U6.12 (RS), U6.15 (GND2), U6.18 (GNDISO), U6.20 (GNDISO)
- net GPIOIN_ISO: now reaches U3.11 (IND)
- net PWM: now reaches U3.14 (OUTA)
- net PWM01: now reaches U3.3 (INA)
- net GPIOIN: now reaches U3.6 (OUTD)
- net 3V3 renamed +3V3
- net +3V3: now also C24.2, C25.2, U6.4 (VIO)
- net 3V3_ISO renamed +3V3_ISO
- new net: C27.1, FB2.1
- new net +5V: C28.2, C29.2, U6.3 (VCC)
- new net +5V_ISO: C26.2, FB1.2
- new net GPIOOUT: U6.9 (AUXIN)
- new net GPIOOUT_ISO: U6.17 (AUXOUT)
- new net VISOOUT: C22.2, C23.2, C27.2, FB1.1, U6.16 (VISOIN), U6.19 (VISOOUT)
- no-connect marks 10 -> 3
Other:
- note removed: "CAN-config"
- note removed: "CAN-transceiver"
- moved on the sheet: C16, C17, C18, C19, C2, U3

Commit message: Updated bob pcb
Parts:
- U2: value SOIC-8NB_18032011 -> 18032011
Connections:
- net +5V_ISO is gone; now on net +3V3_ISO_SPI: C26.2, FB1.2
- net GND_ISO: now also C2.2, U5.15 (GND2)
- net GND_OUT: no longer C2.2, U5.15 (GND2)
- net +3V3_ISO renamed +3V3_ISO_SPI
- net +3V3_ISO_SPI: no longer C19.1, U3.16 (VOUT)
- new net +3V3_ISO_UART: C19.1, U3.16 (VOUT)
Other:
- note added: "CAN"
- moved on the sheet: C19, C22, C23, C24, C25, C26, C27, C28, C29, FB1, FB2, R6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

Commit message: Finished Version 1 BoB pcb
Connections:
- net GND_OUT is gone; now on net GND_ISO: C19.2, C4.2, U3.15 (GND2)
- net +3V3_ISO_SPI: no longer C26.2, FB1.2
- net VISOOUT renamed +3V3_ISO_CAN
- net +3V3_ISO_CAN: now also C26.2, FB1.2
Changed lines of the file:
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@@
 	(wire
 		(pts
-			(xy 54.61 140.97) (xy 55.88 140.97)
+			(xy 49.53 140.97) (xy 55.88 140.97)
 		)
 		(stroke
@@
 	(wire
 		(pts
-			(xy 54.61 148.59) (xy 55.88 148.59)
+			(xy 43.18 125.73) (xy 50.8 125.73)
 		)
 		(stroke
@@
 	(wire
 		(pts
-			(xy 43.18 125.73) (xy 50.8 125.73)
+			(xy 201.93 57.15) (xy 200.66 57.15)
 		)
 		(stroke
@@
 	(wire
 		(pts
-			(xy 201.93 57.15) (xy 200.66 57.15)
+			(xy 81.28 44.45) (xy 81.28 34.29)
 		)
 		(stroke
@@
 	(wire
 		(pts
-			(xy 81.28 44.45) (xy 81.28 34.29)
+			(xy 104.14 62.23) (xy 104.14 66.04)
 		)
 		(stroke
@@
 	(wire
 		(pts
-			(xy 104.14 62.23) (xy 104.14 66.04)
+			(xy 50.8 133.35) (xy 50.8 132.08)
 		)
 		(stroke
@@
 	(wire
 		(pts
-			(xy 50.8 133.35) (xy 50.8 132.08)
+			(xy 49.53 148.59) (xy 55.88 148.59)
 		)
 		(stroke
@@
 	(wire
 		(pts
+			(xy 208.28 134.62) (xy 214.63 134.62)
+		)
+		(stroke
+			(width 0)
+			(type default)
+		)
+	)
+	(wire
+		(pts
 			(xy 78.74 49.53) (xy 82.55 49.53)
 		)
@@
 	(wire
 		(pts
+			(xy 234.95 134.62) (xy 241.3 134.62)
+		)
+		(stroke
+			(width 0)
+			(type default)
+		)
+	)
+	(wire
+		(pts
 			(xy 50.8 34.29) (xy 50.8 38.1)
 		)
@@
 	(wire
 		(pts
-			(xy 54.61 143.51) (xy 55.88 143.51)
+			(xy 49.53 143.51) (xy 55.88 143.51)
 		)
 		(stroke
@@
 	(wire
 		(pts
-			(xy 208.28 134.62) (xy 214.63 134.62)
+			(xy 102.87 62.23) (xy 104.14 62.23)
 		)
 		(stroke
@@
 	(wire
 		(pts
-			(xy 102.87 62.23) (xy 104.14 62.23)
+			(xy 60.96 46.99) (xy 71.12 46.99)
 		)
 		(stroke
@@
 	(wire
 		(pts
-			(xy 60.96 46.99) (xy 71.12 46.99)
+			(xy 185.42 54.61) (xy 201.93 54.61)
 		)
 		(stroke
@@
 	(wire
 		(pts
-			(xy 185.42 54.61) (xy 201.93 54.61)
+			(xy 85.09 129.54) (xy 91.44 129.54)
 		)
 		(stroke
@@
 	(wire
 		(pts
-			(xy 85.09 129.54) (xy 91.44 129.54)
+			(xy 115.57 43.18) (xy 115.57 46.99)
 		)
 		(stroke
@@
 	(wire
 		(pts
-			(xy 115.57 43.18) (xy 115.57 46.99)
+			(xy 236.22 137.16) (xy 236.22 139.7)
 		)
 		(stroke
@@
 	(wire
 		(pts
-			(xy 236.22 137.16) (xy 236.22 139.7)
+			(xy 104.14 59.69) (xy 104.14 62.23)
 		)
 		(stroke
@@
 	(wire
 		(pts
-			(xy 104.14 59.69) (xy 104.14 62.23)
+			(xy 97.79 148.59) (xy 86.36 148.59)
 		)
 		(stroke
@@
 	(wire
 		(pts
-			(xy 234.95 134.62) (xy 241.3 134.62)
-		)
-		(stroke
-			(width 0)
-			(type default)
-		)
-	)
-	(wire
-		(pts
 			(xy 85.09 129.54) (xy 85.09 128.27)
 		)
@@
 	(wire
 		(pts
-			(xy 86.36 148.59) (xy 97.79 148.59)
-		)
-		(stroke
-			(width 0)
-			(type default)
-		)
-	)
-	(wire
-		(pts
 			(xy 50.8 110.49) (xy 50.8 111.76)
 		)
@@
 		)
 	)
-	(label "VISOOUT"
+	(label "+3V3_ISO_CAN"
 		(at 99.06 121.92 180)
 		(effects
@@
 	(hierarchical_label "CAN0_DOUT1"
 		(shape input)
-		(at 54.61 140.97 180)
+		(at 49.53 140.97 180)
 		(effects
 			(font
@@
 	(hierarchical_label "CAN0_DIN1"
 		(shape output)
-		(at 54.61 143.51 180)
+		(at 49.53 143.51 180)
 		(effects
 			(font
@@
 	(hierarchical_label "GPIOOUT"
 		(shape bidirectional)
-		(at 54.61 148.59 180)
+		(at 49.53 148.59 180)
 		(effects
 			(font
@@
 			)
 		)
-		(property "Value" "+3V3_ISO_SPI"
+		(property "Value" "+3V3_ISO_CAN"
 			(at 112.014 111.76 0)
 			(show_name no)
@@
 		(in_pos_files yes)
 		(dnp no)
-		(fields_autoplaced yes)
 		(property "Reference" "#PWR08"
 			(at 43.18 139.7 0)
@@
 		)
 		(property "Value" "GND"
-			(at 43.18 138.43 0)
+			(at 43.18 137.16 0)
 			(show_name no)
 			(do_not_autoplace no)
@@
 			)
 		)
-		(property "Value" "GND_OUT"
+		(property "Value" "GND_ISO"
 			(at 244.094 123.952 0)
 			(show_name no)
@@
 			)
 		)
-		(property "Value" "GND_OUT"
+		(property "Value" "GND_ISO"
 			(at 223.774 49.53 0)
 			(hide yes)

Commit message: Fikset en god del småting i schematic
GPIO IN og OUT var flippet.
Mange små utsene ting.
La til Vortex Logo
Other:
- company: (none) -> Vortex NTNU
- title: (none) -> ORIN-BOB
Changed lines of the file:
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@@
 	(generator_version "10.0")
 	(paper "A4")
+	(title_block
+		(title "ORIN-BOB")
+		(date "2026-10-12")
+		(rev "1.0")
+		(company "Vortex NTNU")
+		(comment 1 "Yamn Sultan Salim")
+	)
 	(text "I2C-config\n"
 		(exclude_from_sim no)
@@
 	)
 	(hierarchical_label "CS"
-		(shape bidirectional)
+		(shape output)
 		(at 107.95 49.53 0)
 		(effects
@@
 	)
 	(hierarchical_label "SPI1_CS0_N1"
-		(shape bidirectional)
+		(shape input)
 		(at 78.74 49.53 180)
 		(effects
@@
 	)
 	(hierarchical_label "SPI1_SCK1"
-		(shape bidirectional)
+		(shape input)
 		(at 78.74 52.07 180)
 		(effects
@@
 	)
 	(hierarchical_label "GPIOIN_ISO"
+		(shape input)
+		(at 241.3 134.62 0)
+		(effects
+			(font
+				(size 1.27 1.27)
+			)
+			(justify left)
+		)
+	)
+	(hierarchical_label "SCLK"
 		(shape output)
-		(at 241.3 134.62 0)
+		(at 107.95 52.07 0)
 		(effects
 			(font
@@
 		)
 	)
-	(hierarchical_label "SCLK"
-		(shape bidirectional)
-		(at 107.95 52.07 0)
-		(effects
-			(font
-				(size 1.27 1.27)
-			)
-			(justify left)
-		)
-	)
 	(hierarchical_label "SCL"
-		(shape bidirectional)
+		(shape output)
 		(at 247.65 54.61 0)
 		(effects

Commit message: Finished: Orin-BoB
Connections:
- net GPIOOUT: now also U3.3 (INA); no longer U6.9 (AUXIN)
- net GPIOOUT_ISO: now also U3.14 (OUTA); no longer U6.17 (AUXOUT)
- net PWM: now also U6.17 (AUXOUT); no longer U3.14 (OUTA)
- net PWM01: now also U6.9 (AUXIN); no longer U3.3 (INA)
