File: orin-bob/orin-bob.kicad_pcb (KiCad board)
At the start: 4 copper layers, 27 parts, among them IC1 TCAN3414DR, J1 613040243121, J2 62501021621, U2 SOIC-8NB_18032011, U3 18024215401H, U4 18024215401H, U5 18024115401H

Commit message: Almost done schematic & PCB
Parts:
- removed C11, C12, C13, C14, C15: 10uF, Capacitor_SMD:C_0201_0603Metric
- removed IC1: TCAN3414DR, Samacsys:SOIC127P600X175-8N
- removed R5: 120, Resistor_SMD:R_0603_1608Metric
- removed U4: 18024215401H, 18024215401H:U_Wurth_WPME-CDIP_SOIC-16WB
- added ?: , , F.Cu at (189.5, 120.5)
- added C22: 0.01uF, Capacitor_SMD:C_0603_1608Metric_Pad1.08x0.95mm_HandSolder, B.Cu at (151.9, 107.0)
- added C23: 0.1uF, Capacitor_SMD:C_0603_1608Metric_Pad1.08x0.95mm_HandSolder, B.Cu at (147.5, 107.0)
- added C24: 0.01uF, Capacitor_SMD:C_0603_1608Metric_Pad1.08x0.95mm_HandSolder, B.Cu at (150.2, 93.0)
- added C25: 0.1uF, Capacitor_SMD:C_0603_1608Metric_Pad1.08x0.95mm_HandSolder, B.Cu at (150.2, 92.0)
- added C26: 10uF, Capacitor_SMD:C_0603_1608Metric_Pad1.08x0.95mm_HandSolder, B.Cu at (149.5, 108.0)
- added C27: 0.22uF, Capacitor_SMD:C_0603_1608Metric_Pad1.08x0.95mm_HandSolder, B.Cu at (144.0, 107.0)
- added C28: 0.1uF, Capacitor_SMD:C_0603_1608Metric_Pad1.08x0.95mm_HandSolder, B.Cu at (148.2, 93.0)
- added C29: 10uF, Capacitor_SMD:C_0603_1608Metric_Pad1.08x0.95mm_HandSolder, B.Cu at (148.2, 92.0)
- added FB1: BLM15HD182SN1D, BLM15HD182SN1D:IND_BLM15_0402_MUR-M, B.Cu at (149.8, 111.5)
- added FB2: BLM15HD182SN1D, BLM15HD182SN1D:IND_BLM15_0402_MUR-M, B.Cu at (145.8, 109.0)
- added R6: 120, Resistor_SMD:R_0603_1608Metric_Pad0.98x0.95mm_HandSolder, B.Cu at (153.6, 106.5)
- added REF**: MountingHole_2.1mm, MountingHole:MountingHole_2.1mm, F.Cu at (140.5, 120.5)
- added U6: ADM3057ExRW, Package_SO:SOIC-20W_7.5x12.8mm_P1.27mm, F.Cu at (146.7, 97.4)
- C1, C16, C17, C18, C19, C2, C3, C4, C5, C6: footprint Capacitor_SMD:C_0201_0603Metric -> Capacitor_SMD:C_0603_1608Metric_Pad1.08x0.95mm_HandSolder; moved to B.Cu
- J1: moved to B.Cu
- R1, R2, R3, R4: footprint Resistor_SMD:R_0603_1608Metric -> Resistor_SMD:R_0603_1608Metric_Pad0.98x0.95mm_HandSolder; moved to B.Cu
- moved R2 74.5 mm to (189.6, 93.8)
- moved R1 74.5 mm to (186.4, 93.8)
- moved C3 73.6 mm to (184.4, 95.7)
- moved C4 72.0 mm to (184.3, 101.8), turned to 90 degrees
- moved R3 72.0 mm to (189.6, 103.5)
- moved R4 72.0 mm to (186.5, 103.5)
- moved U2 71.9 mm to (187.0, 97.5), turned to -90 degrees
- moved C19 54.2 mm to (178.5, 105.8)
- moved J1 51.5 mm to (165.2, 84.4), turned to 180 degrees
- moved C16 49.3 mm to (166.8, 93.8)
- moved U3 49.0 mm to (175.9, 97.5), turned to -90 degrees
- moved C17 48.5 mm to (166.8, 94.8)
- moved C18 47.8 mm to (166.8, 95.8)
- moved J2 42.4 mm to (166.5, 116.3), turned to 180 degrees
- moved U5 23.8 mm to (162.0, 97.4), turned to 180 degrees
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Other:
- board outline added: 54 x 49 mm

Commit message: Updated bob pcb
Parts:
- removed J2: 62501021621, 61201021621:61201021621
- added J10: 653106131822, Wurth_WR-WTB:J_Wurth_WR-WTB_653106131822, F.Cu at (156.5, 120.1)
- added J6: 653104131822, Wurth_WR-WTB:J_Wurth_WR-WTB_653104131822, F.Cu at (189.1, 111.1)
- added J8: 653105131822, Wurth_WR-WTB:J_Wurth_WR-WTB_653105131822, F.Cu at (140.9, 111.8)
- added J9: 653106131822, Wurth_WR-WTB:J_Wurth_WR-WTB_653106131822, F.Cu at (174.2, 120.1)
- R6: moved to F.Cu
- U2: value SOIC-8NB_18032011 -> 18032011
- moved FB1 11.2 mm to (147.2, 100.6), turned to 90 degrees
- moved FB2 11.0 mm to (147.2, 98.1), turned to 0 degrees
- moved R6 9.63 mm to (144.2, 104.6), turned to 180 degrees
- moved C26 7.43 mm to (148.8, 100.6), turned to 90 degrees
- moved C23 7.32 mm to (151.0, 100.6), turned to -90 degrees
- moved C27 6.61 mm to (145.7, 100.6), turned to -90 degrees
- moved C22 6.44 mm to (152.6, 100.6), turned to -90 degrees
- moved C19 5.56 mm to (179.6, 100.4), turned to 180 degrees
- moved C3 4.65 mm to (189.0, 95.0)
- moved C2 4.36 mm to (165.8, 101.8), turned to 90 degrees
- moved R2 3.79 mm to (186.0, 95.0), turned to 90 degrees
- moved C24 3.78 mm to (146.6, 94.2), turned to 90 degrees
- moved C28 3.62 mm to (151.6, 94.2), turned to 90 degrees
- moved R3 3.50 mm to (188.4, 100.2), turned to -90 degrees
- moved R4 3.31 mm to (186.8, 100.2), turned to -90 degrees
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Connections:
- C1 pad 1: /digital_isolator/3V3 -> +3V3
- C16 pad 1: /digital_isolator/3V3 -> +3V3
- C17 pad 1: /digital_isolator/3V3 -> +3V3
- C18 pad 1: /digital_isolator/3V3 -> +3V3
- C19 pad 1: /digital_isolator/3V3_ISO -> +3V3_ISO_UART
- C19 pad 2: GND_OUT -> GND_ISO
- C2 pad 1: /digital_isolator/3V3_ISO -> +3V3_ISO_SPI
- C2 pad 2: GND_OUT -> GND_ISO
- C22 pad 2: Net-(U6-VISOIN) -> +3V3_ISO_CAN
- C23 pad 2: Net-(U6-VISOIN) -> +3V3_ISO_CAN
- C24 pad 2: /digital_isolator/5V -> +3V3
- C25 pad 2: /digital_isolator/5V -> +3V3
- C26 pad 2: /digital_isolator/5V_ISO -> +3V3_ISO_CAN
- C27 pad 2: Net-(U6-VISOIN) -> +3V3_ISO_CAN
- C28 pad 2: /digital_isolator/5V -> +5V
- C29 pad 2: /digital_isolator/5V -> +5V
- C3 pad 1: /digital_isolator/3V3 -> +3V3
- C4 pad 1: /digital_isolator/3V3_ISO -> +3V3_ISO_SPI
- C4 pad 2: GND_OUT -> GND_ISO
- C5 pad 1: /digital_isolator/3V3 -> +3V3
- C6 pad 1: /digital_isolator/3V3 -> +3V3
- FB1 pad 1: Net-(U6-VISOIN) -> +3V3_ISO_CAN
- FB1 pad 2: /digital_isolator/5V_ISO -> +3V3_ISO_CAN
- J1 pad 1: /digital_isolator/3V3 -> +3V3
- J1 pad 12: unconnected-(J1-Pad12) -> /digital_isolator/GPIOIN
- J1 pad 13: unconnected-(J1-Pad13) -> /digital_isolator/PWM01
- J1 pad 17: /digital_isolator/3V3 -> +3V3
- J1 pad 2: /orin-connector/5V -> +5V
- J1 pad 33: unconnected-(J1-Pad33) -> /digital_isolator/GPIOOUT
- J1 pad 4: /orin-connector/5V -> +5V
- R1 pad 1: /digital_isolator/3V3 -> +3V3
- R2 pad 1: /digital_isolator/3V3 -> +3V3
- R3 pad 1: /digital_isolator/3V3_ISO -> +3V3_ISO_SPI
- R4 pad 1: /digital_isolator/3V3_ISO -> +3V3_ISO_SPI
- U2 pad 1: /digital_isolator/3V3 -> +3V3
- U2 pad 8: /digital_isolator/3V3_ISO -> +3V3_ISO_SPI
- U3 pad 1: /digital_isolator/3V3 -> +3V3
- U3 pad 11: unconnected-(U3-IND-Pad11) -> /Connectors/GPIOOUT_ISO
- U3 pad 12: /Connectors/UART1_RX1 -> /Connectors/UART1_RX
- U3 pad 14: unconnected-(U3-OUTA-Pad14) -> /Connectors/PWM
- U3 pad 15: GND_OUT -> GND_ISO
- U3 pad 16: /digital_isolator/3V3_ISO -> +3V3_ISO_UART
- U3 pad 3: unconnected-(U3-INA-Pad3) -> /digital_isolator/PWM01
- U3 pad 6: unconnected-(U3-OUTD-Pad6) -> /digital_isolator/GPIOIN
- U5 pad 1: /digital_isolator/3V3 -> +3V3
- U5 pad 15: GND_OUT -> GND_ISO
- U5 pad 16: /digital_isolator/3V3_ISO -> +3V3_ISO_SPI
- U6 pad 16: Net-(U6-VISOIN) -> +3V3_ISO_CAN
- U6 pad 17: unconnected-(U6-AUXOUT-Pad17) -> /Connectors/GPIOIN_ISO
- U6 pad 19: Net-(U6-VISOIN) -> +3V3_ISO_CAN
- U6 pad 3: /digital_isolator/5V -> +5V
- U6 pad 4: /digital_isolator/5V -> +3V3
- U6 pad 5: /digital_isolator/CAN0_DOUT1 -> /digital_isolator/CAN0_DIN1
- U6 pad 7: /digital_isolator/CAN0_DIN1 -> /digital_isolator/CAN0_DOUT1
- U6 pad 9: GND -> /digital_isolator/GPIOOUT
Routing:
- net /digital_isolator/SPI1_CS0_N1: track 0.00 -> 23.4 mm
- net /Connectors/SCL: track 0.00 -> 19.5 mm, vias 0 -> 1
- net /digital_isolator/SPI1_SCK1: track 0.00 -> 18.8 mm, vias 0 -> 2
- net /digital_isolator/UART1_TX1: track 0.00 -> 18.8 mm
- net /digital_isolator/PWM01: track 0.00 -> 18.6 mm, vias 0 -> 2
- net /Connectors/SDA: track 0.00 -> 18.4 mm, vias 0 -> 1
- net /digital_isolator/UART1_RX1: track 0.00 -> 18.2 mm
- net /digital_isolator/GPIOIN: track 0.00 -> 17.7 mm
- net /Connectors/CS: track 0.00 -> 17.5 mm
- net /Connectors/SCLK: track 0.00 -> 17.4 mm
- net /Connectors/SDO: track 0.00 -> 17.4 mm
- net /Connectors/SDI: track 0.00 -> 17.4 mm
- net /digital_isolator/I2C5_CLK1: track 0.00 -> 16.8 mm
- net /digital_isolator/CAN0_DIN1: track 0.00 -> 16.7 mm
- net /digital_isolator/GPIOOUT: track 0.00 -> 16.7 mm
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- added copper zone on B.Cu, net +3V3
- added copper zone on F.Cu, net +3V3
- added copper zone on In2.Cu, net +3V3
- added copper zone on B.Cu, net +3V3_ISO_CAN
- added copper zone on F.Cu, net +3V3_ISO_CAN
- added copper zone on In2.Cu, net +3V3_ISO_CAN
- added copper zone on B.Cu, net +3V3_ISO_SPI
- added copper zone on F.Cu, net +3V3_ISO_SPI
- added copper zone on In2.Cu, net +3V3_ISO_SPI
- added copper zone on B.Cu, net +3V3_ISO_UART
- added copper zone on F.Cu, net +3V3_ISO_UART
- added copper zone on In2.Cu, net +3V3_ISO_UART
- added copper zone on B.Cu, net +5V
- added copper zone on F.Cu, net +5V
- added copper zone on In2.Cu, net +5V
- added copper zone on B.Cu, net GND
- added copper zone on F.Cu, net GND
- added copper zone on In1.Cu, net GND
- added copper zone on B.Cu, net GND_ISO
- added copper zone on F.Cu, net GND_ISO
- added copper zone on In1.Cu, net GND_ISO
Other:
- board text added: "CAN"
- board text added: "I2C"
- board text added: "SPI"
- board text added: "UART"
- board text added: "Y.S"

Commit message: Finished: Orin-BoB
Parts:
- removed J8: 653105131822, Wurth_WR-WTB:J_Wurth_WR-WTB_653105131822
- added J7: 653104131822, Wurth_WR-WTB:J_Wurth_WR-WTB_653104131822, F.Cu at (141.4, 111.1)
Connections:
- net /digital_isolator/CAN0_DIN1 renamed /Digital-isolator/CAN0_DIN1
- net /digital_isolator/CAN0_DOUT1 renamed /Digital-isolator/CAN0_DOUT1
- net /digital_isolator/GPIOIN renamed /Digital-isolator/GPIOIN
- net /digital_isolator/I2C5_CLK1 renamed /Digital-isolator/I2C5_CLK1
- net /digital_isolator/I2C5_DAT1 renamed /Digital-isolator/I2C5_DAT1
- net /digital_isolator/SPI1_CS0_N1 renamed /Digital-isolator/SPI1_CS0_N1
- net /digital_isolator/SPI1_MISO1 renamed /Digital-isolator/SPI1_MISO1
- net /digital_isolator/SPI1_MOSI1 renamed /Digital-isolator/SPI1_MOSI1
- net /digital_isolator/SPI1_SCK1 renamed /Digital-isolator/SPI1_SCK1
- net /digital_isolator/UART1_RX1 renamed /Digital-isolator/UART1_RX1
- net /digital_isolator/UART1_TX1 renamed /Digital-isolator/UART1_TX1
- net /orin-connector/SPI1_CS1_N1 renamed /ORIN-connector/SPI1_CS1_N1
- J1 pad 13: /digital_isolator/PWM01 -> /Digital-isolator/PWM01
- J1 pad 33: /digital_isolator/GPIOOUT -> /Digital-isolator/GPIOOUT
- J9 pad 2: /Connectors/GPIOOUT_ISO -> /Connectors/GPIOIN_ISO
- J9 pad 5: /Connectors/PWM -> /Connectors/GPIOOUT_ISO
- U3 pad 11: /Connectors/GPIOOUT_ISO -> /Connectors/GPIOIN_ISO
- U3 pad 14: /Connectors/PWM -> /Connectors/GPIOOUT_ISO
- U3 pad 3: /digital_isolator/PWM01 -> /Digital-isolator/GPIOOUT
- U6 pad 17: /Connectors/GPIOIN_ISO -> /Connectors/PWM
- U6 pad 9: /digital_isolator/GPIOOUT -> /Digital-isolator/PWM01
Routing:
- net (no net): track 0.00 -> 35.3 mm, vias 86 -> 87
- net /digital_isolator/PWM01: track 18.6 -> 0.00 mm, vias 2 -> 0
- net /digital_isolator/GPIOOUT: track 16.7 -> 0.00 mm
- net /Connectors/PWM: track 15.8 -> 12.1 mm, vias 0 -> 2
- net GND_ISO: vias 30 -> 32
- net /Digital-isolator/GPIOOUT: vias 0 -> 1
- net +3V3_ISO_CAN: vias 6 -> 4
- removed copper zone on In2.Cu, net +3V3_ISO_CAN

Commit message: orin-interface: add ETH connector sheets and Mate-connectors footprint lib; update orin-bob
Parts:
- added R5: 50, Resistor_SMD:R_0603_1608Metric_Pad0.98x0.95mm_HandSolder, F.Cu at (153.7, 82.8)
- added R7: 50, Resistor_SMD:R_0603_1608Metric_Pad0.98x0.95mm_HandSolder, F.Cu at (144.8, 89.2)
Connections:
- J1 pad 29: /Digital-isolator/CAN0_DIN1 -> Net-(J1-Pad29)
- J1 pad 31: /Digital-isolator/CAN0_DOUT1 -> Net-(J1-Pad31)
- J9 pad 2: /Connectors/GPIOIN_ISO -> /Connectors/GPIOOUT_ISO
- J9 pad 5: /Connectors/GPIOOUT_ISO -> /Connectors/GPIOIN_ISO
Routing:
- net /Digital-isolator/CAN0_DOUT1: track 16.7 -> 2.69 mm
- net Net-(J1-Pad31): track 0.00 -> 12.7 mm
- net /Digital-isolator/CAN0_DIN1: track 16.7 -> 14.2 mm
- net Net-(J1-Pad29): track 0.00 -> 1.89 mm
