File: orin-interface/orin-interface/ETH_CAM1_CON.kicad_sch (KiCad schematic)
At the start: 1 part, among them J8 530470810

Commit message: orin-interface: PoE channels, buses, 3V3 regulator, ERC fixes
Parts:
- J8: footprint CONN08_530470810_MOL -> 530470810:CONN08_530470810_MOL
Changed lines of the file:
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@@
 			)
 		)
-		(property "Footprint" "CONN08_530470810_MOL"
+		(property "Footprint" "530470810:CONN08_530470810_MOL"
 			(at 119.38 57.15 0)
 			(hide yes)
