File: orin-interface/orin-interface/Standard_CONN.kicad_sch (KiCad schematic)
At the start: 1 part, among them J10 691378140024

Commit message: Finished: Orin-BoB
Connections:
- net PWM: now reaches J10.10
- net PWM: now also J10.22
Other:
- moved on the sheet: J10

Commit message: orin-interface: PoE channels, buses, 3V3 regulator, ERC fixes
Connections:
- no-connect marks 0 -> 14
Changed lines of the file:
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@@
 		(color 0 0 0 0)
+	)
+	(no_connect
+		(at 111.76 63.5)
+	)
+	(no_connect
+		(at 111.76 50.8)
+	)
+	(no_connect
+		(at 99.06 58.42)
+	)
+	(no_connect
+		(at 111.76 60.96)
+	)
+	(no_connect
+		(at 99.06 63.5)
+	)
+	(no_connect
+		(at 99.06 66.04)
+	)
+	(no_connect
+		(at 111.76 53.34)
+	)
+	(no_connect
+		(at 111.76 55.88)
+	)
+	(no_connect
+		(at 111.76 66.04)
+	)
+	(no_connect
+		(at 99.06 53.34)
+	)
+	(no_connect
+		(at 111.76 58.42)
+	)
+	(no_connect
+		(at 99.06 55.88)
+	)
+	(no_connect
+		(at 99.06 50.8)
+	)
+	(no_connect
+		(at 99.06 60.96)
 	)
 	(wire
