File: orin-interface/orin-interface/M_CAM_FRONT_L.kicad_sch (KiCad schematic)
At the start: 19 parts, among them T1 749022310

Commit message: Finished: Orin-BoB
Changed lines of the file:
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@@
 	(generator "eeschema")
 	(generator_version "10.0")
-	(paper "A4")
+	(paper "A5")
 	(junction
 		(at 130.81 83.82)
@@
 	)
 	(junction
+		(at 132.08 52.07)
+		(diameter 0)
+		(color 0 0 0 0)
+	)
+	(junction
 		(at 90.17 83.82)
 		(diameter 0)
@@
 		(color 0 0 0 0)
 	)
-	(junction
-		(at 134.62 52.07)
-		(diameter 0)
-		(color 0 0 0 0)
-	)
 	(bus_entry
 		(at 59.69 48.26)
@@
 	(wire
 		(pts
-			(xy 135.89 36.83) (xy 134.62 36.83)
-		)
-		(stroke
-			(width 0)
-			(type default)
-		)
-	)
-	(wire
-		(pts
 			(xy 124.46 69.85) (xy 152.4 69.85)
 		)
@@
 	(wire
 		(pts
-			(xy 134.62 52.07) (xy 135.89 52.07)
+			(xy 132.08 52.07) (xy 135.89 52.07)
 		)
 		(stroke
@@
 	(wire
 		(pts
+			(xy 132.08 36.83) (xy 135.89 36.83)
+		)
+		(stroke
+			(width 0)
+			(type default)
+		)
+	)
+	(wire
+		(pts
 			(xy 90.17 82.55) (xy 90.17 83.82)
 		)
@@
 	(wire
 		(pts
-			(xy 124.46 52.07) (xy 134.62 52.07)
+			(xy 124.46 52.07) (xy 132.08 52.07)
 		)
 		(stroke
@@
 	(wire
 		(pts
-			(xy 134.62 36.83) (xy 134.62 52.07)
-		)
-		(stroke
+			(xy 132.08 36.83) (xy 132.08 52.07)
+		)
+		(stroke

Commit message: orin-interface: PoE channels, buses, 3V3 regulator, ERC fixes
Parts:
- C18, C19, C20, C21, C26, C27, C28, C29, C38, C39: footprint (none) -> Capacitor_SMD:C_0603_1608Metric_Pad1.08x0.95mm_HandSolder
- R29, R33, R37, R41, R45, R46, R47, R48: footprint (none) -> Resistor_SMD:R_0603_1608Metric_Pad0.98x0.95mm_HandSolder
Changed lines of the file:
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@@
 			)
 		)
-		(property "Footprint" ""
+		(property "Footprint" "Resistor_SMD:R_0603_1608Metric_Pad0.98x0.95mm_HandSolder"
 			(at 130.81 74.93 0)
 			(hide yes)
@@
 			)
 		)
-		(property "Footprint" ""
+		(property "Footprint" "Capacitor_SMD:C_0603_1608Metric_Pad1.08x0.95mm_HandSolder"
 			(at 95.25 80.01 0)
 			(hide yes)
@@
 			)
 		)
-		(property "Footprint" ""
+		(property "Footprint" "Resistor_SMD:R_0603_1608Metric_Pad0.98x0.95mm_HandSolder"
 			(at 140.97 74.93 0)
 			(hide yes)
@@
 			)
 		)
-		(property "Footprint" ""
+		(property "Footprint" "Resistor_SMD:R_0603_1608Metric_Pad0.98x0.95mm_HandSolder"
 			(at 90.17 74.93 0)
 			(hide yes)
@@
 			)
 		)
-		(property "Footprint" ""
+		(property "Footprint" "Capacitor_SMD:C_0603_1608Metric_Pad1.08x0.95mm_HandSolder"
 			(at 125.73 80.01 0)
 			(hide yes)
@@
 			)
 		)
-		(property "Footprint" ""
+		(property "Footprint" "Resistor_SMD:R_0603_1608Metric_Pad0.98x0.95mm_HandSolder"
 			(at 135.89 74.93 0)
 			(hide yes)
@@
 			)
 		)
-		(property "Footprint" ""
+		(property "Footprint" "Capacitor_SMD:C_0603_1608Metric_Pad1.08x0.95mm_HandSolder"
 			(at 85.09 80.01 0)
 			(hide yes)
@@
 			)
 		)
-		(property "Footprint" ""
+		(property "Footprint" "Capacitor_SMD:C_0603_1608Metric_Pad1.08x0.95mm_HandSolder"
 			(at 100.33 80.01 0)
 			(hide yes)
@@
 			)
 		)
-		(property "Footprint" ""
+		(property "Footprint" "Capacitor_SMD:C_0603_1608Metric_Pad1.08x0.95mm_HandSolder"
 			(at 90.17 80.01 0)
 			(hide yes)
@@
 			)
 		)
-		(property "Footprint" ""
+		(property "Footprint" "Resistor_SMD:R_0603_1608Metric_Pad0.98x0.95mm_HandSolder"
 			(at 125.73 74.93 0)
 			(hide yes)
@@
 			)
 		)
-		(property "Footprint" ""
+		(property "Footprint" "Resistor_SMD:R_0603_1608Metric_Pad0.98x0.95mm_HandSolder"
 			(at 85.09 74.93 0)
 			(hide yes)
@@
 			)
 		)
-		(property "Footprint" ""
+		(property "Footprint" "Resistor_SMD:R_0603_1608Metric_Pad0.98x0.95mm_HandSolder"
 			(at 95.25 74.93 0)
 			(hide yes)
@@
 			)
 		)
-		(property "Footprint" ""
+		(property "Footprint" "Capacitor_SMD:C_0603_1608Metric_Pad1.08x0.95mm_HandSolder"
 			(at 133.35 88.9 0)
 			(hide yes)
@@
 			)
 		)
-		(property "Footprint" ""
+		(property "Footprint" "Capacitor_SMD:C_0603_1608Metric_Pad1.08x0.95mm_HandSolder"
 			(at 130.81 80.01 0)
 			(hide yes)
@@
 			)
 		)
-		(property "Footprint" ""
+		(property "Footprint" "Capacitor_SMD:C_0603_1608Metric_Pad1.08x0.95mm_HandSolder"
 			(at 92.71 88.9 0)
 			(hide yes)
@@
 			)
 		)
-		(property "Footprint" ""
+		(property "Footprint" "Resistor_SMD:R_0603_1608Metric_Pad0.98x0.95mm_HandSolder"
 			(at 100.33 74.93 0)
 			(hide yes)
@@
 			)
 		)
-		(property "Footprint" ""
+		(property "Footprint" "Capacitor_SMD:C_0603_1608Metric_Pad1.08x0.95mm_HandSolder"
 			(at 135.89 80.01 0)
 			(hide yes)
@@
 			)
 		)
-		(property "Footprint" ""
+		(property "Footprint" "Capacitor_SMD:C_0603_1608Metric_Pad1.08x0.95mm_HandSolder"
 			(at 140.97 80.01 0)
 			(hide yes)

Commit message: orin-interface: add ETH connector sheets and Mate-connectors footprint lib; update orin-bob
Connections:
- net X1+ renamed ETH.X1+
- net X1- renamed ETH.X1-
- net X2+ renamed ETH.X2+
- net X2- renamed ETH.X2-
- net X3+ renamed ETH.X3+
- net X3- renamed ETH.X3-
- net X4+ renamed ETH.X4+
- net X4- renamed ETH.X4-
Changed lines of the file:
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@@
 		)
 	)
-	(label "X4+"
-		(at 148.59 64.77 0)
+	(label "ETH.X4+"
+		(at 143.51 64.77 0)
 		(effects
 			(font
@@
 		)
 	)
-	(label "X2+"
-		(at 148.59 49.53 0)
+	(label "ETH.X2+"
+		(at 143.51 49.53 0)
 		(effects
 			(font
@@
 		)
 	)
-	(label "X1+"
-		(at 148.59 41.91 0)
+	(label "ETH.X1+"
+		(at 143.51 41.91 0)
 		(effects
 			(font
@@
 		)
 	)
-	(label "X3-"
-		(at 148.59 62.23 0)
+	(label "ETH.X3-"
+		(at 143.51 62.23 0)
 		(effects
 			(font
@@
 		)
 	)
-	(label "X1-"
-		(at 148.59 46.99 0)
+	(label "ETH.X1-"
+		(at 143.51 46.99 0)
 		(effects
 			(font
@@
 		)
 	)
-	(label "X4-"
-		(at 148.59 69.85 0)
+	(label "ETH.X4-"
+		(at 143.51 69.85 0)
 		(effects
 			(font
@@
 		)
 	)
-	(label "X3+"
-		(at 148.59 57.15 0)
+	(label "ETH.X3+"
+		(at 143.51 57.15 0)
 		(effects
 			(font
@@
 		)
 	)
-	(label "X2-"
-		(at 148.59 54.61 0)
+	(label "ETH.X2-"
+		(at 143.51 54.61 0)
 		(effects
 			(font
