File: orin-interface/orin-interface/M_CAM_FRONT_R.kicad_sch (KiCad schematic)
At the start: 19 parts, among them T4 749022310

Commit message: orin-interface: PoE channels, buses, 3V3 regulator, ERC fixes
Parts:
- C30, C31, C32, C33, C34, C35, C36, C37, C40, C41: footprint (none) -> Capacitor_SMD:C_0603_1608Metric_Pad1.08x0.95mm_HandSolder
- R30, R34, R38, R42, R49, R50, R51, R52: footprint (none) -> Resistor_SMD:R_0603_1608Metric_Pad0.98x0.95mm_HandSolder
Changed lines of the file:
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@@
 			)
 		)
-		(property "Footprint" ""
+		(property "Footprint" "Resistor_SMD:R_0603_1608Metric_Pad0.98x0.95mm_HandSolder"
 			(at 142.24 78.74 0)
 			(hide yes)
@@
 			)
 		)
-		(property "Footprint" ""
+		(property "Footprint" "Capacitor_SMD:C_0603_1608Metric_Pad1.08x0.95mm_HandSolder"
 			(at 85.09 84.7388 0)
 			(hide yes)
@@
 			)
 		)
-		(property "Footprint" ""
+		(property "Footprint" "Capacitor_SMD:C_0603_1608Metric_Pad1.08x0.95mm_HandSolder"
 			(at 90.17 84.7388 0)
 			(hide yes)
@@
 			)
 		)
-		(property "Footprint" ""
+		(property "Footprint" "Capacitor_SMD:C_0603_1608Metric_Pad1.08x0.95mm_HandSolder"
 			(at 132.08 85.09 0)
 			(hide yes)
@@
 			)
 		)
-		(property "Footprint" ""
+		(property "Footprint" "Resistor_SMD:R_0603_1608Metric_Pad0.98x0.95mm_HandSolder"
 			(at 132.08 78.74 0)
 			(hide yes)
@@
 			)
 		)
-		(property "Footprint" ""
+		(property "Footprint" "Capacitor_SMD:C_0603_1608Metric_Pad1.08x0.95mm_HandSolder"
 			(at 134.62 92.71 0)
 			(hide yes)
@@
 			)
 		)
-		(property "Footprint" ""
+		(property "Footprint" "Capacitor_SMD:C_0603_1608Metric_Pad1.08x0.95mm_HandSolder"
 			(at 95.25 84.7388 0)
 			(hide yes)
@@
 			)
 		)
-		(property "Footprint" ""
+		(property "Footprint" "Capacitor_SMD:C_0603_1608Metric_Pad1.08x0.95mm_HandSolder"
 			(at 127 85.09 0)
 			(hide yes)
@@
 			)
 		)
-		(property "Footprint" ""
+		(property "Footprint" "Capacitor_SMD:C_0603_1608Metric_Pad1.08x0.95mm_HandSolder"
 			(at 92.71 92.71 0)
 			(hide yes)
@@
 			)
 		)
-		(property "Footprint" ""
+		(property "Footprint" "Resistor_SMD:R_0603_1608Metric_Pad0.98x0.95mm_HandSolder"
 			(at 127 78.74 0)
 			(hide yes)
@@
 			)
 		)
-		(property "Footprint" ""
+		(property "Footprint" "Resistor_SMD:R_0603_1608Metric_Pad0.98x0.95mm_HandSolder"
 			(at 137.16 78.74 0)
 			(hide yes)
@@
 			)
 		)
-		(property "Footprint" ""
+		(property "Footprint" "Capacitor_SMD:C_0603_1608Metric_Pad1.08x0.95mm_HandSolder"
 			(at 142.24 85.09 0)
 			(hide yes)
@@
 			)
 		)
-		(property "Footprint" ""
+		(property "Footprint" "Capacitor_SMD:C_0603_1608Metric_Pad1.08x0.95mm_HandSolder"
 			(at 100.33 84.7388 0)
 			(hide yes)
@@
 			)
 		)
-		(property "Footprint" ""
+		(property "Footprint" "Resistor_SMD:R_0603_1608Metric_Pad0.98x0.95mm_HandSolder"
 			(at 85.09 78.74 0)
 			(hide yes)
@@
 			)
 		)
-		(property "Footprint" ""
+		(property "Footprint" "Resistor_SMD:R_0603_1608Metric_Pad0.98x0.95mm_HandSolder"
 			(at 90.17 78.74 0)
 			(hide yes)
@@
 			)
 		)
-		(property "Footprint" ""
+		(property "Footprint" "Resistor_SMD:R_0603_1608Metric_Pad0.98x0.95mm_HandSolder"
 			(at 95.25 78.74 0)
 			(hide yes)
@@
 			)
 		)
-		(property "Footprint" ""
+		(property "Footprint" "Capacitor_SMD:C_0603_1608Metric_Pad1.08x0.95mm_HandSolder"
 			(at 137.16 85.09 0)
 			(hide yes)
@@
 			)
 		)
-		(property "Footprint" ""
+		(property "Footprint" "Resistor_SMD:R_0603_1608Metric_Pad0.98x0.95mm_HandSolder"
 			(at 100.33 78.74 0)
 			(hide yes)

Commit message: orin-interface: add ETH connector sheets and Mate-connectors footprint lib; update orin-bob
Connections:
- net ETH.D3+: no longer T4.9 (D3-)
- net X1+ renamed ETH.X1+
- net X1- renamed ETH.X1-
- net X2+ renamed ETH.X2+
- net X2- renamed ETH.X2-
- net X3+ renamed ETH.X3+
- net X3- renamed ETH.X3-
- net X4+ renamed ETH.X4+
- net X4- renamed ETH.X4-
- new net ETH.D3-: T4.9 (D3-)
Changed lines of the file:
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@@
 		)
 	)
-	(label "X3-"
+	(label "ETH.X3-"
 		(at 144.78 66.04 0)
 		(effects
@@
 		)
 	)
-	(label "X2-"
+	(label "ETH.X2-"
 		(at 144.78 58.42 0)
 		(effects
@@
 		)
 	)
-	(label "X2+"
+	(label "ETH.X2+"
 		(at 144.78 53.34 0)
 		(effects
@@
 		)
 	)
-	(label "X4+"
+	(label "ETH.X4+"
 		(at 144.78 68.58 0)
 		(effects
@@
 		)
 	)
-	(label "X3+"
+	(label "ETH.X3+"
 		(at 144.78 60.96 0)
 		(effects
@@
 		)
 	)
-	(label "X4-"
+	(label "ETH.X4-"
 		(at 144.78 73.66 0)
 		(effects
@@
 		)
 	)
-	(label "X1-"
+	(label "ETH.X1-"
 		(at 144.78 50.8 0)
 		(effects
@@
 		)
 	)
-	(label "X1+"
+	(label "ETH.X1+"
 		(at 144.78 45.72 0)
 		(effects
@@
 		)
 	)
-	(label "ETH.D3+"
+	(label "ETH.D3-"
 		(at 74.93 66.04 0)
 		(effects
