File: orin-interface/orin-interface/PoE_PD.kicad_sch (KiCad schematic)
At the start: 31 parts, among them U2 TPS23861PWR

Commit message: orin-interface: PoE channels, buses, 3V3 regulator, ERC fixes
Parts:
- C12, C13, C14, C15, C16, C17: footprint (none) -> Capacitor_SMD:C_0603_1608Metric_Pad1.08x0.95mm_HandSolder
- R10, R11, R12, R20, R21, R22, R23, R24, R25, R26, R27, R28: footprint (none) -> Resistor_SMD:R_0603_1608Metric_Pad0.98x0.95mm_HandSolder
Connections:
- net +48V: now also C14.1, C15.1, C16.1, C17.1, CR1.1, CR2.1, CR3.1, CR4.1
- net POE1_N: now also CR1.2; no longer CR1.
- net POE2_N: now also CR2.2; no longer CR2.
- net POE3_N: now also CR3.2; no longer CR3.
- net POE4_N: now also CR4.2; no longer CR4.
- net at R22.2, R27.2: now also MOSFET6.1; no longer MOSFET6.
- net at F3.1, R21.2: now also MOSFET6.5; no longer MOSFET6.
- net at U2.10 (GATE3): now also MOSFET6.4; no longer MOSFET6.
- net at F4.1, R23.2: now also MOSFET7.5; no longer MOSFET7.
- net at R20.2, R26.2: now also MOSFET5.1; no longer MOSFET5.
- net at R24.2, R28.2: now also MOSFET7.1; no longer MOSFET7.
- net at F1.1, R10.2: now also MOSFET1.5; no longer MOSFET1.
- net GATE1: now reaches U2.17 (GATE1)
- net GATE1: now also MOSFET1.4; no longer MOSFET1.
- net at R25.2: now also MOSFET1.1; no longer MOSFET1.
- net at U2.14 (GATE4): now also MOSFET7.4; no longer MOSFET7.
- net Drain2: now reaches F2.1, R12.2
- net Drain2: now also MOSFET5.5; no longer MOSFET5.
- net at U2.21 (GATE2): now also MOSFET5.4; no longer MOSFET5.
- removed net POE1_P: C14.1, CR1.
- removed net POE2_P: C15.1, CR2.
- removed net POE3_P: C16.1, CR3.
- removed net POE4: C17.1, CR4.
Other:
- moved on the sheet: R25, R26, R27, R28

Commit message: orin-interface: add ETH connector sheets and Mate-connectors footprint lib; update orin-bob
Parts:
- removed MOSFET5, MOSFET6, MOSFET7: FDMC3612, FDMC3612:MLP8_3P3X3P3_ONS, symbol FDMC3612:FDMC3612
- added MOSFET2, MOSFET3, MOSFET4: FDMC3612, FDMC3612:MLP8_3P3X3P3_ONS, symbol FDMC3612:FDMC3612
Connections:
- net Drain2: now also MOSFET2.5, MOSFET2.6, MOSFET2.7, MOSFET2.8, MOSFET2.9
- net GND: no longer R11.2
- net at R22.2, R27.2: now also MOSFET3.1, MOSFET3.2, MOSFET3.3
- net at U2.10 (GATE3): now also MOSFET3.4
- net at F3.1, R21.2: now also MOSFET3.5, MOSFET3.6, MOSFET3.7, MOSFET3.8, MOSFET3.9
- net at F4.1, R23.2: now also MOSFET4.5, MOSFET4.6, MOSFET4.7, MOSFET4.8, MOSFET4.9
- net at R20.2, R26.2: now also MOSFET2.1, MOSFET2.2, MOSFET2.3
- net at R24.2, R28.2: now also MOSFET4.1, MOSFET4.2, MOSFET4.3
- net SEN1: now reaches MOSFET1.1, R25.2
- net SEN1: now also MOSFET1.2, MOSFET1.3, R11.2
- net at F1.1, MOSFET1.5, R10.2: now also MOSFET1.6, MOSFET1.7, MOSFET1.8, MOSFET1.9
- net at U2.14 (GATE4): now also MOSFET4.4
- net at U2.21 (GATE2): now also MOSFET2.4
Other:
- moved on the sheet: R26
