File: orin-interface/orin-interface/orin-interface.kicad_pcb (KiCad board)
At the start: 2 copper layers, 120 x 136.8 mm, 32 parts, among them J1 694108301002, J10 691378140024, J13 530470810, J14 530470810, J15 530470810, J6 653104131822, J7 64600211622, J8 530470810, J9 691101810004, Q1 BSC094N06LS5ATMA1, T1 749022310, T4 749022310, T5 749022310, T6 749022310, U2 TPS23861PWR, U3 TPS259482AYWPR, U7 LT8357EMSE-PBF, U8 FSV10100V

Commit message: orin-interface: add ETH connector sheets and Mate-connectors footprint lib; update orin-bob
Parts:
- removed J1: 694108301002, 694108301002:CONN3_01002_WRE
- removed J13: 530470810, 530470810:CONN08_530470810_MOL
- removed J9: 691101810004, 691378140024-2:J_Wurth_WR-TBL_691101810004
- removed MOSFET5, MOSFET6, MOSFET7: FDMC3612, FDMC3612:MLP8_3P3X3P3_ONS
- removed the REF** at (239.2, 109.6)
- added C1: 10uF, Capacitor_SMD:C_0603_1608Metric_Pad1.08x0.95mm_HandSolder, B.Cu at (189.6, 56.4)
- added C10: 3.0nF, Capacitor_SMD:C_0603_1608Metric_Pad1.08x0.95mm_HandSolder, B.Cu at (189.5, 52.6)
- added C11: 10uF, Capacitor_SMD:C_0603_1608Metric_Pad1.08x0.95mm_HandSolder, B.Cu at (187.8, 56.4)
- added C12: 0.1uF, Capacitor_SMD:C_0603_1608Metric_Pad1.08x0.95mm_HandSolder, B.Cu at (146.4, 116.1)
- added C13: 0.1uF, Capacitor_SMD:C_0603_1608Metric_Pad1.08x0.95mm_HandSolder, B.Cu at (151.4, 116.1)
- added C14: 0.1uF, Capacitor_SMD:C_0603_1608Metric_Pad1.08x0.95mm_HandSolder, B.Cu at (154.9, 108.1)
- added C15: 0.1uF, Capacitor_SMD:C_0603_1608Metric_Pad1.08x0.95mm_HandSolder, B.Cu at (143.2, 132.5)
- added C16: 0.1uF, Capacitor_SMD:C_0603_1608Metric_Pad1.08x0.95mm_HandSolder, B.Cu at (155.1, 132.5)
- added C17: 0.1uF, Capacitor_SMD:C_0603_1608Metric_Pad1.08x0.95mm_HandSolder, B.Cu at (143.3, 108.2)
- added C18: 10nF, Capacitor_SMD:C_0603_1608Metric_Pad1.08x0.95mm_HandSolder, B.Cu at (167.8, 111.5)
- added C19: 10nF, Capacitor_SMD:C_0603_1608Metric_Pad1.08x0.95mm_HandSolder, B.Cu at (167.8, 105.9)
- added C2: 10nF, Capacitor_SMD:C_0603_1608Metric_Pad1.08x0.95mm_HandSolder, B.Cu at (188.6, 71.8)
- added C20: 10nF, Capacitor_SMD:C_0603_1608Metric_Pad1.08x0.95mm_HandSolder, B.Cu at (167.8, 113.3)
- added C21: 10nF, Capacitor_SMD:C_0603_1608Metric_Pad1.08x0.95mm_HandSolder, B.Cu at (167.8, 117.1)
- added C22: C_Small, Capacitor_SMD:C_0603_1608Metric_Pad1.08x0.95mm_HandSolder, B.Cu at (193.7, 91.0)
- added C26: 10nF, Capacitor_SMD:C_0603_1608Metric_Pad1.08x0.95mm_HandSolder, B.Cu at (172.7, 117.1)
- added C27: 10nF, Capacitor_SMD:C_0603_1608Metric_Pad1.08x0.95mm_HandSolder, B.Cu at (172.7, 115.2)
- added C28: 10nF, Capacitor_SMD:C_0603_1608Metric_Pad1.08x0.95mm_HandSolder, B.Cu at (172.7, 111.5)
- added C29: 10nF, Capacitor_SMD:C_0603_1608Metric_Pad1.08x0.95mm_HandSolder, B.Cu at (172.7, 105.9)
- added C3: 0.1uF, Capacitor_SMD:C_0603_1608Metric_Pad1.08x0.95mm_HandSolder, B.Cu at (194.2, 68.9)
- added C30: 10nF, Capacitor_SMD:C_0603_1608Metric_Pad1.08x0.95mm_HandSolder, B.Cu at (125.5, 123.8)
- added C31: 10nF, Capacitor_SMD:C_0603_1608Metric_Pad1.08x0.95mm_HandSolder, B.Cu at (125.5, 125.7)
- added C32: 10nF, Capacitor_SMD:C_0603_1608Metric_Pad1.08x0.95mm_HandSolder, B.Cu at (125.5, 131.3)
- added C33: 10nF, Capacitor_SMD:C_0603_1608Metric_Pad1.08x0.95mm_HandSolder, B.Cu at (125.5, 135.0)
- added C34: 10nF, Capacitor_SMD:C_0603_1608Metric_Pad1.08x0.95mm_HandSolder, B.Cu at (125.5, 136.9)
- added C35: 10nF, Capacitor_SMD:C_0603_1608Metric_Pad1.08x0.95mm_HandSolder, B.Cu at (130.0, 135.0)
- added C36: 10nF, Capacitor_SMD:C_0603_1608Metric_Pad1.08x0.95mm_HandSolder, B.Cu at (130.0, 129.4)
- added C37: 10nF, Capacitor_SMD:C_0603_1608Metric_Pad1.08x0.95mm_HandSolder, B.Cu at (130.0, 125.7)
- added C38: 10nF, Capacitor_SMD:C_0603_1608Metric_Pad1.08x0.95mm_HandSolder, B.Cu at (172.7, 104.0)
- added C39: 10nF, Capacitor_SMD:C_0603_1608Metric_Pad1.08x0.95mm_HandSolder, B.Cu at (167.8, 104.0)
- added C4: 2.2uF, Capacitor_SMD:C_0603_1608Metric_Pad1.08x0.95mm_HandSolder, F.Cu at (192.6, 56.1)
- added C40: 10nF, Capacitor_SMD:C_0603_1608Metric_Pad1.08x0.95mm_HandSolder, B.Cu at (130.0, 123.8)
- added C41: 10nF, Capacitor_SMD:C_0603_1608Metric_Pad1.08x0.95mm_HandSolder, B.Cu at (130.0, 136.9)
- added C42: 10nF, Capacitor_SMD:C_0603_1608Metric_Pad1.08x0.95mm_HandSolder, B.Cu at (172.7, 135.1)
- added C43: 10nF, Capacitor_SMD:C_0603_1608Metric_Pad1.08x0.95mm_HandSolder, B.Cu at (172.7, 133.1)
- added C44: 10nF, Capacitor_SMD:C_0603_1608Metric_Pad1.08x0.95mm_HandSolder, B.Cu at (172.7, 129.6)
- added C45: 10nF, Capacitor_SMD:C_0603_1608Metric_Pad1.08x0.95mm_HandSolder, B.Cu at (172.7, 124.0)
- added C46: 10nF, Capacitor_SMD:C_0603_1608Metric_Pad1.08x0.95mm_HandSolder, B.Cu at (172.7, 122.2)
- added C47: 10nF, Capacitor_SMD:C_0603_1608Metric_Pad1.08x0.95mm_HandSolder, B.Cu at (167.8, 122.2)
- added C48: 10nF, Capacitor_SMD:C_0603_1608Metric_Pad1.08x0.95mm_HandSolder, B.Cu at (167.8, 124.2)
- added C49: 10nF, Capacitor_SMD:C_0603_1608Metric_Pad1.08x0.95mm_HandSolder, B.Cu at (167.8, 133.2)
- added C5: 10uF, Capacitor_SMD:C_0603_1608Metric_Pad1.08x0.95mm_HandSolder, B.Cu at (178.1, 79.4)
- added C50: 10nF, Capacitor_SMD:C_0603_1608Metric_Pad1.08x0.95mm_HandSolder, B.Cu at (167.8, 131.4)
- added C51: 10nF, Capacitor_SMD:C_0603_1608Metric_Pad1.08x0.95mm_HandSolder, B.Cu at (167.8, 135.2)
- added C52: 10nF, Capacitor_SMD:C_0603_1608Metric_Pad1.08x0.95mm_HandSolder, B.Cu at (125.4, 105.9)
- added C53: 10nF, Capacitor_SMD:C_0603_1608Metric_Pad1.08x0.95mm_HandSolder, B.Cu at (125.4, 107.8)
- added C54: 10nF, Capacitor_SMD:C_0603_1608Metric_Pad1.08x0.95mm_HandSolder, B.Cu at (125.4, 111.5)
- added C55: 10nF, Capacitor_SMD:C_0603_1608Metric_Pad1.08x0.95mm_HandSolder, B.Cu at (125.5, 117.0)
- added C56: 10nF, Capacitor_SMD:C_0603_1608Metric_Pad1.08x0.95mm_HandSolder, B.Cu at (130.0, 117.0)
- added C57: 10nF, Capacitor_SMD:C_0603_1608Metric_Pad1.08x0.95mm_HandSolder, B.Cu at (130.0, 113.3)
- added C58: 10nF, Capacitor_SMD:C_0603_1608Metric_Pad1.08x0.95mm_HandSolder, B.Cu at (130.0, 107.8)
- added C59: 10nF, Capacitor_SMD:C_0603_1608Metric_Pad1.08x0.95mm_HandSolder, B.Cu at (130.0, 105.9)
- added C6: 10uF, Capacitor_SMD:C_0603_1608Metric_Pad1.08x0.95mm_HandSolder, B.Cu at (179.8, 79.4)
- added C60: 10nF, Capacitor_SMD:C_0603_1608Metric_Pad1.08x0.95mm_HandSolder, B.Cu at (125.5, 118.8)
- added C61: 10nF, Capacitor_SMD:C_0603_1608Metric_Pad1.08x0.95mm_HandSolder, B.Cu at (130.0, 118.8)
- added C7: 10uF, Capacitor_SMD:C_0603_1608Metric_Pad1.08x0.95mm_HandSolder, B.Cu at (181.6, 79.4)
- added C8: 10uF, Capacitor_SMD:C_0603_1608Metric_Pad1.08x0.95mm_HandSolder, F.Cu at (183.3, 45.0)
- added C9: 2.2nF, Capacitor_SMD:C_0603_1608Metric_Pad1.08x0.95mm_HandSolder, B.Cu at (189.5, 49.0)
- added D1: 0603_150060RS75000, 150060RS75000:D_Wurth_WL-SMCW-0603, F.Cu at (119.0, 49.0)
- added G***: LOGO, mate-connectors:praying-hands, F.Cu at (117.0, 56.2)
- added J11: 64600411622, Wurth_WR-WTB:J_Wurth_WR-WTB_64600411622, F.Cu at (105.6, 87.2)
- added J16: 634008138121, 615008138021:J_Wurth_WR-MJ_634008138121, F.Cu at (191.5, 129.1)
- added J17: 634008138121, 615008138021:J_Wurth_WR-MJ_634008138121, F.Cu at (107.8, 111.4)
- added J2: 615008142521, 615008138021-THT:J_Wurth_WR-MJ_615008142521, F.Cu at (168.9, 96.0)
- added J3: 615008142521, 615008138021-THT:J_Wurth_WR-MJ_615008142521, F.Cu at (136.4, 96.0)
- added J4: 615008142521, 615008138021-THT:J_Wurth_WR-MJ_615008142521, F.Cu at (152.7, 96.0)
- added J5: 615008142521, 615008138021-THT:J_Wurth_WR-MJ_615008142521, F.Cu at (120.2, 96.0)
- added L2: 15.0 uH, WE-PD:L_Wurth_WE-PD-1260P, F.Cu at (183.5, 61.5)
- added MOSFET2: FDMC3612, FDMC3612:MLP8_3P3X3P3_ONS, B.Cu at (146.3, 132.5)
- added MOSFET3: FDMC3612, FDMC3612:MLP8_3P3X3P3_ONS, B.Cu at (151.8, 132.4)
- added MOSFET4: FDMC3612, FDMC3612:MLP8_3P3X3P3_ONS, B.Cu at (146.3, 108.1)
- added R1: 1M, Resistor_SMD:R_0603_1608Metric_Pad0.98x0.95mm_HandSolder, B.Cu at (191.4, 56.4)
- added R10: 47, Resistor_SMD:R_0603_1608Metric_Pad0.98x0.95mm_HandSolder, B.Cu at (150.9, 103.5)
- added R11: 22.1, Resistor_SMD:R_0603_1608Metric_Pad0.98x0.95mm_HandSolder, B.Cu at (151.0, 112.8)
- added R12: 47, Resistor_SMD:R_0603_1608Metric_Pad0.98x0.95mm_HandSolder, B.Cu at (147.3, 136.7)
- added R13: 470k, Resistor_SMD:R_0603_1608Metric_Pad0.98x0.95mm_HandSolder, B.Cu at (183.7, 48.2)
- added R14: 31.2k, Resistor_SMD:R_0603_1608Metric_Pad0.98x0.95mm_HandSolder, B.Cu at (185.3, 48.2)
- added R15: 470k, Resistor_SMD:R_0603_1608Metric_Pad0.98x0.95mm_HandSolder, B.Cu at (182.0, 48.2)
- added R16: 45.3K, Resistor_SMD:R_0603_1608Metric_Pad0.98x0.95mm_HandSolder, B.Cu at (180.3, 48.2)
- added R18: 576, Resistor_SMD:R_0603_1608Metric_Pad0.98x0.95mm_HandSolder, B.Cu at (189.5, 50.8)
- added R19: 1k, Resistor_SMD:R_0603_1608Metric_Pad0.98x0.95mm_HandSolder, F.Cu at (115.5, 49.0)
- added R2: 107k, Resistor_SMD:R_0603_1608Metric_Pad0.98x0.95mm_HandSolder, B.Cu at (193.2, 56.4)
- added R20: 22.1, Resistor_SMD:R_0603_1608Metric_Pad0.98x0.95mm_HandSolder, B.Cu at (147.2, 128.2)
- added R21: 47, Resistor_SMD:R_0603_1608Metric_Pad0.98x0.95mm_HandSolder, B.Cu at (151.0, 128.2)
- added R22: 22.1, Resistor_SMD:R_0603_1608Metric_Pad0.98x0.95mm_HandSolder, B.Cu at (151.0, 136.7)
- added R23: 47, Resistor_SMD:R_0603_1608Metric_Pad0.98x0.95mm_HandSolder, B.Cu at (145.5, 112.8)
- added R24: 22.1, Resistor_SMD:R_0603_1608Metric_Pad0.98x0.95mm_HandSolder, B.Cu at (145.4, 103.5)
- added R25: 0.255, Resistor_SMD:R_0603_1608Metric_Pad0.98x0.95mm_HandSolder, B.Cu at (152.8, 112.8)
- added R26: 0.255, Resistor_SMD:R_0603_1608Metric_Pad0.98x0.95mm_HandSolder, B.Cu at (145.5, 128.2)
- added R27: 0.255, Resistor_SMD:R_0603_1608Metric_Pad0.98x0.95mm_HandSolder, B.Cu at (152.7, 136.7)
- added R28: 0.255, Resistor_SMD:R_0603_1608Metric_Pad0.98x0.95mm_HandSolder, B.Cu at (147.1, 103.5)
- added R29: 75, Resistor_SMD:R_0603_1608Metric_Pad0.98x0.95mm_HandSolder, B.Cu at (172.7, 107.7)
- added R3: 100k, Resistor_SMD:R_0603_1608Metric_Pad0.98x0.95mm_HandSolder, F.Cu at (194.2, 56.1)
- added R30: 75, Resistor_SMD:R_0603_1608Metric_Pad0.98x0.95mm_HandSolder, B.Cu at (125.5, 133.2)
- added R31: 75, Resistor_SMD:R_0603_1608Metric_Pad0.98x0.95mm_HandSolder, B.Cu at (172.7, 125.8)
- added R32: 75, Resistor_SMD:R_0603_1608Metric_Pad0.98x0.95mm_HandSolder, B.Cu at (125.5, 115.2)
- added R33: 75, Resistor_SMD:R_0603_1608Metric_Pad0.98x0.95mm_HandSolder, B.Cu at (172.7, 109.6)
- added R34: 75, Resistor_SMD:R_0603_1608Metric_Pad0.98x0.95mm_HandSolder, B.Cu at (125.5, 129.4)
- added R35: 75, Resistor_SMD:R_0603_1608Metric_Pad0.98x0.95mm_HandSolder, B.Cu at (172.7, 127.8)
- added R36: 75, Resistor_SMD:R_0603_1608Metric_Pad0.98x0.95mm_HandSolder, B.Cu at (125.4, 113.3)
- added R37: 75, Resistor_SMD:R_0603_1608Metric_Pad0.98x0.95mm_HandSolder, B.Cu at (172.7, 113.3)
- added R38: 75, Resistor_SMD:R_0603_1608Metric_Pad0.98x0.95mm_HandSolder, B.Cu at (125.5, 127.6)
- added R39: 75, Resistor_SMD:R_0603_1608Metric_Pad0.98x0.95mm_HandSolder, B.Cu at (172.7, 131.3)
- added R4: 10k, Resistor_SMD:R_0603_1608Metric_Pad0.98x0.95mm_HandSolder, B.Cu at (188.6, 67.9)
- added R40: 75, Resistor_SMD:R_0603_1608Metric_Pad0.98x0.95mm_HandSolder, B.Cu at (125.4, 109.6)
- added R41: 75, Resistor_SMD:R_0603_1608Metric_Pad0.98x0.95mm_HandSolder, B.Cu at (172.7, 119.0)
- added R42: 75, Resistor_SMD:R_0603_1608Metric_Pad0.98x0.95mm_HandSolder, B.Cu at (125.5, 122.0)
- added R43: 75, Resistor_SMD:R_0603_1608Metric_Pad0.98x0.95mm_HandSolder, B.Cu at (172.7, 136.9)
- added R44: 75, Resistor_SMD:R_0603_1608Metric_Pad0.98x0.95mm_HandSolder, B.Cu at (125.4, 104.0)
- added R45: 75, Resistor_SMD:R_0603_1608Metric_Pad0.98x0.95mm_HandSolder, B.Cu at (167.8, 107.7)
- added R46: 75, Resistor_SMD:R_0603_1608Metric_Pad0.98x0.95mm_HandSolder, B.Cu at (167.8, 109.6)
- added R47: 75, Resistor_SMD:R_0603_1608Metric_Pad0.98x0.95mm_HandSolder, B.Cu at (167.8, 115.2)
- added R48: 75, Resistor_SMD:R_0603_1608Metric_Pad0.98x0.95mm_HandSolder, B.Cu at (167.8, 119.0)
- added R49: 75, Resistor_SMD:R_0603_1608Metric_Pad0.98x0.95mm_HandSolder, B.Cu at (130.0, 133.2)
- added R5: 95.3k, Resistor_SMD:R_0603_1608Metric_Pad0.98x0.95mm_HandSolder, B.Cu at (196.0, 68.9)
- added R50: 75, Resistor_SMD:R_0603_1608Metric_Pad0.98x0.95mm_HandSolder, B.Cu at (130.0, 131.3)
- added R51: 75, Resistor_SMD:R_0603_1608Metric_Pad0.98x0.95mm_HandSolder, B.Cu at (130.0, 127.6)
- added R52: 75, Resistor_SMD:R_0603_1608Metric_Pad0.98x0.95mm_HandSolder, B.Cu at (130.0, 122.0)
- added R53: 75, Resistor_SMD:R_0603_1608Metric_Pad0.98x0.95mm_HandSolder, B.Cu at (167.8, 126.0)
- added R54: 75, Resistor_SMD:R_0603_1608Metric_Pad0.98x0.95mm_HandSolder, B.Cu at (167.8, 127.8)
- added R55: 75, Resistor_SMD:R_0603_1608Metric_Pad0.98x0.95mm_HandSolder, B.Cu at (167.8, 129.7)
- added R56: 75, Resistor_SMD:R_0603_1608Metric_Pad0.98x0.95mm_HandSolder, B.Cu at (167.8, 137.1)
- added R57: 75, Resistor_SMD:R_0603_1608Metric_Pad0.98x0.95mm_HandSolder, B.Cu at (130.0, 115.2)
- added R58: 75, Resistor_SMD:R_0603_1608Metric_Pad0.98x0.95mm_HandSolder, B.Cu at (130.0, 111.5)
- added R59: 75, Resistor_SMD:R_0603_1608Metric_Pad0.98x0.95mm_HandSolder, B.Cu at (130.0, 109.6)
- added R6: 5, Resistor_SMD:R_0603_1608Metric_Pad0.98x0.95mm_HandSolder, B.Cu at (195.6, 61.7)
- added R60: 75, Resistor_SMD:R_0603_1608Metric_Pad0.98x0.95mm_HandSolder, B.Cu at (130.0, 104.0)
- added R7: 10m, Resistor_SMD:R_0603_1608Metric_Pad0.98x0.95mm_HandSolder, B.Cu at (197.2, 61.7)
- added R8: 1M, Resistor_SMD:R_0603_1608Metric_Pad0.98x0.95mm_HandSolder, B.Cu at (190.6, 68.9)
- added R9: 21.5k, Resistor_SMD:R_0603_1608Metric_Pad0.98x0.95mm_HandSolder, B.Cu at (192.4, 68.9)
- added REF**: MATE_WR-TBL_691379180024, mate-connectors:MATE_WR-TBL_691379180024, F.Cu at (150.0, 66.2)
- added U1: 173950336, 173950336:U_Wurth_WPME-FDSM_17395xx36, F.Cu at (191.2, 90.0)
- F1, F2, F3, F4, MOSFET1: moved to B.Cu
- J14, J15: value 530470810 -> 634008138121; footprint 530470810:CONN08_530470810_MOL -> 615008138021:J_Wurth_WR-MJ_634008138121
- J7: footprint Connector_Wuerth:Wuerth_WR-WTB_64800211622_1x02_P1.50mm_Vertical -> Wurth_WR-WTB:J_Wurth_WR-WTB_64600211622
- J8: value 530470810 -> 694106402002; footprint 530470810:CONN08_530470810_MOL -> 694106402002:J_Wurth_WR-DC_694106402002
- moved J6 296.4 mm to (104.0, 68.4), turned to -90 degrees
- moved J15 289.8 mm to (107.8, 129.1), turned to -90 degrees
- moved J8 272.5 mm to (152.6, 145.2), turned to 180 degrees
- moved T6 258.1 mm to (127.8, 111.5), turned to 0 degrees
- moved J7 234.9 mm to (105.6, 97.5)
- moved J14 221.2 mm to (191.6, 111.4), turned to 90 degrees
- moved D4 214.3 mm to (183.8, 48.2)
- moved F2 214.2 mm to (145.5, 136.6), turned to -90 degrees
- moved U3 212.6 mm to (183.6, 52.0)
- moved U2 212.2 mm to (148.9, 121.1)
- moved F4 206.9 mm to (147.2, 112.6), turned to -90 degrees
- moved F3 204.6 mm to (152.7, 128.4), turned to 90 degrees
- moved CR2 203.0 mm to (146.3, 131.9), turned to -90 degrees
- moved Q1 201.5 mm to (186.2, 72.6)
- moved F1 201.2 mm to (152.7, 103.7), turned to 90 degrees
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Connections:
- J14 pad 1: /ETH_CAM_DOWN_CON/ETH.X1- -> /POE_CH1 – CAM_FRONT_L/ETH.D1+
- J14 pad 2: /ETH_CAM_DOWN_CON/ETH.X1+ -> /POE_CH1 – CAM_FRONT_L/ETH.D1-
- J14 pad 3: /ETH_CAM_DOWN_CON/ETH.X2- -> /POE_CH1 – CAM_FRONT_L/ETH.D2+
- J14 pad 4: /ETH_CAM_DOWN_CON/ETH.X2+ -> /POE_CH1 – CAM_FRONT_L/ETH.D2-
- J14 pad 5: /ETH_CAM_DOWN_CON/ETH.X3- -> /POE_CH1 – CAM_FRONT_L/ETH.D3+
- J14 pad 6: /ETH_CAM_DOWN_CON/ETH.X3+ -> /POE_CH1 – CAM_FRONT_L/ETH.D3-
- J14 pad 7: /ETH_CAM_DOWN_CON/ETH.X4- -> /POE_CH1 – CAM_FRONT_L/ETH.D4+
- J14 pad 8: /ETH_CAM_DOWN_CON/ETH.X4+ -> /POE_CH1 – CAM_FRONT_L/ETH.D4-
- J15 pad 1: /M_ACOUSTICS/ETH.X1- -> /POE_CH2 – CAM_FRONT_R/ETH.D1+
- J15 pad 2: /M_ACOUSTICS/ETH.X1+ -> /POE_CH2 – CAM_FRONT_R/ETH.D1-
- J15 pad 3: /M_ACOUSTICS/ETH.X2- -> /POE_CH2 – CAM_FRONT_R/ETH.D2+
- J15 pad 4: /M_ACOUSTICS/ETH.X2+ -> /POE_CH2 – CAM_FRONT_R/ETH.D2-
- J15 pad 5: /M_ACOUSTICS/ETH.X3- -> /POE_CH2 – CAM_FRONT_R/ETH.D3+
- J15 pad 6: /M_ACOUSTICS/ETH.X3+ -> /POE_CH2 – CAM_FRONT_R/ETH.D3-
- J15 pad 7: /M_ACOUSTICS/ETH.X4- -> /POE_CH2 – CAM_FRONT_R/ETH.D4+
- J15 pad 8: /M_ACOUSTICS/ETH.X4+ -> /POE_CH2 – CAM_FRONT_R/ETH.D4-
- J6 pad 2: /CAN_CONN/CANL -> /CAN_CONN/CANH
- J6 pad 3: /CAN_CONN/CANH -> /CAN_CONN/CANL
- J8 pad 1: /M_CAM_FRONT_L/ETH.X1- -> +BATT_P
- J8 pad 2: /M_CAM_FRONT_L/ETH.X1+ -> GND
- J8 pad 3: /M_CAM_FRONT_L/ETH.X2- -> GND
- MOSFET1 pad 1: Net-(MOSFET1-Pad1) -> /PoE_PD/SEN1
- MOSFET1 pad 2: (no net) -> /PoE_PD/SEN1
- MOSFET1 pad 3: (no net) -> /PoE_PD/SEN1
- MOSFET1 pad 6: (no net) -> Net-(F1-Pad1)
- MOSFET1 pad 7: (no net) -> Net-(F1-Pad1)
- MOSFET1 pad 8: (no net) -> Net-(F1-Pad1)
- Q1 pad 1: Net-(Q1-Pad1) -> Net-(U7-SENSE)
- Q1 pad 2: Net-(L1-Pad2) -> Net-(U7-SENSE)
- Q1 pad 4: (no net) -> Net-(Q1-Pad4)
- Q1 pad 5: (no net) -> Net-(L2-Pad2)
- Q1 pad 6: (no net) -> Net-(L2-Pad2)
- Q1 pad 7: (no net) -> Net-(L2-Pad2)
- Q1 pad 8: (no net) -> Net-(L2-Pad2)
- Q1 pad 9: (no net) -> Net-(L2-Pad2)
- T1 pad 13: /M_CAM_FRONT_L/X4- -> /M_CAM_FRONT_L/ETH.X4-
- T1 pad 14: /M_CAM_FRONT_L/X4+ -> /M_CAM_FRONT_L/ETH.X4+
- T1 pad 16: /M_CAM_FRONT_L/X3- -> /M_CAM_FRONT_L/ETH.X3-
- T1 pad 17: /M_CAM_FRONT_L/X3+ -> /M_CAM_FRONT_L/ETH.X3+
- T1 pad 19: /M_CAM_FRONT_L/X2- -> /M_CAM_FRONT_L/ETH.X2-
- T1 pad 20: /M_CAM_FRONT_L/X2+ -> /M_CAM_FRONT_L/ETH.X2+
- T1 pad 22: /M_CAM_FRONT_L/X1- -> /M_CAM_FRONT_L/ETH.X1-
- T1 pad 23: /M_CAM_FRONT_L/X1+ -> /M_CAM_FRONT_L/ETH.X1+
- T4 pad 13: /M_CAM_FRONT_R/X4- -> /M_CAM_FRONT_R/ETH.X4-
- T4 pad 14: /M_CAM_FRONT_R/X4+ -> /M_CAM_FRONT_R/ETH.X4+
- T4 pad 16: /M_CAM_FRONT_R/X3- -> /M_CAM_FRONT_R/ETH.X3-
- T4 pad 17: /M_CAM_FRONT_R/X3+ -> /M_CAM_FRONT_R/ETH.X3+
- T4 pad 19: /M_CAM_FRONT_R/X2- -> /M_CAM_FRONT_R/ETH.X2-
- T4 pad 20: /M_CAM_FRONT_R/X2+ -> /M_CAM_FRONT_R/ETH.X2+
- T4 pad 22: /M_CAM_FRONT_R/X1- -> /M_CAM_FRONT_R/ETH.X1-
- T4 pad 23: /M_CAM_FRONT_R/X1+ -> /M_CAM_FRONT_R/ETH.X1+
- T4 pad 9: /POE_CH2 – CAM_FRONT_R/ETH.D3+ -> /POE_CH2 – CAM_FRONT_R/ETH.D3-
- T5 pad 13: /M_CAM_DOWN/X4- -> /ETH_CAM_DOWN_CON/ETH.X4-
- T5 pad 14: /M_CAM_DOWN/X4+ -> /ETH_CAM_DOWN_CON/ETH.X4+
- T5 pad 16: /M_CAM_DOWN/X3- -> /ETH_CAM_DOWN_CON/ETH.X3-
- T5 pad 17: /M_CAM_DOWN/X3+ -> /ETH_CAM_DOWN_CON/ETH.X3+
- T5 pad 19: /M_CAM_DOWN/X2- -> /ETH_CAM_DOWN_CON/ETH.X2-
- T5 pad 20: /M_CAM_DOWN/X2+ -> /ETH_CAM_DOWN_CON/ETH.X2+
- T5 pad 22: /M_CAM_DOWN/X1- -> /ETH_CAM_DOWN_CON/ETH.X1-
- T5 pad 23: /M_CAM_DOWN/X1+ -> /ETH_CAM_DOWN_CON/ETH.X1+
- T6 pad 13: /M_ACOUSTICS/X4- -> /ETH_ACOUSTICS_CON/ETH.X4-
- T6 pad 14: /M_ACOUSTICS/X4+ -> /ETH_ACOUSTICS_CON/ETH.X4+
- T6 pad 16: /M_ACOUSTICS/X3- -> /ETH_ACOUSTICS_CON/ETH.X3-
- T6 pad 17: /M_ACOUSTICS/X3+ -> /ETH_ACOUSTICS_CON/ETH.X3+
- T6 pad 19: /M_ACOUSTICS/X2- -> /ETH_ACOUSTICS_CON/ETH.X2-
- T6 pad 20: /M_ACOUSTICS/X2+ -> /ETH_ACOUSTICS_CON/ETH.X2+
- T6 pad 22: /M_ACOUSTICS/X1- -> /ETH_ACOUSTICS_CON/ETH.X1-
- T6 pad 23: /M_ACOUSTICS/X1+ -> /ETH_ACOUSTICS_CON/ETH.X1+
- U3 pad 4: /eFuse/FLT -> unconnected-(U3-RCBCTRL-Pad4)
- U8 pad 1: Net-(L1-Pad2) -> Net-(L2-Pad2)
- U8 pad 2: +48V -> Net-(L2-Pad2)
- U8 pad 3: (no net) -> +48V
Routing:
- net +48V: track 0.00 -> 202.7 mm, vias 0 -> 19
- net +BATT_P: track 0.00 -> 131.7 mm, vias 0 -> 7
- net +3V3: track 0.00 -> 67.4 mm, vias 0 -> 2
- net /M_CAM_FRONT_R/ETH.X4-: track 0.00 -> 48.8 mm
- net /ETH_CAM_DOWN_CON/ETH.X1-: track 0.00 -> 47.2 mm
- net /M_CAM_FRONT_R/ETH.X4+: track 0.00 -> 46.1 mm
- net /ETH_CAM_DOWN_CON/ETH.X1+: track 0.00 -> 45.6 mm
- net /M_CAM_FRONT_R/ETH.X3-: track 0.00 -> 44.5 mm
- net /ETH_CAM_DOWN_CON/ETH.X2-: track 0.00 -> 42.6 mm
- net Net-(U2-DRAIN2): track 0.00 -> 42.0 mm, vias 0 -> 1
- net /M_CAM_FRONT_R/ETH.X3+: track 0.00 -> 41.8 mm
- net /ETH_CAM_DOWN_CON/ETH.X2+: track 0.00 -> 41.0 mm
- net /CAN_CONN/PWM: track 0.00 -> 40.9 mm
- net /M_CAM_FRONT_R/ETH.X2-: track 0.00 -> 40.0 mm
- net /ETH_CAM_DOWN_CON/ETH.X3-: track 0.00 -> 38.2 mm
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- added copper zone on B.Cu, net +48V
- added copper zone on F.Cu, net +48V
- added copper zone on B.Cu, net +BATT
- added copper zone on F.Cu, net +BATT
- added copper zone on In2.Cu, net +BATT
- added copper zone on F.Cu, net +BATT_P
- added copper zone on In2.Cu, net +BATT_P
- added copper zone on F.Cu, net /M_CAM_FRONT_L/POE1_N
- added copper zone on B.Cu, net /PoE_PD/Drain2
- added copper zone on B.Cu, net /PoE_PD/SEN1
- added copper zone on F.Cu, net GND
- added copper zone on In1.Cu, net GND
- added copper zone on In2.Cu, net GND
- added copper zone on B.Cu, net Net-(F1-Pad1)
- added copper zone on B.Cu, net Net-(F3-Pad1)
- added copper zone on B.Cu, net Net-(F4-Pad1)
- added copper zone on F.Cu, net Net-(L2-Pad2)
- added copper zone on B.Cu, net Net-(MOSFET2-Pad1)
- added copper zone on B.Cu, net Net-(MOSFET3-Pad1)
- added copper zone on B.Cu, net Net-(MOSFET4-Pad1)
- added copper zone on B.Cu, net Net-(U3-EN_UVLO)
- added copper zone on B.Cu, net Net-(U3-OVLO)
- added copper zone on F.Cu, net Net-(U7-SENSE)
Other:
- board size 120 x 136.8 mm -> 110 x 120.8 mm
- copper layers 2 -> 4
- board text added: "CAN"
- board text added: "GBX"
- board text added: "GBX-R"
- board text added: "IN ACOU"
- board text added: "IN CAM DN"
- board text added: "IN CAM FL"
- board text added: "IN CAM FR"
- board text added: "May Viking bless this board"
- board text added: "O ACOU"
- board text added: "O CAM DN"
- board text added: "O CAM FL"
- board text added: "O CAM FR"
- board text added: "OUTPUT"

Commit message: Still developing
Parts:
- removed C22: C_Small, Capacitor_SMD:C_0603_1608Metric_Pad1.08x0.95mm_HandSolder
- removed J14, J15, J16: 634008138121, 615008138021:J_Wurth_WR-MJ_634008138121
- removed J7: 64600211622, Wurth_WR-WTB:J_Wurth_WR-WTB_64600211622
- removed REF**: MATE_WR-TBL_691379180024, mate-connectors:MATE_WR-TBL_691379180024
- removed U1: 173950336, 173950336:U_Wurth_WPME-FDSM_17395xx36
- added C25: 4.7uF, Capacitor_SMD:C_0603_1608Metric_Pad1.08x0.95mm_HandSolder, B.Cu at (146.8, 124.6)
- added C62: 4.7uF, Capacitor_SMD:C_0603_1608Metric_Pad1.08x0.95mm_HandSolder, F.Cu at (148.0, 132.0)
- added C63: 22uF, Capacitor_SMD:C_0603_1608Metric_Pad1.08x0.95mm_HandSolder, F.Cu at (152.5, 132.0)
- added J1: 691323100002, 691378140024-2:J_Wurth_WR-TBL_691323100002, F.Cu at (154.3, 146.2)
- added J21: 64600411622, Wurth_WR-WTB:J_Wurth_WR-WTB_64600411622, F.Cu at (196.7, 95.8)
- added J9: 615008160421, 615008160421:J_Wurth_WR-MJ_615008160421, F.Cu at (113.0, 123.9)
- added L3: 1pH, Inductor_SMD:L_0603_1608Metric, B.Cu at (146.8, 126.4)
- added U4: 173950336, 173950336:U_Wurth_WPME-FDSM_17395xx36, F.Cu at (147.6, 128.6)
- C5, C6, C7, R6: moved to F.Cu
- CR1, CR2, CR3, CR4, L2, R3, U7: moved to B.Cu
- J10: value 691378140024 -> 694106402002; footprint 691378140024-2:J_Wurth_WR-TBL_691378140024 -> 694106402002:J_Wurth_WR-DC_694106402002
- J11: value 64600411622 -> 615008160421; footprint Wurth_WR-WTB:J_Wurth_WR-WTB_64600411622 -> 615008138021-THT:J_Wurth_WR-MJ_615008160421
- J17: value 634008138121 -> 64600411622; footprint 615008138021:J_Wurth_WR-MJ_634008138121 -> Wurth_WR-WTB:J_Wurth_WR-WTB_64600411622
- J2: value 615008142521 -> 615008160421; footprint 615008138021-THT:J_Wurth_WR-MJ_615008142521 -> 615008160421:J_Wurth_WR-MJ_615008160421
- J3, J4, J5: value 615008142521 -> 615008160721; footprint 615008138021-THT:J_Wurth_WR-MJ_615008142521 -> 615008160721:J_Wurth_WR-MJ_615008160721
- J6: value 653104131822 -> 615008160721; footprint Wurth_WR-WTB:J_Wurth_WR-WTB_653104131822 -> 615008160721:J_Wurth_WR-MJ_615008160721
- J8: value 694106402002 -> 615008160421; footprint 694106402002:J_Wurth_WR-DC_694106402002 -> 615008160421:J_Wurth_WR-MJ_615008160421
- moved R3 114.8 mm to (129.7, 151.1), turned to -90 degrees
- moved R2 113.9 mm to (124.6, 147.4)
- moved C4 113.9 mm to (129.7, 151.1), turned to -90 degrees
- moved R1 111.8 mm to (126.4, 147.4)
- moved C11 107.3 mm to (124.6, 143.1)
- moved C1 107.3 mm to (126.4, 143.1)
- moved R6 107.1 mm to (132.0, 147.9), turned to 180 degrees
- moved R7 106.5 mm to (134.7, 147.9)
- moved R5 104.5 mm to (131.5, 151.1)
- moved U7 103.2 mm to (130.0, 143.9), turned to -90 degrees
- moved C3 102.3 mm to (133.3, 151.1)
- moved R4 99.9 mm to (122.9, 143.1)
- moved R9 98.4 mm to (121.6, 137.2), turned to 90 degrees
- moved C2 98.1 mm to (121.2, 143.1), turned to 90 degrees
- moved C8 96.4 mm to (172.9, 140.9)
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Connections:
- net /M_ACOUSTICS/POE2_N renamed /M_ACOUSTICS/POE4_N
- J10 pad 1: +BATT -> +BATT_P
- J10 pad 3: unconnected-(J10-Pad3) -> GND
- J11 pad 1: GND -> /ETH.D1+
- J11 pad 2: GND -> /ETH.D1-
- J11 pad 3: +BATT_P -> /ETH.D2+
- J11 pad 4: +BATT_P -> /ETH.D2-
- J17 pad 1: /POE_CH4 – ACOUSTICS/ETH.D1+ -> GND
- J17 pad 2: /POE_CH4 – ACOUSTICS/ETH.D1- -> GND
- J17 pad 3: /POE_CH4 – ACOUSTICS/ETH.D2+ -> +BATT_P
- J17 pad 4: /POE_CH4 – ACOUSTICS/ETH.D2- -> +BATT_P
- J2 pad 1: /M_CAM_FRONT_L/ETH.X4- -> /ETH.D1+
- J2 pad 2: /M_CAM_FRONT_L/ETH.X4+ -> /ETH.D1-
- J2 pad 3: /M_CAM_FRONT_L/ETH.X3- -> /ETH.D2+
- J2 pad 4: /M_CAM_FRONT_L/ETH.X3+ -> /ETH.D2-
- J2 pad 5: /M_CAM_FRONT_L/ETH.X2- -> /ETH.D3+
- J2 pad 6: /M_CAM_FRONT_L/ETH.X2+ -> /ETH.D3-
- J2 pad 7: /M_CAM_FRONT_L/ETH.X1- -> /ETH.D4+
- J2 pad 8: /M_CAM_FRONT_L/ETH.X1+ -> /ETH.D4-
- J3 pad 1: /M_CAM_FRONT_R/ETH.X1+ -> /ETH.X4-
- J3 pad 2: /M_CAM_FRONT_R/ETH.X1- -> /ETH.X4+
- J3 pad 3: /M_CAM_FRONT_R/ETH.X2+ -> /ETH.X3-
- J3 pad 4: /M_CAM_FRONT_R/ETH.X2- -> /ETH.X3+
- J3 pad 5: /M_CAM_FRONT_R/ETH.X3+ -> /ETH.X2-
- J3 pad 6: /M_CAM_FRONT_R/ETH.X3- -> /ETH.X2+
- J3 pad 7: /M_CAM_FRONT_R/ETH.X4+ -> /ETH.X1-
- J3 pad 8: /M_CAM_FRONT_R/ETH.X4- -> /ETH.X1+
- J4 pad 1: /ETH_CAM_DOWN_CON/ETH.X1+ -> /ETH.X4-
- J4 pad 2: /ETH_CAM_DOWN_CON/ETH.X1- -> /ETH.X4+
- J4 pad 3: /ETH_CAM_DOWN_CON/ETH.X2+ -> /ETH.X3-
- J4 pad 4: /ETH_CAM_DOWN_CON/ETH.X2- -> /ETH.X3+
- J4 pad 5: /ETH_CAM_DOWN_CON/ETH.X3+ -> /ETH.X2-
- J4 pad 6: /ETH_CAM_DOWN_CON/ETH.X3- -> /ETH.X2+
- J4 pad 7: /ETH_CAM_DOWN_CON/ETH.X4+ -> /ETH.X1-
- J4 pad 8: /ETH_CAM_DOWN_CON/ETH.X4- -> /ETH.X1+
- J5 pad 1: /ETH_ACOUSTICS_CON/ETH.X4- -> /ETH.X1+
- J5 pad 2: /ETH_ACOUSTICS_CON/ETH.X4+ -> /ETH.X1-
- J5 pad 3: /ETH_ACOUSTICS_CON/ETH.X3- -> /ETH.X2+
- J5 pad 4: /ETH_ACOUSTICS_CON/ETH.X3+ -> /ETH.X2-
- J5 pad 5: /ETH_ACOUSTICS_CON/ETH.X2- -> /ETH.X3+
- J5 pad 6: /ETH_ACOUSTICS_CON/ETH.X2+ -> /ETH.X3-
- J5 pad 7: /ETH_ACOUSTICS_CON/ETH.X1- -> /ETH.X4+
- J5 pad 8: /ETH_ACOUSTICS_CON/ETH.X1+ -> /ETH.X4-
- J6 pad 1: /CAN_CONN/PWM -> /ETH.X4-
- J6 pad 2: /CAN_CONN/CANH -> /ETH.X4+
- J6 pad 3: /CAN_CONN/CANL -> /ETH.X3-
- J6 pad 4: GND -> /ETH.X3+
- J8 pad 1: +BATT_P -> /ETH.D4-
- J8 pad 2: GND -> /ETH.D4+
- J8 pad 3: GND -> /ETH.D3-
- T1 pad 11: /POE_CH1 – CAM_FRONT_L/ETH.D4+ -> /ETH.D4+
- T1 pad 12: /POE_CH1 – CAM_FRONT_L/ETH.D4- -> /ETH.D4-
- T1 pad 13: /M_CAM_FRONT_L/ETH.X4- -> /ETH.X4-
- T1 pad 14: /M_CAM_FRONT_L/ETH.X4+ -> /ETH.X4+
- T1 pad 16: /M_CAM_FRONT_L/ETH.X3- -> /ETH.X3-
- T1 pad 17: /M_CAM_FRONT_L/ETH.X3+ -> /ETH.X3+
- T1 pad 19: /M_CAM_FRONT_L/ETH.X2- -> /ETH.X2-
- T1 pad 2: /POE_CH1 – CAM_FRONT_L/ETH.D1+ -> /ETH.D1+
- T1 pad 20: /M_CAM_FRONT_L/ETH.X2+ -> /ETH.X2+
- T1 pad 22: /M_CAM_FRONT_L/ETH.X1- -> /ETH.X1-
- T1 pad 23: /M_CAM_FRONT_L/ETH.X1+ -> /ETH.X1+
- T1 pad 3: /POE_CH1 – CAM_FRONT_L/ETH.D1- -> /ETH.D1-
- T1 pad 5: /POE_CH1 – CAM_FRONT_L/ETH.D2+ -> /ETH.D2+
- T1 pad 6: /POE_CH1 – CAM_FRONT_L/ETH.D2- -> /ETH.D2-
- T1 pad 8: /POE_CH1 – CAM_FRONT_L/ETH.D3+ -> /ETH.D3+
- T1 pad 9: /POE_CH1 – CAM_FRONT_L/ETH.D3- -> /ETH.D3-
- T4 pad 11: /POE_CH2 – CAM_FRONT_R/ETH.D4+ -> /ETH.D4+
- T4 pad 12: /POE_CH2 – CAM_FRONT_R/ETH.D4- -> /ETH.D4-
- T4 pad 13: /M_CAM_FRONT_R/ETH.X4- -> /ETH.X4-
- T4 pad 14: /M_CAM_FRONT_R/ETH.X4+ -> /ETH.X4+
- T4 pad 16: /M_CAM_FRONT_R/ETH.X3- -> /ETH.X3-
- T4 pad 17: /M_CAM_FRONT_R/ETH.X3+ -> /ETH.X3+
- T4 pad 19: /M_CAM_FRONT_R/ETH.X2- -> /ETH.X2-
- T4 pad 2: /POE_CH2 – CAM_FRONT_R/ETH.D1+ -> /ETH.D1+
- T4 pad 20: /M_CAM_FRONT_R/ETH.X2+ -> /ETH.X2+
- T4 pad 22: /M_CAM_FRONT_R/ETH.X1- -> /ETH.X1-
- T4 pad 23: /M_CAM_FRONT_R/ETH.X1+ -> /ETH.X1+
- T4 pad 3: /POE_CH2 – CAM_FRONT_R/ETH.D1- -> /ETH.D1-
- T4 pad 5: /POE_CH2 – CAM_FRONT_R/ETH.D2+ -> /ETH.D2+
- T4 pad 6: /POE_CH2 – CAM_FRONT_R/ETH.D2- -> /ETH.D2-
- T4 pad 8: /POE_CH2 – CAM_FRONT_R/ETH.D3+ -> /ETH.D3+
- T4 pad 9: /POE_CH2 – CAM_FRONT_R/ETH.D3- -> /ETH.D3-
- T5 pad 11: /POE_CH3 – CAM_DOWN/ETH.D4+ -> /ETH.D4+
- T5 pad 12: /POE_CH3 – CAM_DOWN/ETH.D4- -> /ETH.D4-
- T5 pad 13: /ETH_CAM_DOWN_CON/ETH.X4- -> /ETH.X4-
- T5 pad 14: /ETH_CAM_DOWN_CON/ETH.X4+ -> /ETH.X4+
- T5 pad 16: /ETH_CAM_DOWN_CON/ETH.X3- -> /ETH.X3-
- T5 pad 17: /ETH_CAM_DOWN_CON/ETH.X3+ -> /ETH.X3+
- T5 pad 19: /ETH_CAM_DOWN_CON/ETH.X2- -> /ETH.X2-
- T5 pad 2: /POE_CH3 – CAM_DOWN/ETH.D1+ -> /ETH.D1+
- T5 pad 20: /ETH_CAM_DOWN_CON/ETH.X2+ -> /ETH.X2+
- T5 pad 22: /ETH_CAM_DOWN_CON/ETH.X1- -> /ETH.X1-
- T5 pad 23: /ETH_CAM_DOWN_CON/ETH.X1+ -> /ETH.X1+
- T5 pad 3: /POE_CH3 – CAM_DOWN/ETH.D1- -> /ETH.D1-
- T5 pad 5: /POE_CH3 – CAM_DOWN/ETH.D2+ -> /ETH.D2+
- T5 pad 6: /POE_CH3 – CAM_DOWN/ETH.D2- -> /ETH.D2-
- T5 pad 8: /POE_CH3 – CAM_DOWN/ETH.D3+ -> /ETH.D3+
- T5 pad 9: /POE_CH3 – CAM_DOWN/ETH.D3- -> /ETH.D3-
- T6 pad 11: /POE_CH4 – ACOUSTICS/ETH.D4+ -> /ETH.D4+
- T6 pad 12: /POE_CH4 – ACOUSTICS/ETH.D4- -> /ETH.D4-
- T6 pad 13: /ETH_ACOUSTICS_CON/ETH.X4- -> /ETH.X4-
- T6 pad 14: /ETH_ACOUSTICS_CON/ETH.X4+ -> /ETH.X4+
- T6 pad 16: /ETH_ACOUSTICS_CON/ETH.X3- -> /ETH.X3-
- T6 pad 17: /ETH_ACOUSTICS_CON/ETH.X3+ -> /ETH.X3+
- T6 pad 19: /ETH_ACOUSTICS_CON/ETH.X2- -> /ETH.X2-
- T6 pad 2: /POE_CH4 – ACOUSTICS/ETH.D1+ -> /ETH.D1+
- T6 pad 20: /ETH_ACOUSTICS_CON/ETH.X2+ -> /ETH.X2+
- T6 pad 22: /ETH_ACOUSTICS_CON/ETH.X1- -> /ETH.X1-
- T6 pad 23: /ETH_ACOUSTICS_CON/ETH.X1+ -> /ETH.X1+
- T6 pad 3: /POE_CH4 – ACOUSTICS/ETH.D1- -> /ETH.D1-
- T6 pad 5: /POE_CH4 – ACOUSTICS/ETH.D2+ -> /ETH.D2+
- T6 pad 6: /POE_CH4 – ACOUSTICS/ETH.D2- -> /ETH.D2-
- T6 pad 8: /POE_CH4 – ACOUSTICS/ETH.D3+ -> /ETH.D3+
- T6 pad 9: /POE_CH4 – ACOUSTICS/ETH.D3- -> /ETH.D3-
Routing:
- net +48V: track 202.7 -> 2.11 mm, vias 19 -> 0
- net +BATT_P: track 131.7 -> 0.00 mm, vias 7 -> 0
- net /ETH.D2+: track 0.00 -> 105.6 mm
- net /ETH.D1+: track 0.00 -> 102.7 mm
- net /ETH.D2-: track 0.00 -> 101.0 mm
- net /ETH.D1-: track 0.00 -> 98.0 mm
- net +3V3: track 67.4 -> 0.00 mm, vias 2 -> 0
- net /ETH.D3+: track 0.00 -> 51.6 mm
- net /ETH.D4-: track 0.00 -> 49.0 mm
- net /M_CAM_FRONT_R/ETH.X4-: track 48.8 -> 0.00 mm
- net /ETH.D4+: track 0.00 -> 48.2 mm
- net /ETH.D3-: track 0.00 -> 47.9 mm
- net /ETH_CAM_DOWN_CON/ETH.X1-: track 47.2 -> 0.00 mm
- net /M_CAM_FRONT_R/ETH.X4+: track 46.1 -> 0.00 mm
- net /ETH_CAM_DOWN_CON/ETH.X1+: track 45.6 -> 0.00 mm
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- removed copper zone on B.Cu, net +48V
- removed copper zone on F.Cu, net +48V
- removed copper zone on B.Cu, net +BATT
- removed copper zone on F.Cu, net +BATT
- removed copper zone on In2.Cu, net +BATT
- removed copper zone on F.Cu, net +BATT_P
- removed copper zone on In2.Cu, net +BATT_P
- removed copper zone on F.Cu, net /M_CAM_FRONT_L/POE1_N
- removed copper zone on B.Cu, net /PoE_PD/Drain2
- removed copper zone on B.Cu, net /PoE_PD/SEN1
- removed copper zone on F.Cu, net GND
- removed copper zone on In1.Cu, net GND
- removed copper zone on In2.Cu, net GND
- removed copper zone on B.Cu, net Net-(F1-Pad1)
- removed copper zone on B.Cu, net Net-(F3-Pad1)
- removed copper zone on B.Cu, net Net-(F4-Pad1)
- removed copper zone on F.Cu, net Net-(L2-Pad2)
- removed copper zone on B.Cu, net Net-(MOSFET2-Pad1)
- removed copper zone on B.Cu, net Net-(MOSFET3-Pad1)
- removed copper zone on B.Cu, net Net-(MOSFET4-Pad1)
- removed copper zone on B.Cu, net Net-(U3-EN_UVLO)
- removed copper zone on B.Cu, net Net-(U3-OVLO)
- removed copper zone on F.Cu, net Net-(U7-SENSE)
Other:
- outline, holes or cut-outs redrawn
- board text removed: "CAN"
